Commit message: Update tron2/WF_TRON2/urdf/robot.urdf

File: tron2/WF_TRON2/urdf/robot.urdf (robot description, URDF)
Before this commit: robot Tron2, 12 links, 11 joints
Joints:
- joint hip_L_Joint: limit lower=-0.260577657323 upper=3.40339204139 effort=100.0 velocity=15.0 -> lower=-0.260577657323 upper=3.40339204139 effort=80.0 velocity=15.0
- joint yaw_R_Joint: limit lower=-1.50098315672 upper=2.70526034059 effort=20.0 velocity=15.0 -> lower=-1.50098315672 upper=2.70526034059 effort=80.0 velocity=15.0
