Commit message: Feat: 双臂拿掉夹爪

File: tron2/ARM_TRON2A/meshes/robot.urdf (robot description, URDF)
Before this commit: robot ARM_TRON2A, 19 links, 18 joints
Links:
- removed link grasper_L_Link
- removed link grasper_R_Link
Joints:
- removed joint grasper_L_Joint
- removed joint grasper_R_Joint

File: tron2/ARM_TRON2A/urdf/robot.urdf (robot description, URDF)
Before this commit: robot ARM_TRON2A, 19 links, 18 joints
Links:
- removed link grasper_L_Link
- removed link grasper_R_Link
Joints:
- removed joint grasper_L_Joint
- removed joint grasper_R_Joint
