Commit message: modify

File: tron2/ARM_TRON2A/urdf/robot.urdf (robot description, URDF)
Before this commit: robot ARM_TRON2A, 17 links, 16 joints
Links:
- added link left_hand_contact, mass 0.00000001; visual box size=0.001 0.001 0.001
- added link right_hand_contact, mass 0.00000001; visual box size=0.001 0.001 0.001
Joints:
- added joint left_hand_contact_joint: type fixed, parent wrist_roll_L_Link, child left_hand_contact, origin xyz=0 0 0 rpy=0 0 0
- added joint right_hand_contact_joint: type fixed, parent wrist_roll_R_Link, child right_hand_contact, origin xyz=0 0 0 rpy=0 0 0
