Commit message: Feat: TRON2_2.5版本urdf初始化

File: tron2/SF_TRON2/meshes/robot.urdf (robot description, URDF)
Before this commit: robot bipedal_robot, 12 links, 11 joints
Links:
- removed link wheel_L_Link
- removed link wheel_R_Link
- added link foot_L_Link, mass 0.94793; collision mesh filename=/home/wen/robot/urdf/transfer/output/SF_TRON2/urdf/meshes/f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; visual mesh filename=/home/wen/robot/urdf/transfer/output/SF_TRON2/urdf/meshes/f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
- added link foot_R_Link, mass 0.94793; collision mesh filename=/home/wen/robot/urdf/transfer/output/SF_TRON2/urdf/meshes/f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; visual mesh filename=/home/wen/robot/urdf/transfer/output/SF_TRON2/urdf/meshes/f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
- link abad_L_Link: geometry collision mesh filename=/home/wen/robot/urdf/transfer/output/SF_TRON2/urdf/meshes/a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; visual mesh filename=/home/wen/robot/urdf/transfer/output/SF_TRON2/urdf/meshes/a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
- link abad_R_Link: geometry collision mesh filename=/home/wen/robot/urdf/transfer/output/SF_TRON2/urdf/meshes/a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; visual mesh filename=/home/wen/robot/urdf/transfer/output/SF_TRON2/urdf/meshes/a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
- link base_Link: geometry collision mesh filename=/home/wen/robot/urdf/transfer/output/SF_TRON2/urdf/meshes/b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; visual mesh filename=/home/wen/robot/urdf/transfer/output/SF_TRON2/urdf/meshes/b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
- link hip_L_Link: geometry collision mesh filename=/home/wen/robot/urdf/transfer/output/SF_TRON2/urdf/meshes/h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; visual mesh filename=/home/wen/robot/urdf/transfer/output/SF_TRON2/urdf/meshes/h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
- link hip_R_Link: geometry collision mesh filename=/home/wen/robot/urdf/transfer/output/SF_TRON2/urdf/meshes/h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; visual mesh filename=/home/wen/robot/urdf/transfer/output/SF_TRON2/urdf/meshes/h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
- link knee_L_Link: mass 1.9798 -> 1.84166; geometry collision mesh filename=/home/wen/robot/urdf/transfer/output/SF_TRON2/urdf/meshes/k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; visual mesh filename=/home/wen/robot/urdf/transfer/output/SF_TRON2/urdf/meshes/k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
- link knee_R_Link: mass 1.9798 -> 1.84166; geometry collision mesh filename=/home/wen/robot/urdf/transfer/output/SF_TRON2/urdf/meshes/k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; visual mesh filename=/home/wen/robot/urdf/transfer/output/SF_TRON2/urdf/meshes/k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
- link yaw_L_Link: geometry collision mesh filename=/home/wen/robot/urdf/transfer/output/SF_TRON2/urdf/meshes/y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; visual mesh filename=/home/wen/robot/urdf/transfer/output/SF_TRON2/urdf/meshes/y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
- link yaw_R_Link: geometry collision mesh filename=/home/wen/robot/urdf/transfer/output/SF_TRON2/urdf/meshes/y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; visual mesh filename=/home/wen/robot/urdf/transfer/output/SF_TRON2/urdf/meshes/y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
Joints:
- removed joint wheel_L_Joint
- removed joint wheel_R_Joint
- added joint foot_L_Joint: type revolute, parent knee_L_Link, child foot_L_Link, origin xyz=-0.15601 0.07805 -0.31331 rpy=0 0 0, axis 0 1 0, limit lower=1.2482594810263443 upper=-2.230356251123554 effort=40 velocity=31.83
- added joint foot_R_Joint: type revolute, parent knee_R_Link, child foot_R_Link, origin xyz=-0.15601 -0.00425 -0.31331 rpy=0 0 0, axis 0 1 0, limit lower=1.2482594810263443 upper=-2.230356251123554 effort=40 velocity=31.83
- joint abad_L_Joint: limit lower=-3.5894441396515377 upper=2.1526890994098062 effort=140 velocity=12.57 -> lower=-2.679429467661695 upper=3.062703771399649 effort=140 velocity=12.57; origin xyz=-0.00049 0.10649 0.0586 rpy=0 0 0 -> xyz=0.00049 0.10649 0.0586 rpy=0 0 0
- joint abad_R_Joint: limit lower=-3.5894441396515377 upper=2.1526890994098062 effort=140 velocity=12.57 -> lower=-2.679429467661695 upper=3.062703771399649 effort=140 velocity=12.57
- joint hip_L_Joint: axis 0.90138 0 -0.43303 -> 0.89509 0 0.44589; origin xyz=0.0448 0.062 -0.02152 rpy=0 0 0 -> xyz=0.04449 0.062 0.02216 rpy=0 0 0
- joint hip_R_Joint: axis 0.90138 0 -0.43303 -> 0.89509 0 0.44589; limit lower=-0.2605776573227534 upper=2.1131489961203007 effort=140 velocity=12.57 -> lower=-2.1131489961203007 upper=0.2605776573227534 effort=140 velocity=12.57; origin xyz=-0.0448 -0.062 0.02152 rpy=0 0 0 -> xyz=-0.04449 -0.062 -0.02216 rpy=0 0 0
- joint knee_L_Joint: limit lower=-1.7221163729428048 upper=2.7693139241394027 effort=140 velocity=12.57 -> lower=-1.6938420390604967 upper=2.7410395902570945 effort=140 velocity=12.57; origin xyz=-0.10276 -0.04115 -0.21389 rpy=0 0 0 -> xyz=0.10581 -0.04115 -0.2124 rpy=0 0 0
- joint knee_R_Joint: limit lower=-1.7221163729428048 upper=2.7693139241394027 effort=140 velocity=12.57 -> lower=-1.6938420390604967 upper=2.7410395902570945 effort=140 velocity=12.57; origin xyz=-0.10276 0.04115 -0.21389 rpy=0 0 0 -> xyz=0.10581 0.04115 -0.2124 rpy=0 0 0
- joint yaw_L_Joint: axis -0.43303 0 0.90138 -> -0.44589 0 0.89509; origin xyz=-0.0936 0.0 -0.08006 rpy=0 0 0 -> xyz=0.00577 0.0 -0.12304 rpy=0 0 0
- joint yaw_R_Joint: axis -0.43303 0 0.90138 -> -0.44589 0 0.89509; origin xyz=-0.004 0.0 -0.12311 rpy=0 0 0 -> xyz=0.09474 0.0 -0.07872 rpy=0 0 0

File: tron2/SF_TRON2/urdf/robot.urdf (robot description, URDF)
Before this commit: robot bipedal_robot, 12 links, 11 joints
Links:
- removed link wheel_L_Link
- removed link wheel_R_Link
- added link foot_L_Link, mass 0.94793; collision mesh filename=package://sf_robot/meshes/foot_L_Link.STL; visual mesh filename=package://sf_robot/meshes/foot_L_Link.STL
- added link foot_R_Link, mass 0.94793; collision mesh filename=package://sf_robot/meshes/foot_R_Link.STL; visual mesh filename=package://sf_robot/meshes/foot_R_Link.STL
- link abad_L_Link: geometry collision mesh filename=package://sf_robot/meshes/abad_L_Link.STL; visual mesh filename=package://sf_robot/meshes/abad_L_Link.STL
- link abad_R_Link: geometry collision mesh filename=package://sf_robot/meshes/abad_R_Link.STL; visual mesh filename=package://sf_robot/meshes/abad_R_Link.STL
- link base_Link: geometry collision mesh filename=package://sf_robot/meshes/base_Link.STL; visual mesh filename=package://sf_robot/meshes/base_Link.STL
- link hip_L_Link: geometry collision mesh filename=package://sf_robot/meshes/hip_L_Link.STL; visual mesh filename=package://sf_robot/meshes/hip_L_Link.STL
- link hip_R_Link: geometry collision mesh filename=package://sf_robot/meshes/hip_R_Link.STL; visual mesh filename=package://sf_robot/meshes/hip_R_Link.STL
- link knee_L_Link: mass 1.9798 -> 1.84166; geometry collision mesh filename=package://sf_robot/meshes/knee_L_Link.STL; visual mesh filename=package://sf_robot/meshes/knee_L_Link.STL
- link knee_R_Link: mass 1.9798 -> 1.84166; geometry collision mesh filename=package://sf_robot/meshes/knee_R_Link.STL; visual mesh filename=package://sf_robot/meshes/knee_R_Link.STL
- link yaw_L_Link: geometry collision mesh filename=package://sf_robot/meshes/yaw_L_Link.STL; visual mesh filename=package://sf_robot/meshes/yaw_L_Link.STL
- link yaw_R_Link: geometry collision mesh filename=package://sf_robot/meshes/yaw_R_Link.STL; visual mesh filename=package://sf_robot/meshes/yaw_R_Link.STL
Joints:
- removed joint wheel_L_Joint
- removed joint wheel_R_Joint
- added joint foot_L_Joint: type revolute, parent knee_L_Link, child foot_L_Link, origin xyz=-0.15601 0.07805 -0.31331 rpy=0 0 0, axis 0 1 0, limit lower=1.2482594810263443 upper=-2.230356251123554 effort=40 velocity=31.83
- added joint foot_R_Joint: type revolute, parent knee_R_Link, child foot_R_Link, origin xyz=-0.15601 -0.00425 -0.31331 rpy=0 0 0, axis 0 1 0, limit lower=1.2482594810263443 upper=-2.230356251123554 effort=40 velocity=31.83
- joint abad_L_Joint: limit lower=-3.5894441396515377 upper=2.1526890994098062 effort=140 velocity=12.57 -> lower=-2.679429467661695 upper=3.062703771399649 effort=140 velocity=12.57; origin xyz=-0.00049 0.10649 0.0586 rpy=0 0 0 -> xyz=0.00049 0.10649 0.0586 rpy=0 0 0
- joint abad_R_Joint: limit lower=-3.5894441396515377 upper=2.1526890994098062 effort=140 velocity=12.57 -> lower=-2.679429467661695 upper=3.062703771399649 effort=140 velocity=12.57
- joint hip_L_Joint: axis 0.90138 0 -0.43303 -> 0.89509 0 0.44589; origin xyz=0.0448 0.062 -0.02152 rpy=0 0 0 -> xyz=0.04449 0.062 0.02216 rpy=0 0 0
- joint hip_R_Joint: axis 0.90138 0 -0.43303 -> 0.89509 0 0.44589; limit lower=-0.2605776573227534 upper=2.1131489961203007 effort=140 velocity=12.57 -> lower=-2.1131489961203007 upper=0.2605776573227534 effort=140 velocity=12.57; origin xyz=-0.0448 -0.062 0.02152 rpy=0 0 0 -> xyz=-0.04449 -0.062 -0.02216 rpy=0 0 0
- joint knee_L_Joint: limit lower=-1.7221163729428048 upper=2.7693139241394027 effort=140 velocity=12.57 -> lower=-1.6938420390604967 upper=2.7410395902570945 effort=140 velocity=12.57; origin xyz=-0.10276 -0.04115 -0.21389 rpy=0 0 0 -> xyz=0.10581 -0.04115 -0.2124 rpy=0 0 0
- joint knee_R_Joint: limit lower=-1.7221163729428048 upper=2.7693139241394027 effort=140 velocity=12.57 -> lower=-1.6938420390604967 upper=2.7410395902570945 effort=140 velocity=12.57; origin xyz=-0.10276 0.04115 -0.21389 rpy=0 0 0 -> xyz=0.10581 0.04115 -0.2124 rpy=0 0 0
- joint yaw_L_Joint: axis -0.43303 0 0.90138 -> -0.44589 0 0.89509; origin xyz=-0.0936 0.0 -0.08006 rpy=0 0 0 -> xyz=0.00577 0.0 -0.12304 rpy=0 0 0
- joint yaw_R_Joint: axis -0.43303 0 0.90138 -> -0.44589 0 0.89509; origin xyz=-0.004 0.0 -0.12311 rpy=0 0 0 -> xyz=0.09474 0.0 -0.07872 rpy=0 0 0

File: tron2/WF_TRON2/meshes/robot.urdf (robot description, URDF)
Before this commit: robot bipedal_robot, 12 links, 11 joints
Links:
- link abad_L_Link: geometry collision mesh filename=/home/wen/robot/urdf/transfer/output/WF_TRON2/urdf/meshes/a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; visual mesh filename=/home/wen/robot/urdf/transfer/output/WF_TRON2/urdf/meshes/a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
- link abad_R_Link: geometry collision mesh filename=/home/wen/robot/urdf/transfer/output/WF_TRON2/urdf/meshes/a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; visual mesh filename=/home/wen/robot/urdf/transfer/output/WF_TRON2/urdf/meshes/a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
- link base_Link: geometry collision mesh filename=/home/wen/robot/urdf/transfer/output/WF_TRON2/urdf/meshes/b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; visual mesh filename=/home/wen/robot/urdf/transfer/output/WF_TRON2/urdf/meshes/b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
- link hip_L_Link: geometry collision mesh filename=/home/wen/robot/urdf/transfer/output/WF_TRON2/urdf/meshes/h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; visual mesh filename=/home/wen/robot/urdf/transfer/output/WF_TRON2/urdf/meshes/h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
- link hip_R_Link: geometry collision mesh filename=/home/wen/robot/urdf/transfer/output/WF_TRON2/urdf/meshes/h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; visual mesh filename=/home/wen/robot/urdf/transfer/output/WF_TRON2/urdf/meshes/h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
- link knee_L_Link: geometry collision mesh filename=/home/wen/robot/urdf/transfer/output/WF_TRON2/urdf/meshes/k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; visual mesh filename=/home/wen/robot/urdf/transfer/output/WF_TRON2/urdf/meshes/k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
- link knee_R_Link: geometry collision mesh filename=/home/wen/robot/urdf/transfer/output/WF_TRON2/urdf/meshes/k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; visual mesh filename=/home/wen/robot/urdf/transfer/output/WF_TRON2/urdf/meshes/k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
- link wheel_L_Link: geometry collision mesh filename=/home/wen/robot/urdf/transfer/output/WF_TRON2/urdf/meshes/w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; visual mesh filename=/home/wen/robot/urdf/transfer/output/WF_TRON2/urdf/meshes/w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
- link wheel_R_Link: geometry collision mesh filename=/home/wen/robot/urdf/transfer/output/WF_TRON2/urdf/meshes/w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; visual mesh filename=/home/wen/robot/urdf/transfer/output/WF_TRON2/urdf/meshes/w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
- link yaw_L_Link: geometry collision mesh filename=/home/wen/robot/urdf/transfer/output/WF_TRON2/urdf/meshes/y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; visual mesh filename=/home/wen/robot/urdf/transfer/output/WF_TRON2/urdf/meshes/y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
- link yaw_R_Link: geometry collision mesh filename=/home/wen/robot/urdf/transfer/output/WF_TRON2/urdf/meshes/y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; visual mesh filename=/home/wen/robot/urdf/transfer/output/WF_TRON2/urdf/meshes/y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
Joints:
- joint hip_R_Joint: limit lower=-0.2605776573227534 upper=2.1131489961203007 effort=140 velocity=12.57 -> lower=-2.1131489961203007 upper=0.2605776573227534 effort=140 velocity=12.57
- joint yaw_L_Joint: axis -0.43303 0 0.90138 -> 0.43303 0 0.90138
- joint yaw_R_Joint: axis -0.43303 0 0.90138 -> 0.43303 0 0.90138

Commit message: Fix: 脚掌限位的bug

File: tron2/SF_TRON2/meshes/robot.urdf (robot description, URDF)
Before this commit: robot bipedal_robot, 12 links, 11 joints
Joints:
- joint foot_L_Joint: limit lower=1.2482594810263443 upper=-2.230356251123554 effort=40 velocity=31.83 -> lower=-1.2482594810263443 upper=2.230356251123554 effort=40 velocity=31.83
- joint foot_R_Joint: limit lower=1.2482594810263443 upper=-2.230356251123554 effort=40 velocity=31.83 -> lower=-1.2482594810263443 upper=2.230356251123554 effort=40 velocity=31.83

File: tron2/SF_TRON2/urdf/robot.urdf (robot description, URDF)
Before this commit: robot bipedal_robot, 12 links, 11 joints
Joints:
- joint foot_L_Joint: limit lower=1.2482594810263443 upper=-2.230356251123554 effort=40 velocity=31.83 -> lower=-1.2482594810263443 upper=2.230356251123554 effort=40 velocity=31.83
- joint foot_R_Joint: limit lower=1.2482594810263443 upper=-2.230356251123554 effort=40 velocity=31.83 -> lower=-1.2482594810263443 upper=2.230356251123554 effort=40 velocity=31.83
