Commit message: Fix: transmission不够数；轮足的hip_r_joint限位；轮足和双足的knee关节的限位

File: tron2/ARM_TRON2/meshes/robot.urdf (robot description, URDF)
Before this commit: robot bipedal_robot, 20 links, 19 joints
Links:
- link abad_L_Link: geometry collision mesh filename=package://daul_arm_robot/meshes/abad_L_Link.STL; visual mesh filename=package://daul_arm_robot/meshes/abad_L_Link.STL
- link abad_R_Link: geometry collision mesh filename=package://daul_arm_robot/meshes/abad_R_Link.STL; visual mesh filename=package://daul_arm_robot/meshes/abad_R_Link.STL
- link base_2_Link: geometry collision mesh filename=package://daul_arm_robot/meshes/base_2_Link.STL; visual mesh filename=package://daul_arm_robot/meshes/base_2_Link.STL
- link base_3_Link: geometry collision mesh filename=package://daul_arm_robot/meshes/base_3_Link.STL; visual mesh filename=package://daul_arm_robot/meshes/base_3_Link.STL
- link base_Link: geometry collision mesh filename=package://daul_arm_robot/meshes/base_Link.STL; visual mesh filename=package://daul_arm_robot/meshes/base_Link.STL
- link hip_L_Link: geometry collision mesh filename=package://daul_arm_robot/meshes/hip_L_Link.STL; visual mesh filename=package://daul_arm_robot/meshes/hip_L_Link.STL
- link hip_R_Link: geometry collision mesh filename=package://daul_arm_robot/meshes/hip_R_Link.STL; visual mesh filename=package://daul_arm_robot/meshes/hip_R_Link.STL
- link knee_L_Link: geometry collision mesh filename=package://daul_arm_robot/meshes/knee_L_Link.STL; visual mesh filename=package://daul_arm_robot/meshes/knee_L_Link.STL
- link knee_R_Link: geometry collision mesh filename=package://daul_arm_robot/meshes/knee_R_Link.STL; visual mesh filename=package://daul_arm_robot/meshes/knee_R_Link.STL
- link wrist_roll_L_Link: geometry collision mesh filename=package://daul_arm_robot/meshes/wrist_roll_L_Link.STL; visual mesh filename=package://daul_arm_robot/meshes/wrist_roll_L_Link.STL
- link wrist_roll_R_Link: geometry collision mesh filename=package://daul_arm_robot/meshes/wrist_roll_R_Link.STL; visual mesh filename=package://daul_arm_robot/meshes/wrist_roll_R_Link.STL
- link wrist_yaw1_L_Link: geometry collision mesh filename=package://daul_arm_robot/meshes/wrist_yaw1_L_Link.STL; visual mesh filename=package://daul_arm_robot/meshes/wrist_yaw1_L_Link.STL
- link wrist_yaw1_R_Link: geometry collision mesh filename=package://daul_arm_robot/meshes/wrist_yaw1_R_Link.STL; visual mesh filename=package://daul_arm_robot/meshes/wrist_yaw1_R_Link.STL
- link wrist_yaw2_L_Link: geometry collision mesh filename=package://daul_arm_robot/meshes/wrist_yaw2_L_Link.STL; visual mesh filename=package://daul_arm_robot/meshes/wrist_yaw2_L_Link.STL
- link wrist_yaw2_R_Link: geometry collision mesh filename=package://daul_arm_robot/meshes/wrist_yaw2_R_Link.STL; visual mesh filename=package://daul_arm_robot/meshes/wrist_yaw2_R_Link.STL
- link yaw_L_Link: geometry collision mesh filename=package://daul_arm_robot/meshes/yaw_L_Link.STL; visual mesh filename=package://daul_arm_robot/meshes/yaw_L_Link.STL
- link yaw_R_Link: geometry collision mesh filename=package://daul_arm_robot/meshes/yaw_R_Link.STL; visual mesh filename=package://daul_arm_robot/meshes/yaw_R_Link.STL

File: tron2/SF_TRON2/meshes/robot.urdf (robot description, URDF)
Before this commit: robot bipedal_robot, 12 links, 11 joints
Links:
- link abad_L_Link: geometry collision mesh filename=package://sf_robot/meshes/abad_L_Link.STL; visual mesh filename=package://sf_robot/meshes/abad_L_Link.STL
- link abad_R_Link: geometry collision mesh filename=package://sf_robot/meshes/abad_R_Link.STL; visual mesh filename=package://sf_robot/meshes/abad_R_Link.STL
- link base_Link: geometry collision mesh filename=package://sf_robot/meshes/base_Link.STL; visual mesh filename=package://sf_robot/meshes/base_Link.STL
- link foot_L_Link: geometry collision mesh filename=package://sf_robot/meshes/foot_L_Link.STL; visual mesh filename=package://sf_robot/meshes/foot_L_Link.STL
- link foot_R_Link: geometry collision mesh filename=package://sf_robot/meshes/foot_R_Link.STL; visual mesh filename=package://sf_robot/meshes/foot_R_Link.STL
- link hip_L_Link: geometry collision mesh filename=package://sf_robot/meshes/hip_L_Link.STL; visual mesh filename=package://sf_robot/meshes/hip_L_Link.STL
- link hip_R_Link: geometry collision mesh filename=package://sf_robot/meshes/hip_R_Link.STL; visual mesh filename=package://sf_robot/meshes/hip_R_Link.STL
- link knee_L_Link: geometry collision mesh filename=package://sf_robot/meshes/knee_L_Link.STL; visual mesh filename=package://sf_robot/meshes/knee_L_Link.STL
- link knee_R_Link: geometry collision mesh filename=package://sf_robot/meshes/knee_R_Link.STL; visual mesh filename=package://sf_robot/meshes/knee_R_Link.STL
- link yaw_L_Link: geometry collision mesh filename=package://sf_robot/meshes/yaw_L_Link.STL; visual mesh filename=package://sf_robot/meshes/yaw_L_Link.STL
- link yaw_R_Link: geometry collision mesh filename=package://sf_robot/meshes/yaw_R_Link.STL; visual mesh filename=package://sf_robot/meshes/yaw_R_Link.STL
Joints:
- joint knee_L_Joint: limit lower=-1.6938420390604967 upper=2.7410395902570945 effort=140 velocity=12.57 -> lower=-3.5421457169224917 upper=1.6938420390604967 effort=140 velocity=12.57
- joint knee_R_Joint: limit lower=-1.6938420390604967 upper=2.7410395902570945 effort=140 velocity=12.57 -> lower=-3.5421457169224917 upper=1.6938420390604967 effort=140 velocity=12.57

File: tron2/SF_TRON2/urdf/robot.urdf (robot description, URDF)
Before this commit: robot bipedal_robot, 12 links, 11 joints
Joints:
- joint knee_L_Joint: limit lower=-1.6938420390604967 upper=2.7410395902570945 effort=140 velocity=12.57 -> lower=-3.5421457169224917 upper=1.6938420390604967 effort=140 velocity=12.57
- joint knee_R_Joint: limit lower=-1.6938420390604967 upper=2.7410395902570945 effort=140 velocity=12.57 -> lower=-3.5421457169224917 upper=1.6938420390604967 effort=140 velocity=12.57

File: tron2/WF_TRON2/meshes/robot.urdf (robot description, URDF)
Before this commit: robot bipedal_robot, 12 links, 11 joints
Links:
- link abad_L_Link: geometry collision mesh filename=package://wf_robot/meshes/abad_L_Link.STL; visual mesh filename=package://wf_robot/meshes/abad_L_Link.STL
- link abad_R_Link: geometry collision mesh filename=package://wf_robot/meshes/abad_R_Link.STL; visual mesh filename=package://wf_robot/meshes/abad_R_Link.STL
- link base_Link: geometry collision mesh filename=package://wf_robot/meshes/base_Link.STL; visual mesh filename=package://wf_robot/meshes/base_Link.STL
- link hip_L_Link: geometry collision mesh filename=package://wf_robot/meshes/hip_L_Link.STL; visual mesh filename=package://wf_robot/meshes/hip_L_Link.STL
- link hip_R_Link: geometry collision mesh filename=package://wf_robot/meshes/hip_R_Link.STL; visual mesh filename=package://wf_robot/meshes/hip_R_Link.STL
- link knee_L_Link: geometry collision mesh filename=package://wf_robot/meshes/knee_L_Link.STL; visual mesh filename=package://wf_robot/meshes/knee_L_Link.STL
- link knee_R_Link: geometry collision mesh filename=package://wf_robot/meshes/knee_R_Link.STL; visual mesh filename=package://wf_robot/meshes/knee_R_Link.STL
- link wheel_L_Link: geometry collision mesh filename=package://wf_robot/meshes/wheel_L_Link.STL; visual mesh filename=package://wf_robot/meshes/wheel_L_Link.STL
- link wheel_R_Link: geometry collision mesh filename=package://wf_robot/meshes/wheel_R_Link.STL; visual mesh filename=package://wf_robot/meshes/wheel_R_Link.STL
- link yaw_L_Link: geometry collision mesh filename=package://wf_robot/meshes/yaw_L_Link.STL; visual mesh filename=package://wf_robot/meshes/yaw_L_Link.STL
- link yaw_R_Link: geometry collision mesh filename=package://wf_robot/meshes/yaw_R_Link.STL; visual mesh filename=package://wf_robot/meshes/yaw_R_Link.STL
Joints:
- joint knee_L_Joint: limit lower=-1.7221163729428048 upper=2.7693139241394027 effort=140 velocity=12.57 -> lower=-1.7221163729428048 upper=3.5138713830401835 effort=140 velocity=12.57
- joint knee_R_Joint: limit lower=-1.7221163729428048 upper=2.7693139241394027 effort=140 velocity=12.57 -> lower=-1.7221163729428048 upper=3.5138713830401835 effort=140 velocity=12.57

File: tron2/WF_TRON2/urdf/robot.urdf (robot description, URDF)
Before this commit: robot bipedal_robot, 12 links, 11 joints
Joints:
- joint hip_R_Joint: limit lower=-0.2605776573227534 upper=2.1131489961203007 effort=140 velocity=12.57 -> lower=-2.1131489961203007 upper=0.2605776573227534 effort=140 velocity=12.57
- joint knee_L_Joint: limit lower=-1.7221163729428048 upper=2.7693139241394027 effort=140 velocity=12.57 -> lower=-1.7221163729428048 upper=3.5138713830401835 effort=140 velocity=12.57
- joint knee_R_Joint: limit lower=-1.7221163729428048 upper=2.7693139241394027 effort=140 velocity=12.57 -> lower=-1.7221163729428048 upper=3.5138713830401835 effort=140 velocity=12.57
- joint yaw_L_Joint: axis -0.43303 0 0.90138 -> 0.43303 0 0.90138
- joint yaw_R_Joint: axis -0.43303 0 0.90138 -> 0.43303 0 0.90138
