Commit message: feat: 支持ros_package使用

File: tron2/ARM_TRON2/urdf/robot.urdf (robot description, URDF)
Before this commit: robot bipedal_robot, 20 links, 19 joints
Links:
- link abad_L_Link: geometry collision mesh filename=package://robot_description/tron2/ARM_TRON2/meshes/abad_L_L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; visual mesh filename=package://robot_description/tron2/ARM_TRON2/meshes/abad_L_L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
- link abad_R_Link: geometry collision mesh filename=package://robot_description/tron2/ARM_TRON2/meshes/abad_R_L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; visual mesh filename=package://robot_description/tron2/ARM_TRON2/meshes/abad_R_L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
- link base_2_Link: geometry collision mesh filename=package://robot_description/tron2/ARM_TRON2/meshes/base_2_L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; visual mesh filename=package://robot_description/tron2/ARM_TRON2/meshes/base_2_L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
- link base_3_Link: geometry collision mesh filename=package://robot_description/tron2/ARM_TRON2/meshes/base_3_L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; visual mesh filename=package://robot_description/tron2/ARM_TRON2/meshes/base_3_L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
- link base_Link: geometry collision mesh filename=package://robot_description/tron2/ARM_TRON2/meshes/base_Lin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; visual mesh filename=package://robot_description/tron2/ARM_TRON2/meshes/base_Lin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
- link hip_L_Link: geometry collision mesh filename=package://robot_description/tron2/ARM_TRON2/meshes/hip_L_Li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; visual mesh filename=package://robot_description/tron2/ARM_TRON2/meshes/hip_L_Li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
- link hip_R_Link: geometry collision mesh filename=package://robot_description/tron2/ARM_TRON2/meshes/hip_R_Li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; visual mesh filename=package://robot_description/tron2/ARM_TRON2/meshes/hip_R_Li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
- link knee_L_Link: geometry collision mesh filename=package://robot_description/tron2/ARM_TRON2/meshes/knee_L_L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; visual mesh filename=package://robot_description/tron2/ARM_TRON2/meshes/knee_L_L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
- link knee_R_Link: geometry collision mesh filename=package://robot_description/tron2/ARM_TRON2/meshes/knee_R_L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; visual mesh filename=package://robot_description/tron2/ARM_TRON2/meshes/knee_R_L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
- link wrist_roll_L_Link: geometry collision mesh filename=package://robot_description/tron2/ARM_TRON2/meshes/wrist_ro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; visual mesh filename=package://robot_description/tron2/ARM_TRON2/meshes/wrist_ro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
- link wrist_roll_R_Link: geometry collision mesh filename=package://robot_description/tron2/ARM_TRON2/meshes/wrist_ro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; visual mesh filename=package://robot_description/tron2/ARM_TRON2/meshes/wrist_ro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
- link wrist_yaw1_L_Link: geometry collision mesh filename=package://robot_description/tron2/ARM_TRON2/meshes/wrist_ya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; visual mesh filename=package://robot_description/tron2/ARM_TRON2/meshes/wrist_ya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
- link wrist_yaw1_R_Link: geometry collision mesh filename=package://robot_description/tron2/ARM_TRON2/meshes/wrist_ya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; visual mesh filename=package://robot_description/tron2/ARM_TRON2/meshes/wrist_ya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
- link wrist_yaw2_L_Link: geometry collision mesh filename=package://robot_description/tron2/ARM_TRON2/meshes/wrist_ya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; visual mesh filename=package://robot_description/tron2/ARM_TRON2/meshes/wrist_ya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
- link wrist_yaw2_R_Link: geometry collision mesh filename=package://robot_description/tron2/ARM_TRON2/meshes/wrist_ya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; visual mesh filename=package://robot_description/tron2/ARM_TRON2/meshes/wrist_ya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
- link yaw_L_Link: geometry collision mesh filename=package://robot_description/tron2/ARM_TRON2/meshes/yaw_L_Li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; visual mesh filename=package://robot_description/tron2/ARM_TRON2/meshes/yaw_L_Li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
- link yaw_R_Link: geometry collision mesh filename=package://robot_description/tron2/ARM_TRON2/meshes/yaw_R_Li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; visual mesh filename=package://robot_description/tron2/ARM_TRON2/meshes/yaw_R_Li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

File: tron2/SF_TRON2/urdf/robot.urdf (robot description, URDF)
Before this commit: robot bipedal_robot, 12 links, 11 joints
Links:
- link abad_L_Link: geometry collision mesh filename=package://robot_description/tron2/SF_TRON2/meshes/abad_L_Li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; visual mesh filename=package://robot_description/tron2/SF_TRON2/meshes/abad_L_Li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
- link abad_R_Link: geometry collision mesh filename=package://robot_description/tron2/SF_TRON2/meshes/abad_R_Li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; visual mesh filename=package://robot_description/tron2/SF_TRON2/meshes/abad_R_Li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
- link base_Link: geometry collision mesh filename=package://robot_description/tron2/SF_TRON2/meshes/base_Link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; visual mesh filename=package://robot_description/tron2/SF_TRON2/meshes/base_Link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
- link foot_L_Link: geometry collision mesh filename=package://robot_description/tron2/SF_TRON2/meshes/foot_L_Li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; visual mesh filename=package://robot_description/tron2/SF_TRON2/meshes/foot_L_Li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
- link foot_R_Link: geometry collision mesh filename=package://robot_description/tron2/SF_TRON2/meshes/foot_R_Li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; visual mesh filename=package://robot_description/tron2/SF_TRON2/meshes/foot_R_Li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
- link hip_L_Link: geometry collision mesh filename=package://robot_description/tron2/SF_TRON2/meshes/hip_L_Lin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; visual mesh filename=package://robot_description/tron2/SF_TRON2/meshes/hip_L_Lin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
- link hip_R_Link: geometry collision mesh filename=package://robot_description/tron2/SF_TRON2/meshes/hip_R_Lin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; visual mesh filename=package://robot_description/tron2/SF_TRON2/meshes/hip_R_Lin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
- link knee_L_Link: geometry collision mesh filename=package://robot_description/tron2/SF_TRON2/meshes/knee_L_Li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; visual mesh filename=package://robot_description/tron2/SF_TRON2/meshes/knee_L_Li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
- link knee_R_Link: geometry collision mesh filename=package://robot_description/tron2/SF_TRON2/meshes/knee_R_Li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; visual mesh filename=package://robot_description/tron2/SF_TRON2/meshes/knee_R_Li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
- link yaw_L_Link: geometry collision mesh filename=package://robot_description/tron2/SF_TRON2/meshes/yaw_L_Lin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; visual mesh filename=package://robot_description/tron2/SF_TRON2/meshes/yaw_L_Lin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
- link yaw_R_Link: geometry collision mesh filename=package://robot_description/tron2/SF_TRON2/meshes/yaw_R_Lin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; visual mesh filename=package://robot_description/tron2/SF_TRON2/meshes/yaw_R_Lin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

File: tron2/WF_TRON2/urdf/robot.urdf (robot description, URDF)
Before this commit: robot bipedal_robot, 12 links, 11 joints
Links:
- link abad_L_Link: geometry collision mesh filename=package://robot_description/tron2/WF_TRON2/meshes/abad_L_Li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; visual mesh filename=package://robot_description/tron2/WF_TRON2/meshes/abad_L_Li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
- link abad_R_Link: geometry collision mesh filename=package://robot_description/tron2/WF_TRON2/meshes/abad_R_Li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; visual mesh filename=package://robot_description/tron2/WF_TRON2/meshes/abad_R_Li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
- link base_Link: geometry collision mesh filename=package://robot_description/tron2/WF_TRON2/meshes/base_Link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; visual mesh filename=package://robot_description/tron2/WF_TRON2/meshes/base_Link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
- link hip_L_Link: geometry collision mesh filename=package://robot_description/tron2/WF_TRON2/meshes/hip_L_Lin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; visual mesh filename=package://robot_description/tron2/WF_TRON2/meshes/hip_L_Lin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
- link hip_R_Link: geometry collision mesh filename=package://robot_description/tron2/WF_TRON2/meshes/hip_R_Lin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; visual mesh filename=package://robot_description/tron2/WF_TRON2/meshes/hip_R_Lin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
- link knee_L_Link: geometry collision mesh filename=package://robot_description/tron2/WF_TRON2/meshes/knee_L_Li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; visual mesh filename=package://robot_description/tron2/WF_TRON2/meshes/knee_L_Li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
- link knee_R_Link: geometry collision mesh filename=package://robot_description/tron2/WF_TRON2/meshes/knee_R_Li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; visual mesh filename=package://robot_description/tron2/WF_TRON2/meshes/knee_R_Li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
- link wheel_L_Link: geometry collision mesh filename=package://robot_description/tron2/WF_TRON2/meshes/wheel_L_L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; visual mesh filename=package://robot_description/tron2/WF_TRON2/meshes/wheel_L_L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
- link wheel_R_Link: geometry collision mesh filename=package://robot_description/tron2/WF_TRON2/meshes/wheel_R_L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; visual mesh filename=package://robot_description/tron2/WF_TRON2/meshes/wheel_R_L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
- link yaw_L_Link: geometry collision mesh filename=package://robot_description/tron2/WF_TRON2/meshes/yaw_L_Lin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; visual mesh filename=package://robot_description/tron2/WF_TRON2/meshes/yaw_L_Lin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
- link yaw_R_Link: geometry collision mesh filename=package://robot_description/tron2/WF_TRON2/meshes/yaw_R_Lin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; visual mesh filename=package://robot_description/tron2/WF_TRON2/meshes/yaw_R_Lin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

Commit message: Fix: yaw_l_link mesh不对

File: tron2/ARM_TRON2/urdf/robot.urdf (robot description, URDF)
Before this commit: robot bipedal_robot, 20 links, 19 joints
Joints:
- joint yaw_L_Joint: limit lower=-1.4835298641951802 upper=2.705260340591211 effort=40 velocity=31.83 -> lower=-2.705260340591211 upper=1.4835298641951802 effort=40 velocity=31.83
