Commit message: fix: WF_TRON2 imu

File: tron2/WF_TRON2/xacro/gazebo.xacro (robot description, xacro)
@@ -24,8 +24,23 @@
     <!-- IMU sensor configuration -->
     <gazebo reference="limx_imu">
+        <gravity>true</gravity>
+        <sensor name="imu_sensor" type="imu">
+            <always_on>true</always_on>
+            <update_rate>1000</update_rate>
+            <visualize>true</visualize>
+            <topic>__default_topic__</topic>
+            <plugin filename="libgazebo_ros_imu_sensor.so" name="imu_plugin">
+                <topicName>trunk_imu</topicName>
+                <bodyName>limx_imu</bodyName>
+                <updateRateHZ>400.0</updateRateHZ>
+                <gaussianNoise>0.0</gaussianNoise>
+                <xyzOffset>0 0 0</xyzOffset>
+                <rpyOffset>0 0 0</rpyOffset>
+                <frameName>limx_imu</frameName>
+                <initial_orientation_as_reference>false</initial_orientation_as_reference>
+            </plugin>
+            <pose>0 0 0 0 0 0</pose>
+        </sensor>
         <material>Gazebo/Orange</material>
-    </gazebo>
-    <gazebo reference="limx_imu_joint">
-        <disableFixedJointLumping>true</disableFixedJointLumping>
     </gazebo>
     <!-- Base Link -->

File: tron2/WF_TRON2/xacro/robot.xacro (robot description, xacro)
@@ -59,4 +59,10 @@
             <material name="orange"/>
         </visual>
+        <collision>
+            <origin rpy="0 0 0" xyz="0 0 0"/>
+            <geometry>
+                <box size=".001 .001 .001"/>
+            </geometry>
+        </collision>
     </link>
     <!-- Additional IMU link for ros2_control compatibility -->
