Commit message: feat: fix stl import

File: tron2/SF_TRON2/xacro/const.xacro (robot description, xacro)
@@ -94,4 +94,5 @@
     <xacro:property name="foot_offset_x" value="-0.15601"/>
     <xacro:property name="foot_offset_y" value="0.07805"/>
+    <xacro:property name="foot_R_offset_y" value="-0.00425"/>
     <xacro:property name="foot_offset_z" value="-0.31331"/>
     <!-- Joint limits -->

File: tron2/SF_TRON2/xacro/leg.xacro (robot description, xacro)
@@ -20,5 +20,5 @@
                 <origin xyz="0 0 0" rpy="0 0 0"/>
                 <geometry>
-                    <mesh filename="package://robot_description/tron2/SF_TRON2/meshes/abad_${name}_Link.STL"/>
+                    <mesh filename="$(find robot_description)/tron2/SF_TRON2/meshes/abad_${name}_Link.STL"/>
                 </geometry>
                 <material name="grey"/>
@@ -27,5 +27,5 @@
                 <origin xyz="0 0 0" rpy="0 0 0"/>
                 <geometry>
-                    <mesh filename="package://robot_description/tron2/SF_TRON2/meshes/abad_${name}_Link.STL"/>
+                    <mesh filename="$(find robot_description)/tron2/SF_TRON2/meshes/abad_${name}_Link.STL"/>
                 </geometry>
             </collision>
@@ -53,5 +53,5 @@
                 <origin xyz="0 0 0" rpy="0 0 0"/>
                 <geometry>
-                    <mesh filename="package://robot_description/tron2/SF_TRON2/meshes/hip_${name}_Link.STL"/>
+                    <mesh filename="$(find robot_description)/tron2/SF_TRON2/meshes/hip_${name}_Link.STL"/>
                 </geometry>
                 <material name="grey"/>
@@ -60,5 +60,5 @@
                 <origin xyz="0 0 0" rpy="0 0 0"/>
                 <geometry>
-                    <mesh filename="package://robot_description/tron2/SF_TRON2/meshes/hip_${name}_Link.STL"/>
+                    <mesh filename="$(find robot_description)/tron2/SF_TRON2/meshes/hip_${name}_Link.STL"/>
                 </geometry>
             </collision>
@@ -86,5 +86,5 @@
                 <origin xyz="0 0 0" rpy="0 0 0"/>
                 <geometry>
-                    <mesh filename="package://robot_description/tron2/SF_TRON2/meshes/yaw_${name}_Link.STL"/>
+                    <mesh filename="$(find robot_description)/tron2/SF_TRON2/meshes/yaw_${name}_Link.STL"/>
                 </geometry>
                 <material name="grey"/>
@@ -93,5 +93,5 @@
                 <origin xyz="0 0 0" rpy="0 0 0"/>
                 <geometry>
-                    <mesh filename="package://robot_description/tron2/SF_TRON2/meshes/yaw_${name}_Link.STL"/>
+                    <mesh filename="$(find robot_description)/tron2/SF_TRON2/meshes/yaw_${name}_Link.STL"/>
                 </geometry>
             </collision>
@@ -114,5 +114,5 @@
                 <origin xyz="0 0 0" rpy="0 0 0"/>
                 <geometry>
-                    <mesh filename="package://robot_description/tron2/SF_TRON2/meshes/knee_${name}_Link.STL"/>
+                    <mesh filename="$(find robot_description)/tron2/SF_TRON2/meshes/knee_${name}_Link.STL"/>
                 </geometry>
                 <material name="grey"/>
@@ -121,10 +121,15 @@
                 <origin xyz="0 0 0" rpy="0 0 0"/>
                 <geometry>
-                    <mesh filename="package://robot_description/tron2/SF_TRON2/meshes/knee_${name}_Link.STL"/>
+                    <mesh filename="$(find robot_description)/tron2/SF_TRON2/meshes/knee_${name}_Link.STL"/>
                 </geometry>
             </collision>
         </link>
         <joint name="foot_${name}_Joint" type="revolute">
-            <origin xyz="${foot_offset_x} ${foot_offset_y*mirror} ${foot_offset_z}" rpy="0 0 0"/>
+            <xacro:if value="${name == 'L'}">
+                <origin xyz="${foot_offset_x} ${foot_offset_y} ${foot_offset_z}" rpy="0 0 0"/>
+            </xacro:if>
+            <xacro:if value="${name == 'R'}">
+                <origin xyz="${foot_offset_x} ${foot_R_offset_y} ${foot_offset_z}" rpy="0 0 0"/>
+            </xacro:if>
             <parent link="knee_${name}_Link"/>
             <child link="foot_${name}_Link"/>
@@ -142,5 +147,5 @@
                 <origin xyz="0 0 0" rpy="0 0 0"/>
                 <geometry>
-                    <mesh filename="package://robot_description/tron2/SF_TRON2/meshes/foot_${name}_Link.STL"/>
+                    <mesh filename="$(find robot_description)/tron2/SF_TRON2/meshes/foot_${name}_Link.STL"/>
                 </geometry>
                 <material name="grey"/>
@@ -149,5 +154,5 @@
                 <origin xyz="0 0 0" rpy="0 0 0"/>
                 <geometry>
-                    <mesh filename="package://robot_description/tron2/SF_TRON2/meshes/foot_${name}_Link.STL"/>
+                    <mesh filename="$(find robot_description)/tron2/SF_TRON2/meshes/foot_${name}_Link.STL"/>
                 </geometry>
             </collision>

File: tron2/SF_TRON2/xacro/robot.xacro (robot description, xacro)
@@ -21,5 +21,5 @@
             <origin xyz="0 0 0" rpy="0 0 0"/>
             <geometry>
-                <mesh filename="package://robot_description/tron2/SF_TRON2/meshes/base_Link.STL"/>
+                <mesh filename="$(find robot_description)/tron2/SF_TRON2/meshes/base_Link.STL"/>
             </geometry>
             <material name="grey"/>
@@ -28,5 +28,5 @@
             <origin xyz="0 0 0" rpy="0 0 0"/>
             <geometry>
-                <mesh filename="package://robot_description/tron2/SF_TRON2/meshes/base_Link.STL"/>
+                <mesh filename="$(find robot_description)/tron2/SF_TRON2/meshes/base_Link.STL"/>
             </geometry>
         </collision>
@@ -70,10 +70,10 @@
             </geometry>
         </visual>
-        <collision>
+        <!-- <collision>
             <origin rpy="0 0 0" xyz="0 0 0"/>
             <geometry>
                 <box size=".001 .001 .001"/>
             </geometry>
-        </collision>
+        </collision> -->
     </link>
     <!-- Left and Right Legs -->

Commit message: fix: 右腿关节数据错误

File: tron2/SF_TRON2/xacro/const.xacro (robot description, xacro)
@@ -79,12 +79,21 @@
     <xacro:property name="abad_offset_y" value="0.10649"/>
     <xacro:property name="abad_offset_z" value="0.0586"/>
+    <xacro:property name="abad_R_offset_x" value="-0.00049"/>
+    <xacro:property name="abad_R_offset_y" value="-0.10631"/>
+    <xacro:property name="abad_R_offset_z" value="0.0586"/>
     <!-- Hip joint position -->
     <xacro:property name="hip_offset_x" value="0.04449"/>
     <xacro:property name="hip_offset_y" value="0.062"/>
     <xacro:property name="hip_offset_z" value="0.02216"/>
+    <xacro:property name="hip_R_offset_x" value="-0.04449"/>
+    <xacro:property name="hip_R_offset_y" value="-0.062"/>
+    <xacro:property name="hip_R_offset_z" value="-0.02216"/>
     <!-- Yaw joint position -->
     <xacro:property name="yaw_offset_x" value="0.00577"/>
     <xacro:property name="yaw_offset_y" value="0.0"/>
     <xacro:property name="yaw_offset_z" value="-0.12304"/>
+    <xacro:property name="yaw_R_offset_x" value="0.09474"/>
+    <xacro:property name="yaw_R_offset_y" value="0.0"/>
+    <xacro:property name="yaw_R_offset_z" value="-0.07872"/>
     <!-- Knee joint position -->
     <xacro:property name="knee_offset_x" value="0.10581"/>

File: tron2/SF_TRON2/xacro/leg.xacro (robot description, xacro)
@@ -4,5 +4,10 @@
     <xacro:macro name="leg" params="name mirror *origin">
         <joint name="abad_${name}_Joint" type="revolute">
-            <origin xyz="${abad_offset_x} ${abad_offset_y*mirror} ${abad_offset_z}" rpy="0 0 0"/>
+            <xacro:if value="${name == 'L'}">
+                <origin xyz="${abad_offset_x} ${abad_offset_y} ${abad_offset_z}" rpy="0 0 0"/>
+            </xacro:if>
+            <xacro:if value="${name == 'R'}">
+                <origin xyz="${abad_R_offset_x} ${abad_R_offset_y} ${abad_R_offset_z}" rpy="0 0 0"/>
+            </xacro:if>
             <parent link="base_Link"/>
             <child link="abad_${name}_Link"/>
@@ -32,5 +37,10 @@
         </link>
         <joint name="hip_${name}_Joint" type="revolute">
-            <origin xyz="${hip_offset_x} ${hip_offset_y*mirror} ${hip_offset_z}" rpy="0 0 0"/>
+            <xacro:if value="${name == 'L'}">
+                <origin xyz="${hip_offset_x} ${hip_offset_y} ${hip_offset_z}" rpy="0 0 0"/>
+            </xacro:if>
+            <xacro:if value="${name == 'R'}">
+                <origin xyz="${hip_R_offset_x} ${hip_R_offset_y} ${hip_R_offset_z}" rpy="0 0 0"/>
+            </xacro:if>
             <parent link="abad_${name}_Link"/>
             <child link="hip_${name}_Link"/>
@@ -65,5 +75,10 @@
         </link>
         <joint name="yaw_${name}_Joint" type="revolute">
-            <origin xyz="${yaw_offset_x} ${yaw_offset_y*mirror} ${yaw_offset_z}" rpy="0 0 0"/>
+            <xacro:if value="${name == 'L'}">
+                <origin xyz="${yaw_offset_x} ${yaw_offset_y} ${yaw_offset_z}" rpy="0 0 0"/>
+            </xacro:if>
+            <xacro:if value="${name == 'R'}">
+                <origin xyz="${yaw_R_offset_x} ${yaw_R_offset_y} ${yaw_R_offset_z}" rpy="0 0 0"/>
+            </xacro:if>
             <parent link="hip_${name}_Link"/>
             <child link="yaw_${name}_Link"/>
