Commit message: fix: invalid imu sensor for ros2

File: tron2/SF_TRON2/xacro/robot.xacro (robot description, xacro)
@@ -51,4 +51,29 @@
         </visual>
     </link>
+    <!-- Additional IMU link for ros2_control compatibility -->
+    <joint name="imu_Joint" type="fixed">
+        <parent link="base_Link"/>
+        <child link="imu_Link"/>
+        <origin rpy="0 0 0" xyz="0 0 0"/>
+    </joint>
+    <link name="imu_Link">
+        <inertial>
+            <mass value="0.001"/>
+            <origin rpy="0 0 0" xyz="0 0 0"/>
+            <inertia ixx="0.0001" ixy="0" ixz="0" iyy="0.0001" iyz="0" izz="0.0001"/>
+        </inertial>
+        <visual>
+            <origin rpy="0 0 0" xyz="0 0 0"/>
+            <geometry>
+                <box size="0.015 0.015 0.004"/>
+            </geometry>
+        </visual>
+        <collision>
+            <origin rpy="0 0 0" xyz="0 0 0"/>
+            <geometry>
+                <box size=".001 .001 .001"/>
+            </geometry>
+        </collision>
+    </link>
     <!-- Left and Right Legs -->
     <xacro:leg name="L" mirror="1">
@@ -76,5 +101,5 @@
             <xacro:leg_ros2_control_interface leg_name="R"/>
             <sensor name="imu_sensor">
-                <frame_id name="limx_imu"/>
+                <frame_id name="imu_Link"/>
                 <state_interface name="orientation.x"/>
                 <state_interface name="orientation.y"/>

File: tron2/WF_TRON2/xacro/robot.xacro (robot description, xacro)
@@ -60,4 +60,29 @@
         </visual>
     </link>
+    <!-- Additional IMU link for ros2_control compatibility -->
+    <joint name="imu_Joint" type="fixed">
+        <parent link="base_Link"/>
+        <child link="imu_Link"/>
+        <origin rpy="0 0 0" xyz="0 0 0"/>
+    </joint>
+    <link name="imu_Link">
+        <inertial>
+            <mass value="0.001"/>
+            <origin rpy="0 0 0" xyz="0 0 0"/>
+            <inertia ixx="0.0001" ixy="0" ixz="0" iyy="0.0001" iyz="0" izz="0.0001"/>
+        </inertial>
+        <visual>
+            <origin rpy="0 0 0" xyz="0 0 0"/>
+            <geometry>
+                <box size="0.015 0.015 0.004"/>
+            </geometry>
+        </visual>
+        <collision>
+            <origin rpy="0 0 0" xyz="0 0 0"/>
+            <geometry>
+                <box size=".001 .001 .001"/>
+            </geometry>
+        </collision>
+    </link>
     <!-- Left and Right Legs -->
     <xacro:leg name="L" mirror="1">
@@ -76,5 +101,5 @@
             <xacro:leg_ros2_control_interface leg_name="R"/>
             <sensor name="imu_sensor">
-                <frame_id name="limx_imu"/>
+                <frame_id name="imu_Link"/>
                 <state_interface name="orientation.x"/>
                 <state_interface name="orientation.y"/>

Commit message: feat: cancel fix

File: tron2/SF_TRON2/xacro/robot.xacro (robot description, xacro)
@@ -10,13 +10,4 @@
     <xacro:include filename="$(find robot_description)/tron2/SF_TRON2/xacro/gazebo.xacro"/>
     <xacro:include filename="$(find robot_description)/tron2/SF_TRON2/xacro/ros2_control_interface.xacro"/>
-    <!-- 支撑关节 - 将机器人悬挂在0.8米高度 -->
-    <!-- 世界固定点 -->
-    <link name="world"/>
-    <!-- 悬挂关节 -->
-    <joint name="world_to_base" type="fixed">
-        <origin xyz="0 0 1.5" rpy="0 0 0"/>
-        <parent link="world"/>
-        <child link="base_Link"/>
-    </joint>
     <!-- Base Link -->
     <link name="base_Link">
