Commit message: Feat: 轮足和脚掌yaw限位左右不对称，内旋>外旋

File: tron2/SF_TRON2/urdf/robot.urdf (robot description, URDF)
Before this commit: robot bipedal_robot, 12 links, 11 joints
Joints:
- joint yaw_L_Joint: limit lower=-1.4835298641951802 upper=2.705260340591211 effort=40 velocity=31.83 -> lower=-2.705260340591211 upper=1.4835298641951802 effort=40 velocity=31.83

File: tron2/WF_TRON2/urdf/robot.urdf (robot description, URDF)
Before this commit: robot bipedal_robot, 12 links, 11 joints
Joints:
- joint yaw_L_Joint: limit lower=-1.4835298641951802 upper=2.705260340591211 effort=40 velocity=31.83 -> lower=-2.705260340591211 upper=1.4835298641951802 effort=40 velocity=31.83

Commit message: Feat: 完成V3双足和双轮足的URDF和USD文件生成

File: tron2/SF_TRON2/urdf/robot.urdf (robot description, URDF)
Before this commit: robot bipedal_robot, 12 links, 11 joints
Links:
- link abad_L_Link: mass 2.42561 -> 2.15; geometry collision mesh filename=package://robot_description/tron2/SF_TRON3/meshes/abad_L_Li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; visual mesh filename=package://robot_description/tron2/SF_TRON3/meshes/abad_L_Li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
- link abad_R_Link: mass 2.42561 -> 2.15; geometry collision mesh filename=package://robot_description/tron2/SF_TRON3/meshes/abad_R_Li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; visual mesh filename=package://robot_description/tron2/SF_TRON3/meshes/abad_R_Li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
- link base_Link: mass 8.04083 -> 10.92; geometry collision mesh filename=package://robot_description/tron2/SF_TRON3/meshes/base_Link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; visual mesh filename=package://robot_description/tron2/SF_TRON3/meshes/base_Link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
- link foot_L_Link: mass 0.94793 -> 0.9; geometry collision mesh filename=package://robot_description/tron2/SF_TRON3/meshes/foot_L_Li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; visual mesh filename=package://robot_description/tron2/SF_TRON3/meshes/foot_L_Li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
- link foot_R_Link: mass 0.94793 -> 0.9; geometry collision mesh filename=package://robot_description/tron2/SF_TRON3/meshes/foot_R_Li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; visual mesh filename=package://robot_description/tron2/SF_TRON3/meshes/foot_R_Li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
- link hip_L_Link: mass 0.50271 -> 0.65; geometry collision mesh filename=package://robot_description/tron2/SF_TRON3/meshes/hip_L_Lin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; visual mesh filename=package://robot_description/tron2/SF_TRON3/meshes/hip_L_Lin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
- link hip_R_Link: mass 0.50271 -> 0.65; geometry collision mesh filename=package://robot_description/tron2/SF_TRON3/meshes/hip_R_Lin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; visual mesh filename=package://robot_description/tron2/SF_TRON3/meshes/hip_R_Lin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
- link knee_L_Link: mass 1.84166 -> 3.92; geometry collision mesh filename=package://robot_description/tron2/SF_TRON3/meshes/knee_L_Li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; visual mesh filename=package://robot_description/tron2/SF_TRON3/meshes/knee_L_Li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
- link knee_R_Link: mass 1.84166 -> 3.92; geometry collision mesh filename=package://robot_description/tron2/SF_TRON3/meshes/knee_R_Li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; visual mesh filename=package://robot_description/tron2/SF_TRON3/meshes/knee_R_Li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
- link yaw_L_Link: mass 3.43624 -> 1.58; geometry collision mesh filename=package://robot_description/tron2/SF_TRON3/meshes/yaw_L_Lin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; visual mesh filename=package://robot_description/tron2/SF_TRON3/meshes/yaw_L_Lin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
- link yaw_R_Link: mass 3.43624 -> 1.58; geometry collision mesh filename=package://robot_description/tron2/SF_TRON3/meshes/yaw_R_Lin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; visual mesh filename=package://robot_description/tron2/SF_TRON3/meshes/yaw_R_Lin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
Joints:
- joint abad_L_Joint: limit lower=-2.679429467661695 upper=3.062703771399649 effort=140 velocity=12.57 -> lower=-3.141592653589793 upper=2.600540585471551 effort=130 velocity=12.57; origin xyz=0.00049 0.10649 0.0586 rpy=0 0 0 -> xyz=-0.00045 0.09949 0.06046 rpy=0 0 0
- joint abad_R_Joint: limit lower=-2.679429467661695 upper=3.062703771399649 effort=140 velocity=12.57 -> lower=-3.141592653589793 upper=2.600540585471551 effort=130 velocity=12.57; origin xyz=-0.00049 -0.10631 0.0586 rpy=0 0 0 -> xyz=-0.00045 -0.09949 0.06046 rpy=0 0 0
- joint foot_L_Joint: limit lower=-1.2482594810263443 upper=2.230356251123554 effort=40 velocity=31.83 -> lower=-1.6929693744344996 upper=1.6929693744344996 effort=40 velocity=31.83; origin xyz=-0.15601 0.07805 -0.31331 rpy=0 0 0 -> xyz=0.0 0.0065 -0.35 rpy=0 0 0
- joint foot_R_Joint: limit lower=-1.2482594810263443 upper=2.230356251123554 effort=40 velocity=31.83 -> lower=-1.6929693744344996 upper=1.6929693744344996 effort=40 velocity=31.83; origin xyz=-0.15601 -0.00425 -0.31331 rpy=0 0 0 -> xyz=0 -0.0065 -0.35 rpy=0 0 0
- joint hip_L_Joint: axis 0.89509 0 0.44589 -> 1 0 0; limit lower=-0.2605776573227534 upper=2.1131489961203007 effort=140 velocity=12.57 -> lower=-0.2617993877991494 upper=2.792526803190927 effort=130 velocity=12.57; origin xyz=0.04449 0.062 0.02216 rpy=0 0 0 -> xyz=0.04164 0.0681 0.0 rpy=0 0 0
- joint hip_R_Joint: axis 0.89509 0 0.44589 -> 1 0 0; limit lower=-2.1131489961203007 upper=0.2605776573227534 effort=140 velocity=12.57 -> lower=-2.792526803190927 upper=0.2617993877991494 effort=130 velocity=12.57; origin xyz=-0.04449 -0.062 -0.02216 rpy=0 0 0 -> xyz=0.04164 -0.0681 0 rpy=0 0 0
- joint knee_L_Joint: limit lower=-3.5421457169224917 upper=1.6938420390604967 effort=140 velocity=12.57 -> lower=-2.5656340004316647 upper=2.5656340004316647 effort=130 velocity=12.57; origin xyz=0.10581 -0.04115 -0.2124 rpy=0 0 0 -> xyz=0.0 0.0305 -0.2358 rpy=0 0 0
- joint knee_R_Joint: limit lower=-3.5421457169224917 upper=1.6938420390604967 effort=140 velocity=12.57 -> lower=-2.5656340004316647 upper=2.5656340004316647 effort=130 velocity=12.57; origin xyz=0.10581 0.04115 -0.2124 rpy=0 0 0 -> xyz=0 -0.0305 -0.2358 rpy=0 0 0
- joint yaw_L_Joint: axis -0.44589 0 0.89509 -> 0 0 1; limit lower=-2.705260340591211 upper=1.4835298641951802 effort=40 velocity=31.83 -> lower=-2.705260340591211 upper=1.4835298641951802 effort=60 velocity=14.66; origin xyz=0.00577 0.0 -0.12304 rpy=0 0 0 -> xyz=-0.0416 0.0 -0.1142 rpy=0 0 0
- joint yaw_R_Joint: axis -0.44589 0 0.89509 -> 0 0 1; limit lower=-1.4835298641951802 upper=2.705260340591211 effort=40 velocity=31.83 -> lower=-1.4835298641951802 upper=2.705260340591211 effort=60 velocity=14.66; origin xyz=0.09474 0.0 -0.07872 rpy=0 0 0 -> xyz=-0.0416 0 -0.1142 rpy=0 0 0

File: tron2/WF_TRON2/urdf/robot.urdf (robot description, URDF)
Before this commit: robot bipedal_robot, 12 links, 11 joints
Links:
- link abad_L_Link: mass 2.42561 -> 2.15; geometry collision mesh filename=package://robot_description/tron2/meshes_wf_v3/meshes/abad_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; visual mesh filename=package://robot_description/tron2/meshes_wf_v3/meshes/abad_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
- link abad_R_Link: mass 2.42561 -> 2.15; geometry collision mesh filename=package://robot_description/tron2/meshes_wf_v3/meshes/abad_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; visual mesh filename=package://robot_description/tron2/meshes_wf_v3/meshes/abad_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
- link base_Link: mass 8.04083 -> 10.92; geometry collision mesh filename=package://robot_description/tron2/meshes_wf_v3/meshes/base_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; visual mesh filename=package://robot_description/tron2/meshes_wf_v3/meshes/base_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
- link hip_L_Link: mass 0.50271 -> 0.65; geometry collision mesh filename=package://robot_description/tron2/meshes_wf_v3/meshes/hip_L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; visual mesh filename=package://robot_description/tron2/meshes_wf_v3/meshes/hip_L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
- link hip_R_Link: mass 0.50271 -> 0.65; geometry collision mesh filename=package://robot_description/tron2/meshes_wf_v3/meshes/hip_R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; visual mesh filename=package://robot_description/tron2/meshes_wf_v3/meshes/hip_R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
- link knee_L_Link: mass 1.9798 -> 4.00; geometry collision mesh filename=package://robot_description/tron2/meshes_wf_v3/meshes/knee_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; visual mesh filename=package://robot_description/tron2/meshes_wf_v3/meshes/knee_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
- link knee_R_Link: mass 1.9798 -> 4.00; geometry collision mesh filename=package://robot_description/tron2/meshes_wf_v3/meshes/knee_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; visual mesh filename=package://robot_description/tron2/meshes_wf_v3/meshes/knee_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
- link wheel_L_Link: geometry collision cylinder length=0.045 radius=0.1; visual mesh filename=package://robot_description/tron2/meshes_wf_v3/meshes/wheel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
- link wheel_R_Link: geometry collision cylinder length=0.045 radius=0.1; visual mesh filename=package://robot_description/tron2/meshes_wf_v3/meshes/wheel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
- link yaw_L_Link: mass 3.43624 -> 1.58; geometry collision mesh filename=package://robot_description/tron2/meshes_wf_v3/meshes/yaw_L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; visual mesh filename=package://robot_description/tron2/meshes_wf_v3/meshes/yaw_L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
- link yaw_R_Link: mass 3.43624 -> 1.58; geometry collision mesh filename=package://robot_description/tron2/meshes_wf_v3/meshes/yaw_R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; visual mesh filename=package://robot_description/tron2/meshes_wf_v3/meshes/yaw_R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
Joints:
- joint abad_L_Joint: limit lower=-3.5894441396515377 upper=2.1526890994098062 effort=140 velocity=12.57 -> lower=-3.141592653589793 upper=2.600540585471551 effort=130 velocity=13.0; origin xyz=-0.00049 0.10649 0.0586 rpy=0 0 0 -> xyz=-0.00045 0.09949 0.06046 rpy=0 0 0
- joint abad_R_Joint: limit lower=-3.5894441396515377 upper=2.1526890994098062 effort=140 velocity=12.57 -> lower=-3.141592653589793 upper=2.600540585471551 effort=130 velocity=13.0; origin xyz=-0.00049 -0.10631 0.0586 rpy=0 0 0 -> xyz=-0.00045 -0.09949 0.06046 rpy=0 0 0
- joint hip_L_Joint: axis 0.90138 0 -0.43303 -> 1 0 0; limit lower=-0.2605776573227534 upper=2.1131489961203007 effort=140 velocity=12.57 -> lower=-0.2617993877991494 upper=2.79111111 effort=130 velocity=13.0; origin xyz=0.0448 0.062 -0.02152 rpy=0 0 0 -> xyz=0.04164 0.0681 0.0 rpy=0 0 0
- joint hip_R_Joint: axis 0.90138 0 -0.43303 -> 1 0 0; limit lower=-2.1131489961203007 upper=0.2605776573227534 effort=140 velocity=12.57 -> lower=-2.79111111 upper=0.2617993877991494 effort=130 velocity=13.0; origin xyz=-0.0448 -0.062 0.02152 rpy=0 0 0 -> xyz=0.04164 -0.0681 0 rpy=0 0 0
- joint knee_L_Joint: limit lower=-1.7221163729428048 upper=3.5138713830401835 effort=140 velocity=12.57 -> lower=-2.5656340004316647 upper=2.5656340004316647 effort=130 velocity=13.0; origin xyz=-0.10276 -0.04115 -0.21389 rpy=0 0 0 -> xyz=0.0 0.0305 -0.2358 rpy=0 0 0
- joint knee_R_Joint: limit lower=-1.7221163729428048 upper=3.5138713830401835 effort=140 velocity=12.57 -> lower=-2.5656340004316647 upper=2.5656340004316647 effort=130 velocity=13.0; origin xyz=-0.10276 0.04115 -0.21389 rpy=0 0 0 -> xyz=0 -0.0305 -0.2358 rpy=0 0 0
- joint wheel_L_Joint: limit lower=-1745329.2519943293 upper=1745329.2519943293 effort=22 velocity=41.89 -> lower=-1745329.2519943293 upper=1745329.2519943293 effort=20 velocity=76.25; origin xyz=0.15161 0.09165 -0.31546 rpy=0 0 0 -> xyz=0.0 0.015 -0.35 rpy=0 0 0
- joint wheel_R_Joint: limit lower=-1745329.2519943293 upper=1745329.2519943293 effort=22 velocity=41.89 -> lower=-1745329.2519943293 upper=1745329.2519943293 effort=20 velocity=76.25; origin xyz=0.15161 -0.09165 -0.31546 rpy=0 0 0 -> xyz=0 -0.015 -0.35 rpy=0 0 0
- joint yaw_L_Joint: axis 0.43303 0 0.90138 -> 0 0 1; limit lower=-2.705260340591211 upper=1.4835298641951802 effort=40 velocity=31.83 -> lower=-2.705260340591211 upper=1.4835298641951802 effort=60 velocity=14.66; origin xyz=-0.0936 0.0 -0.08006 rpy=0 0 0 -> xyz=-0.0416 0.0 -0.1142 rpy=0 0 0
- joint yaw_R_Joint: axis 0.43303 0 0.90138 -> 0 0 1; limit lower=-1.4835298641951802 upper=2.705260340591211 effort=40 velocity=31.83 -> lower=-1.4835298641951802 upper=2.705260340591211 effort=60 velocity=14.66; origin xyz=-0.004 0.0 -0.12311 rpy=0 0 0 -> xyz=-0.0416 0 -0.1142 rpy=0 0 0

Commit message: fix: mesh path

File: tron2/SF_TRON2/urdf/robot.urdf (robot description, URDF)
Before this commit: robot bipedal_robot, 12 links, 11 joints
Links:
- link abad_L_Link: geometry collision mesh filename=package://robot_description/tron2/SF_TRON2/urdf/meshes/abad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; visual mesh filename=package://robot_description/tron2/SF_TRON2/urdf/meshes/abad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
- link abad_R_Link: geometry collision mesh filename=package://robot_description/tron2/SF_TRON2/urdf/meshes/abad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; visual mesh filename=package://robot_description/tron2/SF_TRON2/urdf/meshes/abad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
- link base_Link: geometry collision mesh filename=package://robot_description/tron2/SF_TRON2/urdf/meshes/base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; visual mesh filename=package://robot_description/tron2/SF_TRON2/urdf/meshes/base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
- link foot_L_Link: geometry collision mesh filename=package://robot_description/tron2/SF_TRON2/urdf/meshes/foot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; visual mesh filename=package://robot_description/tron2/SF_TRON2/urdf/meshes/foot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
- link foot_R_Link: geometry collision mesh filename=package://robot_description/tron2/SF_TRON2/urdf/meshes/foot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; visual mesh filename=package://robot_description/tron2/SF_TRON2/urdf/meshes/foot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
- link hip_L_Link: geometry collision mesh filename=package://robot_description/tron2/SF_TRON2/urdf/meshes/hip_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; visual mesh filename=package://robot_description/tron2/SF_TRON2/urdf/meshes/hip_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
- link hip_R_Link: geometry collision mesh filename=package://robot_description/tron2/SF_TRON2/urdf/meshes/hip_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; visual mesh filename=package://robot_description/tron2/SF_TRON2/urdf/meshes/hip_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
- link knee_L_Link: geometry collision mesh filename=package://robot_description/tron2/SF_TRON2/urdf/meshes/knee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; visual mesh filename=package://robot_description/tron2/SF_TRON2/urdf/meshes/knee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
- link knee_R_Link: geometry collision mesh filename=package://robot_description/tron2/SF_TRON2/urdf/meshes/knee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; visual mesh filename=package://robot_description/tron2/SF_TRON2/urdf/meshes/knee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
- link yaw_L_Link: geometry collision mesh filename=package://robot_description/tron2/SF_TRON2/urdf/meshes/yaw_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; visual mesh filename=package://robot_description/tron2/SF_TRON2/urdf/meshes/yaw_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
- link yaw_R_Link: geometry collision mesh filename=package://robot_description/tron2/SF_TRON2/urdf/meshes/yaw_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; visual mesh filename=package://robot_description/tron2/SF_TRON2/urdf/meshes/yaw_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

File: tron2/WF_TRON2/urdf/robot.urdf (robot description, URDF)
Before this commit: robot bipedal_robot, 12 links, 11 joints
Links:
- link abad_L_Link: geometry collision mesh filename=package://robot_description/tron2/WF_TRON2/urdf/meshes/abad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; visual mesh filename=package://robot_description/tron2/WF_TRON2/urdf/meshes/abad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
- link abad_R_Link: geometry collision mesh filename=package://robot_description/tron2/WF_TRON2/urdf/meshes/abad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; visual mesh filename=package://robot_description/tron2/WF_TRON2/urdf/meshes/abad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
- link base_Link: geometry collision mesh filename=package://robot_description/tron2/WF_TRON2/urdf/meshes/base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; visual mesh filename=package://robot_description/tron2/WF_TRON2/urdf/meshes/base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
- link hip_L_Link: geometry collision mesh filename=package://robot_description/tron2/WF_TRON2/urdf/meshes/hip_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; visual mesh filename=package://robot_description/tron2/WF_TRON2/urdf/meshes/hip_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
- link hip_R_Link: geometry collision mesh filename=package://robot_description/tron2/WF_TRON2/urdf/meshes/hip_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; visual mesh filename=package://robot_description/tron2/WF_TRON2/urdf/meshes/hip_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
- link knee_L_Link: geometry collision mesh filename=package://robot_description/tron2/WF_TRON2/urdf/meshes/knee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; visual mesh filename=package://robot_description/tron2/WF_TRON2/urdf/meshes/knee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
- link knee_R_Link: geometry collision mesh filename=package://robot_description/tron2/WF_TRON2/urdf/meshes/knee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; visual mesh filename=package://robot_description/tron2/WF_TRON2/urdf/meshes/knee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
- link wheel_L_Link: geometry collision cylinder length=0.045 radius=0.1; visual mesh filename=package://robot_description/tron2/WF_TRON2/urdf/meshes/whee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
- link wheel_R_Link: geometry collision cylinder length=0.045 radius=0.1; visual mesh filename=package://robot_description/tron2/WF_TRON2/urdf/meshes/whee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
- link yaw_L_Link: geometry collision mesh filename=package://robot_description/tron2/WF_TRON2/urdf/meshes/yaw_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; visual mesh filename=package://robot_description/tron2/WF_TRON2/urdf/meshes/yaw_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
- link yaw_R_Link: geometry collision mesh filename=package://robot_description/tron2/WF_TRON2/urdf/meshes/yaw_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; visual mesh filename=package://robot_description/tron2/WF_TRON2/urdf/meshes/yaw_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
