Commit message: feat: v4.0 urdf and xacro

File: tron2/SF_TRON2/urdf/robot.urdf (robot description, URDF)
Before this commit: robot bipedal_robot, 12 links, 11 joints
Links:
- link abad_L_Link: mass 2.15 -> 2.16; geometry collision mesh filename=../meshes/abad_L_Link.STL; visual mesh filename=../meshes/abad_L_Link.STL
- link abad_R_Link: mass 2.15 -> 2.16; geometry collision mesh filename=../meshes/abad_R_Link.STL; visual mesh filename=../meshes/abad_R_Link.STL
- link base_Link: mass 10.92 -> 10.94; geometry collision mesh filename=../meshes/base_Link.STL; visual mesh filename=../meshes/base_Link.STL
- link foot_L_Link: mass 0.9 -> 0.90; geometry collision mesh filename=../meshes/foot_L_Link.STL; visual mesh filename=../meshes/foot_L_Link.STL
- link foot_R_Link: mass 0.9 -> 0.90; geometry collision mesh filename=../meshes/foot_R_Link.STL; visual mesh filename=../meshes/foot_R_Link.STL
- link hip_L_Link: mass 0.65 -> 0.62; geometry collision mesh filename=../meshes/hip_L_Link.STL; visual mesh filename=../meshes/hip_L_Link.STL
- link hip_R_Link: mass 0.65 -> 0.62; geometry collision mesh filename=../meshes/hip_R_Link.STL; visual mesh filename=../meshes/hip_R_Link.STL
- link knee_L_Link: mass 3.92 -> 3.39; geometry collision mesh filename=../meshes/knee_L_Link.STL; visual mesh filename=../meshes/knee_L_Link.STL
- link knee_R_Link: mass 3.92 -> 3.39; geometry collision mesh filename=../meshes/knee_R_Link.STL; visual mesh filename=../meshes/knee_R_Link.STL
- link yaw_L_Link: mass 1.58 -> 1.82; geometry collision mesh filename=../meshes/yaw_L_Link.STL; visual mesh filename=../meshes/yaw_L_Link.STL
- link yaw_R_Link: mass 1.58 -> 1.82; geometry collision mesh filename=../meshes/yaw_R_Link.STL; visual mesh filename=../meshes/yaw_R_Link.STL
Joints:
- joint foot_L_Joint: origin xyz=0.0 0.0065 -0.35 rpy=0 0 0 -> xyz=0.0 0.07148 -0.35 rpy=0 0 0
- joint foot_R_Joint: origin xyz=0 -0.0065 -0.35 rpy=0 0 0 -> xyz=0.0 -0.07148 -0.35 rpy=0 0 0
- joint hip_L_Joint: limit lower=-0.2617993877991494 upper=2.792526803190927 effort=130 velocity=12.57 -> lower=-0.2617993877991494 upper=2.9670597283903604 effort=130 velocity=12.57; origin xyz=0.04164 0.0681 0.0 rpy=0 0 0 -> xyz=-0.0416 0.0681 0.0 rpy=0 0 0
- joint hip_R_Joint: limit lower=-2.792526803190927 upper=0.2617993877991494 effort=130 velocity=12.57 -> lower=-2.9670597283903604 upper=0.2617993877991494 effort=130 velocity=12.57; origin xyz=0.04164 -0.0681 0 rpy=0 0 0 -> xyz=-0.0416 -0.0681 0.0 rpy=0 0 0
- joint knee_L_Joint: limit lower=-2.5656340004316647 upper=2.5656340004316647 effort=130 velocity=12.57 -> lower=-0.5235987755982988 upper=2.6179938779914944 effort=60 velocity=14.66; origin xyz=0.0 0.0305 -0.2358 rpy=0 0 0 -> xyz=0.0 -0.03432 -0.2366 rpy=0 0 0
- joint knee_R_Joint: limit lower=-2.5656340004316647 upper=2.5656340004316647 effort=130 velocity=12.57 -> lower=-0.5235987755982988 upper=2.6179938779914944 effort=60 velocity=14.66; origin xyz=0 -0.0305 -0.2358 rpy=0 0 0 -> xyz=0.0 0.03432 -0.2366 rpy=0 0 0
- joint yaw_L_Joint: limit lower=-2.705260340591211 upper=1.4835298641951802 effort=60 velocity=14.66 -> lower=-0.5235987755982988 upper=4.625122517784973 effort=60 velocity=14.66; origin xyz=-0.0416 0.0 -0.1142 rpy=0 0 0 -> xyz=0.0416 0.0 -0.1142 rpy=0 0 0
- joint yaw_R_Joint: limit lower=-1.4835298641951802 upper=2.705260340591211 effort=60 velocity=14.66 -> lower=-4.625122517784973 upper=0.5235987755982988 effort=60 velocity=14.66; origin xyz=-0.0416 0 -0.1142 rpy=0 0 0 -> xyz=0.0416 -0.0 -0.1142 rpy=0 0 0

File: tron2/SF_TRON2/xacro/const.xacro (robot description, xacro)
@@ -9,66 +9,66 @@
     <xacro:property name="imu_mass" value="0.01"/>
     <!-- Base Link parameters -->
-    <xacro:property name="base_mass" value="10.92"/>
-    <xacro:property name="base_com_x" value="0.0067"/>
+    <xacro:property name="base_mass" value="10.94"/>
+    <xacro:property name="base_com_x" value="0.00656"/>
     <xacro:property name="base_com_y" value="0.001"/>
-    <xacro:property name="base_com_z" value="0.11976"/>
-    <xacro:property name="base_ixx" value="0.10676912"/>
-    <xacro:property name="base_ixy" value="0.00070697"/>
-    <xacro:property name="base_ixz" value="0.00165993"/>
-    <xacro:property name="base_iyy" value="0.11048777"/>
-    <xacro:property name="base_iyz" value="0.00109598"/>
-    <xacro:property name="base_izz" value="0.07980999"/>
+    <xacro:property name="base_com_z" value="0.12055"/>
+    <xacro:property name="base_ixx" value="0.10814592"/>
+    <xacro:property name="base_ixy" value="0.00070438"/>
+    <xacro:property name="base_ixz" value="0.00180329"/>
+    <xacro:property name="base_iyy" value="0.1118876"/>
+    <xacro:property name="base_iyz" value="0.00110226"/>
+    <xacro:property name="base_izz" value="0.07968023"/>
     <!-- Abad Link parameters (left) -->
-    <xacro:property name="abad_mass" value="2.15"/>
-    <xacro:property name="abad_com_x" value="0.00382"/>
-    <xacro:property name="abad_com_y" value="0.0658"/>
-    <xacro:property name="abad_com_z" value="0.00024"/>
-    <xacro:property name="abad_ixx" value="0.00455282"/>
-    <xacro:property name="abad_ixy" value="-0.00003068"/>
-    <xacro:property name="abad_ixz" value="-0.00000099"/>
-    <xacro:property name="abad_iyy" value="0.00368823"/>
-    <xacro:property name="abad_iyz" value="-0.00000618"/>
-    <xacro:property name="abad_izz" value="0.00372679"/>
+    <xacro:property name="abad_mass" value="2.16"/>
+    <xacro:property name="abad_com_x" value="-0.00585"/>
+    <xacro:property name="abad_com_y" value="0.06636"/>
+    <xacro:property name="abad_com_z" value="-0.0004"/>
+    <xacro:property name="abad_ixx" value="0.00461832"/>
+    <xacro:property name="abad_ixy" value="0.00000691"/>
+    <xacro:property name="abad_ixz" value="0.00000837"/>
+    <xacro:property name="abad_iyy" value="0.0036266"/>
+    <xacro:property name="abad_iyz" value="0.00000188"/>
+    <xacro:property name="abad_izz" value="0.00371921"/>
     <!-- Hip Link parameters (left) -->
-    <xacro:property name="hip_mass" value="0.65"/>
-    <xacro:property name="hip_com_x" value="-0.04048"/>
-    <xacro:property name="hip_com_y" value="0.00011"/>
-    <xacro:property name="hip_com_z" value="-0.05235"/>
-    <xacro:property name="hip_ixx" value="0.00174455"/>
-    <xacro:property name="hip_ixy" value="-0.00000634"/>
-    <xacro:property name="hip_ixz" value="0.00003090"/>
-    <xacro:property name="hip_iyy" value="0.00252619"/>
-    <xacro:property name="hip_iyz" value="0.00000728"/>
-    <xacro:property name="hip_izz" value="0.00172929"/>
+    <xacro:property name="hip_mass" value="0.62"/>
+    <xacro:property name="hip_com_x" value="0.03454"/>
+    <xacro:property name="hip_com_y" value="0.00074"/>
+    <xacro:property name="hip_com_z" value="-0.05537"/>
+    <xacro:property name="hip_ixx" value="0.00161988"/>
+    <xacro:property name="hip_ixy" value="-0.00000677"/>
+    <xacro:property name="hip_ixz" value="0.00005921"/>
+    <xacro:property name="hip_iyy" value="0.00229105"/>
+    <xacro:property name="hip_iyz" value="-0.00000259"/>
+    <xacro:property name="hip_izz" value="0.00163377"/>
     <!-- Yaw Link parameters (left) -->
-    <xacro:property name="yaw_mass" value="1.58"/>
-    <xacro:property name="yaw_com_x" value="0.00006"/>
-    <xacro:property name="yaw_com_y" value="0.01051"/>
-    <xacro:property name="yaw_com_z" value="-0.06665"/>
-    <xacro:property name="yaw_ixx" value="0.01072218"/>
-    <xacro:property name="yaw_ixy" value="0.00000079"/>
-    <xacro:property name="yaw_ixz" value="-0.00000667"/>
-    <xacro:property name="yaw_iyy" value="0.01045244"/>
-    <xacro:property name="yaw_iyz" value="0.00197942"/>
-    <xacro:property name="yaw_izz" value="0.00217735"/>
+    <xacro:property name="yaw_mass" value="1.82"/>
+    <xacro:property name="yaw_com_x" value="0.00294"/>
+    <xacro:property name="yaw_com_y" value="-0.00009"/>
+    <xacro:property name="yaw_com_z" value="-0.08263"/>
+    <xacro:property name="yaw_ixx" value="0.01407104"/>
+    <xacro:property name="yaw_ixy" value="-0.00000181"/>
+    <xacro:property name="yaw_ixz" value="0.00037981"/>
+    <xacro:property name="yaw_iyy" value="0.0137125"/>
+    <xacro:property name="yaw_iyz" value="-0.00003338"/>
+    <xacro:property name="yaw_izz" value="0.00304924"/>
     <!-- Knee Link parameters (left) -->
-    <xacro:property name="knee_mass" value="3.92"/>
-    <xacro:property name="knee_com_x" value="-0.00009"/>
-    <xacro:property name="knee_com_y" value="-0.03303"/>
-    <xacro:property name="knee_com_z" value="-0.12123"/>
-    <xacro:property name="knee_ixx" value="0.09179022"/>
-    <xacro:property name="knee_ixy" value="0.00000828"/>
-    <xacro:property name="knee_ixz" value="0.00011012"/>
-    <xacro:property name="knee_iyy" value="0.09202670"/>
-    <xacro:property name="knee_iyz" value="0.00154530"/>
-    <xacro:property name="knee_izz" value="0.00521320"/>
+    <xacro:property name="knee_mass" value="3.39"/>
+    <xacro:property name="knee_com_x" value="0.00024"/>
+    <xacro:property name="knee_com_y" value="0.03439"/>
+    <xacro:property name="knee_com_z" value="-0.14948"/>
+    <xacro:property name="knee_ixx" value="0.07632531"/>
+    <xacro:property name="knee_ixy" value="0.00001890"/>
+    <xacro:property name="knee_ixz" value="0.00006976"/>
+    <xacro:property name="knee_iyy" value="0.07685607"/>
+    <xacro:property name="knee_iyz" value="0.00075049"/>
+    <xacro:property name="knee_izz" value="0.00384986"/>
     <!-- Foot Link parameters -->
-    <xacro:property name="foot_mass" value="0.9"/>
+    <xacro:property name="foot_mass" value="0.90"/>
     <xacro:property name="foot_com_x" value="0.01691"/>
     <xacro:property name="foot_com_y" value="-0.03589"/>
     <xacro:property name="foot_com_z" value="-0.04454"/>
-    <xacro:property name="foot_ixx" value="0.00125165"/>
+    <xacro:property name="foot_ixx" value="0.00125164"/>
     <xacro:property name="foot_ixy" value="0.00001843"/>
-    <xacro:property name="foot_ixz" value="0.00014741"/>
+    <xacro:property name="foot_ixz" value="0.00014738"/>
     <xacro:property name="foot_iyy" value="0.00296403"/>
     <xacro:property name="foot_iyz" value="-0.00008693"/>
@@ -83,25 +83,25 @@
     <xacro:property name="abad_R_offset_z" value="0.06046"/>
     <!-- Hip joint position -->
-    <xacro:property name="hip_offset_x" value="0.04164"/>
+    <xacro:property name="hip_offset_x" value="-0.0416"/>
     <xacro:property name="hip_offset_y" value="0.0681"/>
     <xacro:property name="hip_offset_z" value="0.0"/>
-    <xacro:property name="hip_R_offset_x" value="0.04164"/>
+    <xacro:property name="hip_R_offset_x" value="-0.0416"/>
     <xacro:property name="hip_R_offset_y" value="-0.0681"/>
     <xacro:property name="hip_R_offset_z" value="0.0"/>
     <!-- Yaw joint position -->
-    <xacro:property name="yaw_offset_x" value="-0.0416"/>
+    <xacro:property name="yaw_offset_x" value="0.0416"/>
     <xacro:property name="yaw_offset_y" value="0.0"/>
     <xacro:property name="yaw_offset_z" value="-0.1142"/>
-    <xacro:property name="yaw_R_offset_x" value="-0.0416"/>
-    <xacro:property name="yaw_R_offset_y" value="0.0"/>
+    <xacro:property name="yaw_R_offset_x" value="0.0416"/>
+    <xacro:property name="yaw_R_offset_y" value="-0.0"/>
     <xacro:property name="yaw_R_offset_z" value="-0.1142"/>
     <!-- Knee joint position -->
     <xacro:property name="knee_offset_x" value="0.0"/>
-    <xacro:property name="knee_offset_y" value="0.0305"/>
-    <xacro:property name="knee_offset_z" value="-0.2358"/>
+    <xacro:property name="knee_offset_y" value="-0.03432"/>
+    <xacro:property name="knee_offset_z" value="-0.2366"/>
     <!-- Foot joint position -->
     <xacro:property name="foot_offset_x" value="0.0"/>
-    <xacro:property name="foot_offset_y" value="0.0065"/>
-    <xacro:property name="foot_R_offset_y" value="-0.0065"/>
+    <xacro:property name="foot_offset_y" value="0.07148"/>
+    <xacro:property name="foot_R_offset_y" value="-0.07148"/>
     <xacro:property name="foot_offset_z" value="-0.35"/>
     <!-- Joint limits -->
@@ -113,21 +113,21 @@
     <!-- Hip joint limits -->
     <xacro:property name="hip_L_lower" value="-0.2617993877991494"/>
-    <xacro:property name="hip_L_upper" value="2.792526803190927"/>
-    <xacro:property name="hip_R_lower" value="-2.792526803190927"/>
+    <xacro:property name="hip_L_upper" value="2.9670597283903604"/>
+    <xacro:property name="hip_R_lower" value="-2.9670597283903604"/>
     <xacro:property name="hip_R_upper" value="0.2617993877991494"/>
     <xacro:property name="hip_effort" value="130"/>
     <xacro:property name="hip_velocity" value="12.57"/>
     <!-- Yaw joint limits -->
-    <xacro:property name="yaw_L_lower" value="-2.705260340591211"/>
-    <xacro:property name="yaw_L_upper" value="1.4835298641951802"/>
-    <xacro:property name="yaw_R_lower" value="-1.4835298641951802"/>
-    <xacro:property name="yaw_R_upper" value="2.705260340591211"/>
+    <xacro:property name="yaw_L_lower" value="-0.5235987755982988"/>
+    <xacro:property name="yaw_L_upper" value="4.625122517784973"/>
+    <xacro:property name="yaw_R_lower" value="-4.625122517784973"/>
+    <xacro:property name="yaw_R_upper" value="0.5235987755982988"/>
     <xacro:property name="yaw_effort" value="60"/>
     <xacro:property name="yaw_velocity" value="14.66"/>
     <!-- Knee joint limits -->
-    <xacro:property name="knee_lower" value="-2.5656340004316647"/>
-    <xacro:property name="knee_upper" value="2.5656340004316647"/>
-    <xacro:property name="knee_effort" value="130"/>
-    <xacro:property name="knee_velocity" value="12.57"/>
+    <xacro:property name="knee_lower" value="-0.5235987755982988"/>
+    <xacro:property name="knee_upper" value="2.6179938779914944"/>
+    <xacro:property name="knee_effort" value="60"/>
+    <xacro:property name="knee_velocity" value="14.66"/>
     <!-- Foot joint limits -->
     <xacro:property name="foot_lower" value="-1.6929693744344996"/>

File: tron2/SF_TRON2/xacro/leg.xacro (robot description, xacro)
@@ -25,5 +25,5 @@
                 <origin xyz="0 0 0" rpy="0 0 0"/>
                 <geometry>
-                    <mesh filename="$(find robot_description)/tron2/SF_TRON2/urdf/meshes/abad_${name}_Link.STL"/>
+                    <mesh filename="$(find robot_description)/tron2/SF_TRON2/meshes/abad_${name}_Link.STL"/>
                 </geometry>
                 <material name="grey"/>
@@ -32,5 +32,5 @@
                 <origin xyz="0 0 0" rpy="0 0 0"/>
                 <geometry>
-                    <mesh filename="$(find robot_description)/tron2/SF_TRON2/urdf/meshes/abad_${name}_Link.STL"/>
+                    <mesh filename="$(find robot_description)/tron2/SF_TRON2/meshes/abad_${name}_Link.STL"/>
                 </geometry>
             </collision>
@@ -63,5 +63,5 @@
                 <origin xyz="0 0 0" rpy="0 0 0"/>
                 <geometry>
-                    <mesh filename="$(find robot_description)/tron2/SF_TRON2/urdf/meshes/hip_${name}_Link.STL"/>
+                    <mesh filename="$(find robot_description)/tron2/SF_TRON2/meshes/hip_${name}_Link.STL"/>
                 </geometry>
                 <material name="grey"/>
@@ -70,5 +70,5 @@
                 <origin xyz="0 0 0" rpy="0 0 0"/>
                 <geometry>
-                    <mesh filename="$(find robot_description)/tron2/SF_TRON2/urdf/meshes/hip_${name}_Link.STL"/>
+                    <mesh filename="$(find robot_description)/tron2/SF_TRON2/meshes/hip_${name}_Link.STL"/>
                 </geometry>
             </collision>
@@ -101,5 +101,5 @@
                 <origin xyz="0 0 0" rpy="0 0 0"/>
                 <geometry>
-                    <mesh filename="$(find robot_description)/tron2/SF_TRON2/urdf/meshes/yaw_${name}_Link.STL"/>
+                    <mesh filename="$(find robot_description)/tron2/SF_TRON2/meshes/yaw_${name}_Link.STL"/>
                 </geometry>
                 <material name="grey"/>
@@ -108,5 +108,5 @@
                 <origin xyz="0 0 0" rpy="0 0 0"/>
                 <geometry>
-                    <mesh filename="$(find robot_description)/tron2/SF_TRON2/urdf/meshes/yaw_${name}_Link.STL"/>
+                    <mesh filename="$(find robot_description)/tron2/SF_TRON2/meshes/yaw_${name}_Link.STL"/>
                 </geometry>
             </collision>
@@ -129,5 +129,5 @@
                 <origin xyz="0 0 0" rpy="0 0 0"/>
                 <geometry>
-                    <mesh filename="$(find robot_description)/tron2/SF_TRON2/urdf/meshes/knee_${name}_Link.STL"/>
+                    <mesh filename="$(find robot_description)/tron2/SF_TRON2/meshes/knee_${name}_Link.STL"/>
                 </geometry>
                 <material name="grey"/>
@@ -136,5 +136,5 @@
                 <origin xyz="0 0 0" rpy="0 0 0"/>
                 <geometry>
-                    <mesh filename="$(find robot_description)/tron2/SF_TRON2/urdf/meshes/knee_${name}_Link.STL"/>
+                    <mesh filename="$(find robot_description)/tron2/SF_TRON2/meshes/knee_${name}_Link.STL"/>
                 </geometry>
             </collision>
@@ -162,5 +162,5 @@
                 <origin xyz="0 0 0" rpy="0 0 0"/>
                 <geometry>
-                    <mesh filename="$(find robot_description)/tron2/SF_TRON2/urdf/meshes/foot_${name}_Link.STL"/>
+                    <mesh filename="$(find robot_description)/tron2/SF_TRON2/meshes/foot_${name}_Link.STL"/>
                 </geometry>
                 <material name="grey"/>
@@ -169,5 +169,5 @@
                 <origin xyz="0 0 0" rpy="0 0 0"/>
                 <geometry>
-                    <mesh filename="$(find robot_description)/tron2/SF_TRON2/urdf/meshes/foot_${name}_Link.STL"/>
+                    <mesh filename="$(find robot_description)/tron2/SF_TRON2/meshes/foot_${name}_Link.STL"/>
                 </geometry>
             </collision>

File: tron2/SF_TRON2/xacro/robot.xacro (robot description, xacro)
@@ -21,5 +21,5 @@
             <origin xyz="0 0 0" rpy="0 0 0"/>
             <geometry>
-                <mesh filename="$(find robot_description)/tron2/SF_TRON2/urdf/meshes/base_Link.STL"/>
+                <mesh filename="$(find robot_description)/tron2/SF_TRON2/meshes/base_Link.STL"/>
             </geometry>
             <material name="grey"/>
@@ -28,5 +28,5 @@
             <origin xyz="0 0 0" rpy="0 0 0"/>
             <geometry>
-                <mesh filename="$(find robot_description)/tron2/SF_TRON2/urdf/meshes/base_Link.STL"/>
+                <mesh filename="$(find robot_description)/tron2/SF_TRON2/meshes/base_Link.STL"/>
             </geometry>
         </collision>
