Commit message: Feat: modify joint effort for sim2real, and proximal_roll limit joint pos

File: tron2/DA_TRON2A/meshes/robot.urdf (robot description, URDF)
Before this commit: robot bipedal_robot, 20 links, 19 joints
Joints:
- joint proximal_pitch_L_Joint: limit lower=-3.141592653589793 upper=2.600540585471551 effort=200 velocity=18.3 -> lower=-3.141592653589793 upper=2.600540585471551 effort=150 velocity=18.3
- joint proximal_pitch_R_Joint: limit lower=-3.141592653589793 upper=2.600540585471551 effort=200 velocity=18.3 -> lower=-3.141592653589793 upper=2.600540585471551 effort=150 velocity=18.3
- joint proximal_roll_L_Joint: limit lower=-0.2617993877991494 upper=3.2288591161895095 effort=200 velocity=18.3 -> lower=-0.2617993877991494 upper=3.19395248 effort=150 velocity=18.3
- joint proximal_roll_R_Joint: limit lower=-3.2288591161895095 upper=0.2617993877991494 effort=200 velocity=18.3 -> lower=-3.19395248 upper=0.2617993877991494 effort=150 velocity=18.3
- joint proximal_yaw_L_Joint: limit lower=-3.6651914291880923 upper=1.4835298641951802 effort=70 velocity=22.52 -> lower=-3.6651914291880923 upper=1.4835298641951802 effort=60 velocity=22.52
- joint proximal_yaw_R_Joint: limit lower=-1.4835298641951802 upper=3.6651914291880923 effort=70 velocity=22.52 -> lower=-1.4835298641951802 upper=3.6651914291880923 effort=60 velocity=22.52

File: tron2/DA_TRON2A/urdf/robot.urdf (robot description, URDF)
Before this commit: robot bipedal_robot, 20 links, 19 joints
Joints:
- joint proximal_pitch_L_Joint: limit lower=-3.141592653589793 upper=2.600540585471551 effort=200 velocity=18.3 -> lower=-3.141592653589793 upper=2.600540585471551 effort=150 velocity=18.3
- joint proximal_pitch_R_Joint: limit lower=-3.141592653589793 upper=2.600540585471551 effort=200 velocity=18.3 -> lower=-3.141592653589793 upper=2.600540585471551 effort=150 velocity=18.3
- joint proximal_roll_L_Joint: limit lower=-0.2617993877991494 upper=3.2288591161895095 effort=200 velocity=18.3 -> lower=-0.2617993877991494 upper=3.19395248 effort=150 velocity=18.3
- joint proximal_roll_R_Joint: limit lower=-3.2288591161895095 upper=0.2617993877991494 effort=200 velocity=18.3 -> lower=-3.19395248 upper=0.2617993877991494 effort=150 velocity=18.3
- joint proximal_yaw_L_Joint: limit lower=-3.6651914291880923 upper=1.4835298641951802 effort=70 velocity=22.52 -> lower=-3.6651914291880923 upper=1.4835298641951802 effort=60 velocity=22.52
- joint proximal_yaw_R_Joint: limit lower=-1.4835298641951802 upper=3.6651914291880923 effort=70 velocity=22.52 -> lower=-1.4835298641951802 upper=3.6651914291880923 effort=60 velocity=22.52

File: tron2/SFYG_TRON2A/urdf/robot.urdf (robot description, URDF)
Before this commit: robot bipedal_robot, 27 links, 26 joints
Joints:
- joint ankle_pitch_L_Joint: limit lower=-1.6231562043547265 upper=1.6231562043547265 effort=70.0 velocity=22.52 -> lower=-1.6231562043547265 upper=1.6231562043547265 effort=60 velocity=22.52
- joint ankle_pitch_R_Joint: limit lower=-1.6231562043547265 upper=1.6231562043547265 effort=70.0 velocity=22.52 -> lower=-1.6231562043547265 upper=1.6231562043547265 effort=60 velocity=22.52
- joint knee_L_Joint: limit lower=-0.2617993877991494 upper=2.6179938779914944 effort=200.0 velocity=18.3 -> lower=-0.2617993877991494 upper=2.6179938779914944 effort=150 velocity=18.3
- joint knee_R_Joint: limit lower=-0.2617993877991494 upper=2.6179938779914944 effort=200.0 velocity=18.3 -> lower=-0.2617993877991494 upper=2.6179938779914944 effort=150 velocity=18.3
- joint proximal_pitch_L_Joint: limit lower=-3.141592653589793 upper=2.600540585471551 effort=200.0 velocity=18.3 -> lower=-3.141592653589793 upper=2.600540585471551 effort=150 velocity=18.3
- joint proximal_pitch_R_Joint: limit lower=-3.141592653589793 upper=2.600540585471551 effort=200.0 velocity=18.3 -> lower=-3.141592653589793 upper=2.600540585471551 effort=150 velocity=18.3
- joint proximal_roll_L_Joint: limit lower=-0.2617993877991494 upper=3.2288591161895095 effort=200.0 velocity=18.3 -> lower=-0.2617993877991494 upper=3.19395248 effort=150 velocity=18.3
- joint proximal_roll_R_Joint: limit lower=-3.2288591161895095 upper=0.2617993877991494 effort=200.0 velocity=18.3 -> lower=-3.19395248 upper=0.2617993877991494 effort=150 velocity=18.3
- joint proximal_yaw_L_Joint: limit lower=-0.5235987755982988 upper=4.625122517784973 effort=70.0 velocity=22.52 -> lower=-0.5235987755982988 upper=4.625122517784973 effort=60 velocity=22.52
- joint proximal_yaw_R_Joint: limit lower=-4.625122517784973 upper=0.5235987755982988 effort=70.0 velocity=22.52 -> lower=-4.625122517784973 upper=0.5235987755982988 effort=60 velocity=22.52

File: tron2/SFYG_TRON2A/urdf/robot_rl.urdf (robot description, URDF)
Before this commit: robot bipedal_robot, 25 links, 24 joints
Joints:
- joint ankle_pitch_L_Joint: limit lower=-1.6231562043547265 upper=1.6231562043547265 effort=70.0 velocity=22.52 -> lower=-1.6231562043547265 upper=1.6231562043547265 effort=60 velocity=22.52
- joint ankle_pitch_R_Joint: limit lower=-1.6231562043547265 upper=1.6231562043547265 effort=70.0 velocity=22.52 -> lower=-1.6231562043547265 upper=1.6231562043547265 effort=60 velocity=22.52
- joint knee_L_Joint: limit lower=-0.2617993877991494 upper=2.6179938779914944 effort=200.0 velocity=18.3 -> lower=-0.2617993877991494 upper=2.6179938779914944 effort=150 velocity=18.3
- joint knee_R_Joint: limit lower=-0.2617993877991494 upper=2.6179938779914944 effort=200.0 velocity=18.3 -> lower=-0.2617993877991494 upper=2.6179938779914944 effort=150 velocity=18.3
- joint proximal_pitch_L_Joint: limit lower=-3.141592653589793 upper=2.600540585471551 effort=200.0 velocity=18.3 -> lower=-3.141592653589793 upper=2.600540585471551 effort=150 velocity=18.3
- joint proximal_pitch_R_Joint: limit lower=-3.141592653589793 upper=2.600540585471551 effort=200.0 velocity=18.3 -> lower=-3.141592653589793 upper=2.600540585471551 effort=150 velocity=18.3
- joint proximal_roll_L_Joint: limit lower=-0.2617993877991494 upper=3.2288591161895095 effort=200.0 velocity=18.3 -> lower=-0.2617993877991494 upper=3.19395248 effort=150 velocity=18.3
- joint proximal_roll_R_Joint: limit lower=-3.2288591161895095 upper=0.2617993877991494 effort=200.0 velocity=18.3 -> lower=-3.19395248 upper=0.2617993877991494 effort=150 velocity=18.3
- joint proximal_yaw_L_Joint: limit lower=-0.5235987755982988 upper=4.625122517784973 effort=70.0 velocity=22.52 -> lower=-0.5235987755982988 upper=4.625122517784973 effort=60 velocity=22.52
- joint proximal_yaw_R_Joint: limit lower=-4.625122517784973 upper=0.5235987755982988 effort=70.0 velocity=22.52 -> lower=-4.625122517784973 upper=0.5235987755982988 effort=60 velocity=22.52

File: tron2/SFYG_TRON2A/xacro/robot.urdf.xacro (robot description, xacro)
@@ -298,5 +298,5 @@
     <child link="proximal_pitch_L_Link" />
     <axis xyz="0 0.99619 -0.087155" />
-    <limit lower="-3.141592653589793" upper="2.600540585471551" effort="200" velocity="18.3" />
+    <limit lower="-3.141592653589793" upper="2.600540585471551" effort="150" velocity="18.3" />
   </joint>
   <joint name="proximal_roll_L_Joint" type="revolute">
@@ -305,5 +305,5 @@
     <child link="proximal_roll_L_Link" />
     <axis xyz="1 0 0" />
-    <limit lower="-0.2617993877991494" upper="3.2288591161895095" effort="200" velocity="18.3" />
+    <limit lower="-0.2617993877991494" upper="3.19395248" effort="150" velocity="18.3" />
   </joint>
   <joint name="proximal_yaw_L_Joint" type="revolute">
@@ -312,5 +312,5 @@
     <child link="proximal_yaw_L_Link" />
     <axis xyz="0 0 1" />
-    <limit lower="-0.5235987755982988" upper="4.625122517784973" effort="70" velocity="22.52" />
+    <limit lower="-0.5235987755982988" upper="4.625122517784973" effort="60" velocity="22.52" />
   </joint>
   <joint name="knee_L_Joint" type="revolute">
@@ -319,5 +319,5 @@
     <child link="knee_L_Link" />
     <axis xyz="0 1 0" />
-    <limit lower="-0.2617993877991494" upper="2.6179938779914944" effort="200" velocity="18.3" />
+    <limit lower="-0.2617993877991494" upper="2.6179938779914944" effort="150" velocity="18.3" />
   </joint>
   <joint name="ankle_pitch_L_Joint" type="revolute">
@@ -326,5 +326,5 @@
     <child link="ankle_pitch_L_Link" />
     <axis xyz="0 1 0" />
-    <limit lower="-1.6231562043547263" upper="1.6231562043547263" effort="70" velocity="22.52" />
+    <limit lower="-1.6231562043547263" upper="1.6231562043547263" effort="60" velocity="22.52" />
   </joint>
   <joint name="proximal_pitch_R_Joint" type="revolute">
@@ -333,5 +333,5 @@
     <child link="proximal_pitch_R_Link" />
     <axis xyz="0 0.99619 0.087155" />
-    <limit lower="-3.141592653589793" upper="2.600540585471551" effort="200" velocity="18.3" />
+    <limit lower="-3.141592653589793" upper="2.600540585471551" effort="150" velocity="18.3" />
   </joint>
   <joint name="proximal_roll_R_Joint" type="revolute">
@@ -340,5 +340,5 @@
     <child link="proximal_roll_R_Link" />
     <axis xyz="1 0 0" />
-    <limit lower="-3.2288591161895095" upper="0.2617993877991494" effort="200" velocity="18.3" />
+    <limit lower="-3.19395248" upper="0.2617993877991494" effort="150" velocity="18.3" />
   </joint>
   <joint name="proximal_yaw_R_Joint" type="revolute">
@@ -347,5 +347,5 @@
     <child link="proximal_yaw_R_Link" />
     <axis xyz="0 0 1" />
-    <limit lower="-4.625122517784973" upper="0.5235987755982988" effort="70" velocity="22.52" />
+    <limit lower="-4.625122517784973" upper="0.5235987755982988" effort="60" velocity="22.52" />
   </joint>
   <joint name="knee_R_Joint" type="revolute">
@@ -354,5 +354,5 @@
     <child link="knee_R_Link" />
     <axis xyz="0 1 0" />
-    <limit lower="-0.2617993877991494" upper="2.6179938779914944" effort="200" velocity="18.3" />
+    <limit lower="-0.2617993877991494" upper="2.6179938779914944" effort="150" velocity="18.3" />
   </joint>
   <joint name="ankle_pitch_R_Joint" type="revolute">
@@ -361,5 +361,5 @@
     <child link="ankle_pitch_R_Link" />
     <axis xyz="0 1 0" />
-    <limit lower="-1.6231562043547263" upper="1.6231562043547263" effort="70" velocity="22.52" />
+    <limit lower="-1.6231562043547263" upper="1.6231562043547263" effort="60" velocity="22.52" />
   </joint>
   <!-- Gazebo Material / Friction (shared) -->

File: tron2/SF_TRON2A/meshes/robot.urdf (robot description, URDF)
Before this commit: robot bipedal_robot, 12 links, 11 joints
Joints:
- joint ankle_pitch_L_Joint: limit lower=-1.6231562043547263 upper=1.6231562043547263 effort=70 velocity=22.52 -> lower=-1.6231562043547263 upper=1.6231562043547263 effort=60 velocity=22.52
- joint ankle_pitch_R_Joint: limit lower=-1.6231562043547263 upper=1.6231562043547263 effort=70 velocity=22.52 -> lower=-1.6231562043547263 upper=1.6231562043547263 effort=60 velocity=22.52
- joint knee_L_Joint: limit lower=-0.2617993877991494 upper=2.6179938779914944 effort=200 velocity=18.3 -> lower=-0.2617993877991494 upper=2.6179938779914944 effort=150 velocity=18.3
- joint knee_R_Joint: limit lower=-0.2617993877991494 upper=2.6179938779914944 effort=200 velocity=18.3 -> lower=-0.2617993877991494 upper=2.6179938779914944 effort=150 velocity=18.3
- joint proximal_pitch_L_Joint: limit lower=-3.141592653589793 upper=2.600540585471551 effort=200 velocity=18.3 -> lower=-3.141592653589793 upper=2.600540585471551 effort=150 velocity=18.3
- joint proximal_pitch_R_Joint: limit lower=-3.141592653589793 upper=2.600540585471551 effort=200 velocity=18.3 -> lower=-3.141592653589793 upper=2.600540585471551 effort=150 velocity=18.3
- joint proximal_roll_L_Joint: limit lower=-0.2617993877991494 upper=3.2288591161895095 effort=200 velocity=18.3 -> lower=-0.2617993877991494 upper=3.19395248 effort=150 velocity=18.3
- joint proximal_roll_R_Joint: limit lower=-3.2288591161895095 upper=0.2617993877991494 effort=200 velocity=18.3 -> lower=-3.19395248 upper=0.2617993877991494 effort=150 velocity=18.3
- joint proximal_yaw_L_Joint: limit lower=-0.5235987755982988 upper=4.625122517784973 effort=70 velocity=22.52 -> lower=-0.5235987755982988 upper=4.625122517784973 effort=60 velocity=22.52
- joint proximal_yaw_R_Joint: limit lower=-4.625122517784973 upper=0.5235987755982988 effort=70 velocity=22.52 -> lower=-4.625122517784973 upper=0.5235987755982988 effort=60 velocity=22.52

File: tron2/SF_TRON2A/urdf/robot.urdf (robot description, URDF)
Before this commit: robot bipedal_robot, 14 links, 13 joints
Joints:
- joint ankle_pitch_L_Joint: limit lower=-1.6231562043547263 upper=1.6231562043547263 effort=70 velocity=22.52 -> lower=-1.6231562043547263 upper=1.6231562043547263 effort=60 velocity=22.52
- joint ankle_pitch_R_Joint: limit lower=-1.6231562043547263 upper=1.6231562043547263 effort=70 velocity=22.52 -> lower=-1.6231562043547263 upper=1.6231562043547263 effort=60 velocity=22.52
- joint knee_L_Joint: limit lower=-0.2617993877991494 upper=2.6179938779914944 effort=200 velocity=18.3 -> lower=-0.2617993877991494 upper=2.6179938779914944 effort=150 velocity=18.3
- joint knee_R_Joint: limit lower=-0.2617993877991494 upper=2.6179938779914944 effort=200 velocity=18.3 -> lower=-0.2617993877991494 upper=2.6179938779914944 effort=150 velocity=18.3
- joint proximal_pitch_L_Joint: limit lower=-3.141592653589793 upper=2.600540585471551 effort=200 velocity=18.3 -> lower=-3.141592653589793 upper=2.600540585471551 effort=150 velocity=18.3
- joint proximal_pitch_R_Joint: limit lower=-3.141592653589793 upper=2.600540585471551 effort=200 velocity=18.3 -> lower=-3.141592653589793 upper=2.600540585471551 effort=150 velocity=18.3
- joint proximal_roll_L_Joint: limit lower=-0.2617993877991494 upper=3.2288591161895095 effort=200 velocity=18.3 -> lower=-0.2617993877991494 upper=3.19395248 effort=150 velocity=18.3
- joint proximal_roll_R_Joint: limit lower=-3.2288591161895095 upper=0.2617993877991494 effort=200 velocity=18.3 -> lower=-3.19395248 upper=0.2617993877991494 effort=150 velocity=18.3
- joint proximal_yaw_L_Joint: limit lower=-0.5235987755982988 upper=4.625122517784973 effort=70 velocity=22.52 -> lower=-0.5235987755982988 upper=4.625122517784973 effort=60 velocity=22.52
- joint proximal_yaw_R_Joint: limit lower=-4.625122517784973 upper=0.5235987755982988 effort=70 velocity=22.52 -> lower=-4.625122517784973 upper=0.5235987755982988 effort=60 velocity=22.52

File: tron2/WFYG_TRON2A/meshes/robot.urdf (robot description, URDF)
Before this commit: robot bipedal_robot, 12 links, 11 joints
Joints:
- joint knee_L_Joint: limit lower=-2.6179938779914944 upper=0.2617993877991494 effort=200 velocity=18.3 -> lower=-2.6179938779914944 upper=0.2617993877991494 effort=150 velocity=18.3
- joint knee_R_Joint: limit lower=-2.6179938779914944 upper=0.2617993877991494 effort=200 velocity=18.3 -> lower=-2.6179938779914944 upper=0.2617993877991494 effort=150 velocity=18.3
- joint proximal_pitch_L_Joint: limit lower=-3.141592653589793 upper=2.600540585471551 effort=200 velocity=18.3 -> lower=-3.141592653589793 upper=2.600540585471551 effort=150 velocity=18.3
- joint proximal_pitch_R_Joint: limit lower=-3.141592653589793 upper=2.600540585471551 effort=200 velocity=18.3 -> lower=-3.141592653589793 upper=2.600540585471551 effort=150 velocity=18.3
- joint proximal_roll_L_Joint: limit lower=-0.2617993877991494 upper=3.2288591161895095 effort=200 velocity=18.3 -> lower=-0.2617993877991494 upper=3.19395248 effort=150 velocity=18.3
- joint proximal_roll_R_Joint: limit lower=-3.2288591161895095 upper=0.2617993877991494 effort=200 velocity=18.3 -> lower=-3.19395248 upper=0.2617993877991494 effort=150 velocity=18.3
- joint proximal_yaw_L_Joint: limit lower=-3.6651914291880923 upper=1.4835298641951802 effort=70 velocity=22.52 -> lower=-3.6651914291880923 upper=1.4835298641951802 effort=60 velocity=22.52
- joint proximal_yaw_R_Joint: limit lower=-1.4835298641951802 upper=3.6651914291880923 effort=70 velocity=22.52 -> lower=-1.4835298641951802 upper=3.6651914291880923 effort=60 velocity=22.52

File: tron2/WFYG_TRON2A/urdf/robot.urdf (robot description, URDF)
Before this commit: robot bipedal_robot, 27 links, 26 joints
Joints:
- joint knee_L_Joint: limit lower=-2.6179938779914944 upper=0.2617993877991494 effort=200.0 velocity=18.3 -> lower=-2.6179938779914944 upper=0.2617993877991494 effort=150 velocity=18.3
- joint knee_R_Joint: limit lower=-2.6179938779914944 upper=0.2617993877991494 effort=200.0 velocity=18.3 -> lower=-2.6179938779914944 upper=0.2617993877991494 effort=150 velocity=18.3
- joint proximal_pitch_L_Joint: limit lower=-3.141592653589793 upper=2.600540585471551 effort=200.0 velocity=18.3 -> lower=-3.141592653589793 upper=2.600540585471551 effort=150 velocity=18.3
- joint proximal_pitch_R_Joint: limit lower=-3.141592653589793 upper=2.600540585471551 effort=200.0 velocity=18.3 -> lower=-3.141592653589793 upper=2.600540585471551 effort=150 velocity=18.3
- joint proximal_roll_L_Joint: limit lower=-0.2617993877991494 upper=3.2288591161895095 effort=200.0 velocity=18.3 -> lower=-0.2617993877991494 upper=3.19395248 effort=150 velocity=18.3
- joint proximal_roll_R_Joint: limit lower=-3.2288591161895095 upper=0.2617993877991494 effort=200.0 velocity=18.3 -> lower=-3.19395248 upper=0.2617993877991494 effort=150 velocity=18.3
- joint proximal_yaw_L_Joint: limit lower=-3.6651914291880923 upper=1.4835298641951802 effort=70.0 velocity=22.52 -> lower=-3.6651914291880923 upper=1.4835298641951802 effort=60 velocity=22.52
- joint proximal_yaw_R_Joint: limit lower=-1.4835298641951802 upper=3.6651914291880923 effort=70.0 velocity=22.52 -> lower=-1.4835298641951802 upper=3.6651914291880923 effort=60 velocity=22.52

File: tron2/WFYG_TRON2A/urdf/robot_rl.urdf (robot description, URDF)
Before this commit: robot bipedal_robot, 25 links, 24 joints
Joints:
- joint knee_L_Joint: limit lower=-2.6179938779914944 upper=0.2617993877991494 effort=200.0 velocity=18.3 -> lower=-2.6179938779914944 upper=0.2617993877991494 effort=150 velocity=18.3
- joint knee_R_Joint: limit lower=-2.6179938779914944 upper=0.2617993877991494 effort=200.0 velocity=18.3 -> lower=-2.6179938779914944 upper=0.2617993877991494 effort=150 velocity=18.3
- joint proximal_pitch_L_Joint: limit lower=-3.141592653589793 upper=2.600540585471551 effort=200.0 velocity=18.3 -> lower=-3.141592653589793 upper=2.600540585471551 effort=150 velocity=18.3
- joint proximal_pitch_R_Joint: limit lower=-3.141592653589793 upper=2.600540585471551 effort=200.0 velocity=18.3 -> lower=-3.141592653589793 upper=2.600540585471551 effort=150 velocity=18.3
- joint proximal_roll_L_Joint: limit lower=-0.2617993877991494 upper=3.2288591161895095 effort=200.0 velocity=18.3 -> lower=-0.2617993877991494 upper=3.19395248 effort=150 velocity=18.3
- joint proximal_roll_R_Joint: limit lower=-3.2288591161895095 upper=0.2617993877991494 effort=200.0 velocity=18.3 -> lower=-3.19395248 upper=0.2617993877991494 effort=150 velocity=18.3
- joint proximal_yaw_L_Joint: limit lower=-3.6651914291880923 upper=1.4835298641951802 effort=70.0 velocity=22.52 -> lower=-3.6651914291880923 upper=1.4835298641951802 effort=60 velocity=22.52
- joint proximal_yaw_R_Joint: limit lower=-1.4835298641951802 upper=3.6651914291880923 effort=70.0 velocity=22.52 -> lower=-1.4835298641951802 upper=3.6651914291880923 effort=60 velocity=22.52

File: tron2/WFYG_TRON2A/xacro/robot.urdf.xacro (robot description, xacro)
@@ -304,5 +304,5 @@
     <child link="proximal_pitch_L_Link" />
     <axis xyz="0 0.99619 -0.087155" />
-    <limit lower="-3.141592653589793" upper="2.600540585471551" effort="200" velocity="18.3" />
+    <limit lower="-3.141592653589793" upper="2.600540585471551" effort="150" velocity="18.3" />
   </joint>
   <joint name="proximal_roll_L_Joint" type="revolute">
@@ -311,5 +311,5 @@
     <child link="proximal_roll_L_Link" />
     <axis xyz="1 0 0" />
-    <limit lower="-0.2617993877991494" upper="3.2288591161895095" effort="200" velocity="18.3" />
+    <limit lower="-0.2617993877991494" upper="3.19395248" effort="150" velocity="18.3" />
   </joint>
   <joint name="proximal_yaw_L_Joint" type="revolute">
@@ -318,5 +318,5 @@
     <child link="proximal_yaw_L_Link" />
     <axis xyz="0 0 1" />
-    <limit lower="-3.6651914291880923" upper="1.4835298641951802" effort="70" velocity="22.52" />
+    <limit lower="-3.6651914291880923" upper="1.4835298641951802" effort="60" velocity="22.52" />
   </joint>
   <joint name="knee_L_Joint" type="revolute">
@@ -325,5 +325,5 @@
     <child link="knee_L_Link" />
     <axis xyz="0 1 0" />
-    <limit lower="-2.6179938779914944" upper="0.2617993877991494" effort="200" velocity="18.3" />
+    <limit lower="-2.6179938779914944" upper="0.2617993877991494" effort="150" velocity="18.3" />
   </joint>
   <joint name="wheel_L_Joint" type="revolute">
@@ -339,5 +339,5 @@
     <child link="proximal_pitch_R_Link" />
     <axis xyz="0 0.99619 0.087155" />
-    <limit lower="-3.141592653589793" upper="2.600540585471551" effort="200" velocity="18.3" />
+    <limit lower="-3.141592653589793" upper="2.600540585471551" effort="150" velocity="18.3" />
   </joint>
   <joint name="proximal_roll_R_Joint" type="revolute">
@@ -346,5 +346,5 @@
     <child link="proximal_roll_R_Link" />
     <axis xyz="1 0 0" />
-    <limit lower="-3.2288591161895095" upper="0.2617993877991494" effort="200" velocity="18.3" />
+    <limit lower="-3.19395248" upper="0.2617993877991494" effort="150" velocity="18.3" />
   </joint>
   <joint name="proximal_yaw_R_Joint" type="revolute">
@@ -353,5 +353,5 @@
     <child link="proximal_yaw_R_Link" />
     <axis xyz="0 0 1" />
-    <limit lower="-1.4835298641951802" upper="3.6651914291880923" effort="70" velocity="22.52" />
+    <limit lower="-1.4835298641951802" upper="3.6651914291880923" effort="60" velocity="22.52" />
   </joint>
   <joint name="knee_R_Joint" type="revolute">
@@ -360,5 +360,5 @@
     <child link="knee_R_Link" />
     <axis xyz="0 1 0" />
-    <limit lower="-2.6179938779914944" upper="0.2617993877991494" effort="200" velocity="18.3" />
+    <limit lower="-2.6179938779914944" upper="0.2617993877991494" effort="150" velocity="18.3" />
   </joint>
   <joint name="wheel_R_Joint" type="revolute">
