Commit message: Feat: modify joint effort for sim2real, and proximal_roll limit joint pos

File: tron2/WF_TRON2A/urdf/robot.urdf (robot description, URDF)
Before this commit: robot bipedal_robot, 12 links, 11 joints
Joints:
- joint knee_L_Joint: limit lower=-2.6179938779914944 upper=0.2617993877991494 effort=200 velocity=18.3 -> lower=-2.6179938779914944 upper=0.2617993877991494 effort=150 velocity=18.3
- joint knee_R_Joint: limit lower=-2.6179938779914944 upper=0.2617993877991494 effort=200 velocity=18.3 -> lower=-2.6179938779914944 upper=0.2617993877991494 effort=150 velocity=18.3
- joint proximal_pitch_L_Joint: limit lower=-3.141592653589793 upper=2.600540585471551 effort=200 velocity=18.3 -> lower=-3.141592653589793 upper=2.600540585471551 effort=150 velocity=18.3
- joint proximal_pitch_R_Joint: limit lower=-3.141592653589793 upper=2.600540585471551 effort=200 velocity=18.3 -> lower=-3.141592653589793 upper=2.600540585471551 effort=150 velocity=18.3
- joint proximal_roll_L_Joint: limit lower=-0.2617993877991494 upper=3.2288591161895095 effort=200 velocity=18.3 -> lower=-0.2617993877991494 upper=3.19395248 effort=150 velocity=18.3
- joint proximal_roll_R_Joint: limit lower=-3.2288591161895095 upper=0.2617993877991494 effort=200 velocity=18.3 -> lower=-3.19395248 upper=0.2617993877991494 effort=150 velocity=18.3
- joint proximal_yaw_L_Joint: limit lower=-3.6651914291880923 upper=1.4835298641951802 effort=70 velocity=22.52 -> lower=-3.6651914291880923 upper=1.4835298641951802 effort=60 velocity=22.52
- joint proximal_yaw_R_Joint: limit lower=-1.4835298641951802 upper=3.6651914291880923 effort=70 velocity=22.52 -> lower=-1.4835298641951802 upper=3.6651914291880923 effort=60 velocity=22.52

File: tron2/WF_TRON2A/urdf/robot_primitive.urdf (robot description, URDF)
Before this commit: robot bipedal_robot, 12 links, 11 joints
Joints:
- joint knee_L_Joint: limit lower=-2.6179938779914944 upper=0.2617993877991494 effort=200 velocity=18.3 -> lower=-2.6179938779914944 upper=0.2617993877991494 effort=150 velocity=18.3
- joint knee_R_Joint: limit lower=-2.6179938779914944 upper=0.2617993877991494 effort=200 velocity=18.3 -> lower=-2.6179938779914944 upper=0.2617993877991494 effort=150 velocity=18.3
- joint proximal_pitch_L_Joint: limit lower=-3.141592653589793 upper=2.600540585471551 effort=200 velocity=18.3 -> lower=-3.141592653589793 upper=2.600540585471551 effort=150 velocity=18.3
- joint proximal_pitch_R_Joint: limit lower=-3.141592653589793 upper=2.600540585471551 effort=200 velocity=18.3 -> lower=-3.141592653589793 upper=2.600540585471551 effort=150 velocity=18.3
- joint proximal_roll_L_Joint: limit lower=-0.2617993877991494 upper=3.2288591161895095 effort=200 velocity=18.3 -> lower=-0.2617993877991494 upper=3.19395248 effort=150 velocity=18.3
- joint proximal_roll_R_Joint: limit lower=-3.2288591161895095 upper=0.2617993877991494 effort=200 velocity=18.3 -> lower=-3.19395248 upper=0.2617993877991494 effort=150 velocity=18.3
- joint proximal_yaw_L_Joint: limit lower=-3.6651914291880923 upper=1.4835298641951802 effort=70 velocity=22.52 -> lower=-3.6651914291880923 upper=1.4835298641951802 effort=60 velocity=22.52
- joint proximal_yaw_R_Joint: limit lower=-1.4835298641951802 upper=3.6651914291880923 effort=70 velocity=22.52 -> lower=-1.4835298641951802 upper=3.6651914291880923 effort=60 velocity=22.52

File: tron2/WF_TRON2A/urdf/robot_rl.urdf (robot description, URDF)
Before this commit: robot bipedal_robot, 12 links, 11 joints
Joints:
- joint knee_L_Joint: limit lower=-2.6179938779914944 upper=0.2617993877991494 effort=200 velocity=18.3 -> lower=-2.6179938779914944 upper=0.2617993877991494 effort=150 velocity=18.3
- joint knee_R_Joint: limit lower=-2.6179938779914944 upper=0.2617993877991494 effort=200 velocity=18.3 -> lower=-2.6179938779914944 upper=0.2617993877991494 effort=150 velocity=18.3
- joint proximal_pitch_L_Joint: limit lower=-3.141592653589793 upper=2.600540585471551 effort=200 velocity=18.3 -> lower=-3.141592653589793 upper=2.600540585471551 effort=150 velocity=18.3
- joint proximal_pitch_R_Joint: limit lower=-3.141592653589793 upper=2.600540585471551 effort=200 velocity=18.3 -> lower=-3.141592653589793 upper=2.600540585471551 effort=150 velocity=18.3
- joint proximal_roll_L_Joint: limit lower=-0.2617993877991494 upper=3.2288591161895095 effort=200 velocity=18.3 -> lower=-0.2617993877991494 upper=3.19395248 effort=150 velocity=18.3
- joint proximal_roll_R_Joint: limit lower=-3.2288591161895095 upper=0.2617993877991494 effort=200 velocity=18.3 -> lower=-3.19395248 upper=0.2617993877991494 effort=150 velocity=18.3
- joint proximal_yaw_L_Joint: limit lower=-3.6651914291880923 upper=1.4835298641951802 effort=70 velocity=22.52 -> lower=-3.6651914291880923 upper=1.4835298641951802 effort=60 velocity=22.52
- joint proximal_yaw_R_Joint: limit lower=-1.4835298641951802 upper=3.6651914291880923 effort=70 velocity=22.52 -> lower=-1.4835298641951802 upper=3.6651914291880923 effort=60 velocity=22.52
