Commit message: feat: regenerate WF_TRON2A

File: tron2/WF_TRON2A/urdf/robot.urdf (robot description, URDF)
Before this commit: robot bipedal_robot, 12 links, 11 joints
Links:
- added link base_imu, mass 0.01
- added link d435_Link; visual box size=0.01 0.01 0.001
- added link d435_optical_frame
- link base_Link: geometry collision mesh filename=package://bipedal_robot/meshes/base_Link.STL; visual mesh filename=package://bipedal_robot/meshes/base_Link.STL
- link knee_L_Link: geometry collision mesh filename=package://bipedal_robot/meshes/knee_L_Link.STL; visual mesh filename=package://bipedal_robot/meshes/knee_L_Link.STL
- link knee_R_Link: geometry collision mesh filename=package://bipedal_robot/meshes/knee_R_Link.STL; visual mesh filename=package://bipedal_robot/meshes/knee_R_Link.STL
- link proximal_pitch_L_Link: geometry collision mesh filename=package://bipedal_robot/meshes/proximal_pitch_L_Link.STL; visual mesh filename=package://bipedal_robot/meshes/proximal_pitch_L_Link.STL
- link proximal_pitch_R_Link: geometry collision mesh filename=package://bipedal_robot/meshes/proximal_pitch_R_Link.STL; visual mesh filename=package://bipedal_robot/meshes/proximal_pitch_R_Link.STL
- link proximal_roll_L_Link: geometry collision mesh filename=package://bipedal_robot/meshes/proximal_roll_L_Link.STL; visual mesh filename=package://bipedal_robot/meshes/proximal_roll_L_Link.STL
- link proximal_roll_R_Link: geometry collision mesh filename=package://bipedal_robot/meshes/proximal_roll_R_Link.STL; visual mesh filename=package://bipedal_robot/meshes/proximal_roll_R_Link.STL
- link proximal_yaw_L_Link: geometry collision mesh filename=package://bipedal_robot/meshes/proximal_yaw_L_Link.STL; visual mesh filename=package://bipedal_robot/meshes/proximal_yaw_L_Link.STL
- link proximal_yaw_R_Link: geometry collision mesh filename=package://bipedal_robot/meshes/proximal_yaw_R_Link.STL; visual mesh filename=package://bipedal_robot/meshes/proximal_yaw_R_Link.STL
- link wheel_L_Link: geometry collision cylinder length=0.045 radius=0.1; visual mesh filename=package://bipedal_robot/meshes/wheel_L_Link.STL
- link wheel_R_Link: geometry collision cylinder length=0.045 radius=0.1; visual mesh filename=package://bipedal_robot/meshes/wheel_R_Link.STL
Joints:
- added joint base_imu_Joint: type fixed, parent base_Link, child base_imu, origin xyz=0.0 0.0 0.0 rpy=0.0 0.0 0.0
- added joint d435_joint: type fixed, parent limx_imu, child d435_Link, origin xyz=0.12213 0.01759 0.00599 rpy=0.0 1.063778179 0.0
- added joint d435_optical_joint: type fixed, parent d435_Link, child d435_optical_frame, origin xyz=0 0 0 rpy=-1.5707963267948966 0 -1.5707963267948966
- joint knee_L_Joint: axis 0 1 0 -> 0.0 1.0 0.0; limit lower=-2.6179938779914944 upper=0.2617993877991494 effort=150 velocity=18.3 -> lower=-2.6179938779914944 upper=0.2617993877991494 effort=150.0 velocity=18.3; origin xyz=0.004 0.032 -0.2126 rpy=0 0 0 -> xyz=0.004 0.032 -0.2126 rpy=0.0 0.0 0.0
- joint knee_R_Joint: axis 0 1 0 -> 0.0 1.0 0.0; limit lower=-2.6179938779914944 upper=0.2617993877991494 effort=150 velocity=18.3 -> lower=-2.6179938779914944 upper=0.2617993877991494 effort=150.0 velocity=18.3; origin xyz=0.004 -0.032 -0.2126 rpy=0 0 0 -> xyz=0.004 -0.032 -0.2126 rpy=0.0 0.0 0.0
- joint limx_imu_joint: origin xyz=0. 0. 0. rpy=0. 0. 0. -> xyz=0.0 0.0 0.0 rpy=0.0 0.0 0.0
- joint proximal_pitch_L_Joint: axis 0 0.99619 -0.087155 -> 0.0 0.9961947268929313 -0.0871554135479712; limit lower=-3.141592653589793 upper=2.600540585471551 effort=150 velocity=18.3 -> lower=-3.141592653589793 upper=2.600540585471551 effort=150.0 velocity=18.3; origin xyz=-0.00044 0.09178 0.05474 rpy=0 0 0 -> xyz=-0.00044 0.09178 0.05474 rpy=0.0 0.0 0.0
- joint proximal_pitch_R_Joint: axis 0 0.99619 0.087155 -> 0.0 0.9961947268929313 0.0871554135479712; limit lower=-3.141592653589793 upper=2.600540585471551 effort=150 velocity=18.3 -> lower=-3.141592653589793 upper=2.600540585471551 effort=150.0 velocity=18.3; origin xyz=-0.00044 -0.09178 0.05474 rpy=0 0 0 -> xyz=-0.00044 -0.09178 0.05474 rpy=0.0 0.0 0.0
- joint proximal_roll_L_Joint: axis 1 0 0 -> 1.0 0.0 0.0; limit lower=-0.2617993877991494 upper=3.19395248 effort=150 velocity=18.3 -> lower=-0.2617993877991494 upper=3.1939524787897455 effort=150.0 velocity=18.3; origin xyz=-0.032 0.0758 -0.00663 rpy=0 0 0 -> xyz=-0.032 0.0758 -0.00663 rpy=0.0 0.0 0.0
- joint proximal_roll_R_Joint: axis 1 0 0 -> 1.0 0.0 0.0; limit lower=-3.19395248 upper=0.2617993877991494 effort=150 velocity=18.3 -> lower=-3.1939524787897455 upper=0.2617993877991494 effort=150.0 velocity=18.3; origin xyz=-0.032 -0.0758 -0.00663 rpy=0 0 0 -> xyz=-0.032 -0.0758 -0.00663 rpy=0.0 0.0 0.0
- joint proximal_yaw_L_Joint: axis 0 0 1 -> 0.0 0.0 1.0; limit lower=-3.6651914291880923 upper=1.4835298641951802 effort=60 velocity=22.52 -> lower=-3.6651914291880923 upper=1.4835298641951802 effort=60.0 velocity=22.52; origin xyz=0.032 0.0 -0.1374 rpy=0 0 0 -> xyz=0.032 0.0 -0.1374 rpy=0.0 0.0 0.0
- joint proximal_yaw_R_Joint: axis 0 0 1 -> 0.0 0.0 1.0; limit lower=-1.4835298641951802 upper=3.6651914291880923 effort=60 velocity=22.52 -> lower=-1.4835298641951802 upper=3.6651914291880923 effort=60.0 velocity=22.52; origin xyz=0.032 -0.0 -0.1374 rpy=0 0 0 -> xyz=0.032 -0.0 -0.1374 rpy=0.0 0.0 0.0
- joint wheel_L_Joint: axis 0 1 0 -> 0.0 1.0 0.0; limit lower=-1745329.2519943293 upper=1745329.2519943293 effort=22 velocity=41.89 -> lower=-1745329.2519943295 upper=1745329.2519943295 effort=22.0 velocity=41.89; origin xyz=-0.004 0.013 -0.35 rpy=0 0 0 -> xyz=-0.004 0.013 -0.35 rpy=0.0 0.0 0.0
- joint wheel_R_Joint: axis 0 1 0 -> 0.0 1.0 0.0; limit lower=-1745329.2519943293 upper=1745329.2519943293 effort=22 velocity=41.89 -> lower=-1745329.2519943295 upper=1745329.2519943295 effort=22.0 velocity=41.89; origin xyz=-0.004 -0.013 -0.35 rpy=0 0 0 -> xyz=-0.004 -0.013 -0.35 rpy=0.0 0.0 0.0

File: tron2/WF_TRON2A/urdf/robot_rl.urdf (robot description, URDF)
Before this commit: robot bipedal_robot, 12 links, 11 joints
Links:
- removed link limx_imu
- added link base_imu, mass 0.01
Joints:
- removed joint limx_imu_joint
- added joint base_imu_Joint: type fixed, parent base_Link, child base_imu, origin xyz=0.0 0.0 0.0 rpy=0.0 0.0 0.0
- joint knee_L_Joint: axis 0 1 0 -> 0.0 1.0 0.0; limit lower=-2.6179938779914944 upper=0.2617993877991494 effort=150 velocity=18.3 -> lower=-2.6179938779914944 upper=0.2617993877991494 effort=150.0 velocity=18.3; origin xyz=0.004 0.032 -0.2126 rpy=0 0 0 -> xyz=0.004 0.032 -0.2126 rpy=0.0 0.0 0.0
- joint knee_R_Joint: axis 0 1 0 -> 0.0 1.0 0.0; limit lower=-2.6179938779914944 upper=0.2617993877991494 effort=150 velocity=18.3 -> lower=-2.6179938779914944 upper=0.2617993877991494 effort=150.0 velocity=18.3; origin xyz=0.004 -0.032 -0.2126 rpy=0 0 0 -> xyz=0.004 -0.032 -0.2126 rpy=0.0 0.0 0.0
- joint proximal_pitch_L_Joint: axis 0 0.99619 -0.087155 -> 0.0 0.9961947268929313 -0.0871554135479712; limit lower=-3.141592653589793 upper=2.600540585471551 effort=150 velocity=18.3 -> lower=-3.141592653589793 upper=2.600540585471551 effort=150.0 velocity=18.3; origin xyz=-0.00044 0.09178 0.05474 rpy=0 0 0 -> xyz=-0.00044 0.09178 0.05474 rpy=0.0 0.0 0.0
- joint proximal_pitch_R_Joint: axis 0 0.99619 0.087155 -> 0.0 0.9961947268929313 0.0871554135479712; limit lower=-3.141592653589793 upper=2.600540585471551 effort=150 velocity=18.3 -> lower=-3.141592653589793 upper=2.600540585471551 effort=150.0 velocity=18.3; origin xyz=-0.00044 -0.09178 0.05474 rpy=0 0 0 -> xyz=-0.00044 -0.09178 0.05474 rpy=0.0 0.0 0.0
- joint proximal_roll_L_Joint: axis 1 0 0 -> 1.0 0.0 0.0; limit lower=-0.2617993877991494 upper=3.19395248 effort=150 velocity=18.3 -> lower=-0.2617993877991494 upper=3.1939524787897455 effort=150.0 velocity=18.3; origin xyz=-0.032 0.0758 -0.00663 rpy=0 0 0 -> xyz=-0.032 0.0758 -0.00663 rpy=0.0 0.0 0.0
- joint proximal_roll_R_Joint: axis 1 0 0 -> 1.0 0.0 0.0; limit lower=-3.19395248 upper=0.2617993877991494 effort=150 velocity=18.3 -> lower=-3.1939524787897455 upper=0.2617993877991494 effort=150.0 velocity=18.3; origin xyz=-0.032 -0.0758 -0.00663 rpy=0 0 0 -> xyz=-0.032 -0.0758 -0.00663 rpy=0.0 0.0 0.0
- joint proximal_yaw_L_Joint: axis 0 0 1 -> 0.0 0.0 1.0; limit lower=-3.6651914291880923 upper=1.4835298641951802 effort=60 velocity=22.52 -> lower=-3.6651914291880923 upper=1.4835298641951802 effort=60.0 velocity=22.52; origin xyz=0.032 0.0 -0.1374 rpy=0 0 0 -> xyz=0.032 0.0 -0.1374 rpy=0.0 0.0 0.0
- joint proximal_yaw_R_Joint: axis 0 0 1 -> 0.0 0.0 1.0; limit lower=-1.4835298641951802 upper=3.6651914291880923 effort=60 velocity=22.52 -> lower=-1.4835298641951802 upper=3.6651914291880923 effort=60.0 velocity=22.52; origin xyz=0.032 -0.0 -0.1374 rpy=0 0 0 -> xyz=0.032 -0.0 -0.1374 rpy=0.0 0.0 0.0
- joint wheel_L_Joint: axis 0 1 0 -> 0.0 1.0 0.0; limit lower=-1745329.2519943293 upper=1745329.2519943293 effort=22 velocity=41.89 -> lower=-1745329.2519943295 upper=1745329.2519943295 effort=22.0 velocity=41.89; origin xyz=-0.004 0.013 -0.35 rpy=0 0 0 -> xyz=-0.004 0.013 -0.35 rpy=0.0 0.0 0.0
- joint wheel_R_Joint: axis 0 1 0 -> 0.0 1.0 0.0; limit lower=-1745329.2519943293 upper=1745329.2519943293 effort=22 velocity=41.89 -> lower=-1745329.2519943295 upper=1745329.2519943295 effort=22.0 velocity=41.89; origin xyz=-0.004 -0.013 -0.35 rpy=0 0 0 -> xyz=-0.004 -0.013 -0.35 rpy=0.0 0.0 0.0
