Commit message: Fix: update axis of the first joint in SF

File: tron2/SF_TRON2A/urdf/robot.urdf (robot description, URDF)
Before this commit: robot bipedal_robot, 12 links, 11 joints
Joints:
- joint ankle_pitch_R_Joint: axis 0 1 0 -> 0 0.99619 0.087155
- joint proximal_pitch_L_Joint: axis 0 1 0 -> 0 0.99619 -0.087155

Commit message: Feat/sf tron2 rotate yaw 180

File: tron2/SF_TRON2A/urdf/robot.urdf (robot description, URDF)
Before this commit: robot bipedal_robot, 14 links, 13 joints
Links:
- link ankle_pitch_L_Link: geometry collision mesh filename=package://robot_description/tron2/SF_TRON2B/meshes/ankle_pi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; visual mesh filename=package://robot_description/tron2/SF_TRON2B/meshes/ankle_pi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
- link ankle_pitch_R_Link: geometry collision mesh filename=package://robot_description/tron2/SF_TRON2B/meshes/ankle_pi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; visual mesh filename=package://robot_description/tron2/SF_TRON2B/meshes/ankle_pi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
- link base_Link: geometry collision mesh filename=package://robot_description/tron2/SF_TRON2B/meshes/base_Lin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; visual mesh filename=package://robot_description/tron2/SF_TRON2B/meshes/base_Lin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
- link knee_L_Link: geometry collision mesh filename=package://robot_description/tron2/SF_TRON2B/meshes/knee_L_L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; visual mesh filename=package://robot_description/tron2/SF_TRON2B/meshes/knee_L_L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
- link knee_R_Link: geometry collision mesh filename=package://robot_description/tron2/SF_TRON2B/meshes/knee_R_L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; visual mesh filename=package://robot_description/tron2/SF_TRON2B/meshes/knee_R_L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
- link proximal_pitch_L_Link: geometry collision mesh filename=package://robot_description/tron2/SF_TRON2B/meshes/proximal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; visual mesh filename=package://robot_description/tron2/SF_TRON2B/meshes/proximal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
- link proximal_pitch_R_Link: geometry collision mesh filename=package://robot_description/tron2/SF_TRON2B/meshes/proximal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; visual mesh filename=package://robot_description/tron2/SF_TRON2B/meshes/proximal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
- link proximal_roll_L_Link: geometry collision mesh filename=package://robot_description/tron2/SF_TRON2B/meshes/proximal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; visual mesh filename=package://robot_description/tron2/SF_TRON2B/meshes/proximal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
- link proximal_roll_R_Link: geometry collision mesh filename=package://robot_description/tron2/SF_TRON2B/meshes/proximal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; visual mesh filename=package://robot_description/tron2/SF_TRON2B/meshes/proximal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
- link proximal_yaw_L_Link: geometry collision mesh filename=package://robot_description/tron2/SF_TRON2B/meshes/proximal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; visual mesh filename=package://robot_description/tron2/SF_TRON2B/meshes/proximal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
- link proximal_yaw_R_Link: geometry collision mesh filename=package://robot_description/tron2/SF_TRON2B/meshes/proximal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; visual mesh filename=package://robot_description/tron2/SF_TRON2B/meshes/proximal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
Joints:
- joint ankle_pitch_L_Joint: axis 0 1 0 -> 0.0 1.0 0.0; limit lower=-1.6231562043547263 upper=1.6231562043547263 effort=60 velocity=22.52 -> lower=-1.6231562043547265 upper=1.6231562043547265 effort=60.0 velocity=22.52; origin xyz=0.004 0.06775 -0.35 rpy=0 0 0 -> xyz=-0.004 -0.06775 -0.35 rpy=0.0 0.0 0.0
- joint ankle_pitch_R_Joint: axis 0 1 0 -> 0.0 1.0 0.0; limit lower=-1.6231562043547263 upper=1.6231562043547263 effort=60 velocity=22.52 -> lower=-1.6231562043547265 upper=1.6231562043547265 effort=60.0 velocity=22.52; origin xyz=0.004 -0.06775 -0.35 rpy=0 0 0 -> xyz=-0.004 0.06775 -0.35 rpy=-0.0 0.0 -0.0
- joint d435_joint: origin xyz=0.12213 0.01759 0.00599 rpy=0 1.063778179 0 -> xyz=0.12213 0.01759 0.00599 rpy=0.0 1.063778179 0.0
- joint knee_L_Joint: axis 0 1 0 -> 0.0 1.0 0.0; limit lower=-0.2617993877991494 upper=2.6179938779914944 effort=150 velocity=18.3 -> lower=-2.6179938779914944 upper=0.2617993877991494 effort=150.0 velocity=18.3; origin xyz=-0.004 -0.032 -0.2126 rpy=0 0 0 -> xyz=0.004 0.032 -0.2126 rpy=0.0 0.0 0.0
- joint knee_R_Joint: axis 0 1 0 -> 0.0 1.0 0.0; limit lower=-0.2617993877991494 upper=2.6179938779914944 effort=150 velocity=18.3 -> lower=-2.6179938779914944 upper=0.2617993877991494 effort=150.0 velocity=18.3; origin xyz=-0.004 0.032 -0.2126 rpy=0 0 0 -> xyz=0.004 -0.032 -0.2126 rpy=-0.0 0.0 -0.0
- joint limx_imu_joint: origin xyz=0. 0. 0. rpy=0. 0. 0. -> xyz=0.0 0.0 0.0 rpy=0.0 0.0 0.0
- joint proximal_pitch_L_Joint: axis 0 0.99619 -0.087155 -> 0.0 0.9961947268929313 -0.0871554135479712; limit lower=-3.141592653589793 upper=2.600540585471551 effort=150 velocity=18.3 -> lower=-3.141592653589793 upper=2.600540585471551 effort=150.0 velocity=18.3; origin xyz=-0.00044 0.09178 0.05474 rpy=0 0 0 -> xyz=-0.00044 0.09178 0.05474 rpy=0.0 0.0 0.0
- joint proximal_pitch_R_Joint: axis 0 0.99619 0.087155 -> 0.0 0.9961947268929313 0.0871554135479712; limit lower=-3.141592653589793 upper=2.600540585471551 effort=150 velocity=18.3 -> lower=-3.141592653589793 upper=2.600540585471551 effort=150.0 velocity=18.3; origin xyz=-0.00044 -0.09178 0.05474 rpy=0 0 0 -> xyz=-0.00044 -0.09178 0.05474 rpy=0.0 0.0 0.0
- joint proximal_roll_L_Joint: axis 1 0 0 -> 1.0 0.0 0.0; limit lower=-0.2617993877991494 upper=3.19395248 effort=150 velocity=18.3 -> lower=-0.2617993877991494 upper=3.19395248 effort=150.0 velocity=18.3; origin xyz=-0.032 0.0758 -0.00663 rpy=0 0 0 -> xyz=-0.032 0.0758 -0.00663 rpy=0.0 0.0 0.0
- joint proximal_roll_R_Joint: axis 1 0 0 -> 1.0 0.0 0.0; limit lower=-3.19395248 upper=0.2617993877991494 effort=150 velocity=18.3 -> lower=-3.19395248 upper=0.2617993877991494 effort=150.0 velocity=18.3; origin xyz=-0.032 -0.0758 -0.00663 rpy=0 0 0 -> xyz=-0.032 -0.0758 -0.00663 rpy=-0.0 0.0 -0.0
- joint proximal_yaw_L_Joint: axis 0 0 1 -> 0.0 0.0 1.0; limit lower=-0.5235987755982988 upper=4.625122517784973 effort=60 velocity=22.52 -> lower=-3.6651914291880923 upper=1.4835298641951802 effort=60.0 velocity=22.52; origin xyz=0.032 0.0 -0.1374 rpy=0 0 0 -> xyz=0.032 0.0 -0.1374 rpy=0.0 0.0 0.0
- joint proximal_yaw_R_Joint: axis 0 0 1 -> 0.0 0.0 1.0; limit lower=-4.625122517784973 upper=0.5235987755982988 effort=60 velocity=22.52 -> lower=-1.4835298641951802 upper=3.6651914291880923 effort=60.0 velocity=22.52; origin xyz=0.032 -0.0 -0.1374 rpy=0 0 0 -> xyz=0.032 -0.0 -0.1374 rpy=-0.0 0.0 -0.0

Commit message: feat: regenerate SF_TRON2A

File: tron2/SF_TRON2A/urdf/robot.urdf (robot description, URDF)
Before this commit: robot bipedal_robot, 14 links, 13 joints
Links:
- added link base_imu, mass 0.01
- link ankle_pitch_L_Link: geometry collision box size=0.14 0.06 0.025; collision sphere radius=0.0025
- link ankle_pitch_R_Link: geometry collision box size=0.14 0.06 0.025; collision sphere radius=0.0025
- link base_Link: geometry collision mesh filename=package://bipedal_robot/meshes/base_Link.STL; visual mesh filename=package://bipedal_robot/meshes/base_Link.STL
- link knee_L_Link: geometry collision mesh filename=package://bipedal_robot/meshes/knee_L_Link.STL; visual mesh filename=package://bipedal_robot/meshes/knee_L_Link.STL
- link knee_R_Link: geometry collision mesh filename=package://bipedal_robot/meshes/knee_R_Link.STL; visual mesh filename=package://bipedal_robot/meshes/knee_R_Link.STL
- link proximal_pitch_L_Link: geometry collision mesh filename=package://bipedal_robot/meshes/proximal_pitch_L_Link.STL; visual mesh filename=package://bipedal_robot/meshes/proximal_pitch_L_Link.STL
- link proximal_pitch_R_Link: geometry collision mesh filename=package://bipedal_robot/meshes/proximal_pitch_R_Link.STL; visual mesh filename=package://bipedal_robot/meshes/proximal_pitch_R_Link.STL
- link proximal_roll_L_Link: geometry collision mesh filename=package://bipedal_robot/meshes/proximal_roll_L_Link.STL; visual mesh filename=package://bipedal_robot/meshes/proximal_roll_L_Link.STL
- link proximal_roll_R_Link: geometry collision mesh filename=package://bipedal_robot/meshes/proximal_roll_R_Link.STL; visual mesh filename=package://bipedal_robot/meshes/proximal_roll_R_Link.STL
- link proximal_yaw_L_Link: geometry collision mesh filename=package://bipedal_robot/meshes/proximal_yaw_L_Link.STL; visual mesh filename=package://bipedal_robot/meshes/proximal_yaw_L_Link.STL
- link proximal_yaw_R_Link: geometry collision mesh filename=package://bipedal_robot/meshes/proximal_yaw_R_Link.STL; visual mesh filename=package://bipedal_robot/meshes/proximal_yaw_R_Link.STL
Joints:
- added joint base_imu_Joint: type fixed, parent base_Link, child base_imu, origin xyz=0.0 0.0 0.0 rpy=0.0 0.0 0.0
- joint ankle_pitch_R_Joint: origin xyz=-0.004 0.06775 -0.35 rpy=-0.0 0.0 -0.0 -> xyz=-0.004 0.06775 -0.35 rpy=0.0 0.0 0.0
- joint knee_R_Joint: origin xyz=0.004 -0.032 -0.2126 rpy=-0.0 0.0 -0.0 -> xyz=0.004 -0.032 -0.2126 rpy=0.0 0.0 0.0
- joint proximal_pitch_L_Joint: axis 0.0 0.9961947268929313 -0.0871554135479712 -> 0.0 0.996194726892931 -0.0871554135479712
- joint proximal_pitch_R_Joint: axis 0.0 0.9961947268929313 0.0871554135479712 -> 0.0 0.996194726892931 0.0871554135479712
- joint proximal_roll_L_Joint: limit lower=-0.2617993877991494 upper=3.19395248 effort=150.0 velocity=18.3 -> lower=-0.2617993877991494 upper=3.1939524787897455 effort=150.0 velocity=18.3
- joint proximal_roll_R_Joint: limit lower=-3.19395248 upper=0.2617993877991494 effort=150.0 velocity=18.3 -> lower=-3.1939524787897455 upper=0.2617993877991494 effort=150.0 velocity=18.3; origin xyz=-0.032 -0.0758 -0.00663 rpy=-0.0 0.0 -0.0 -> xyz=-0.032 -0.0758 -0.00663 rpy=0.0 0.0 0.0
- joint proximal_yaw_R_Joint: origin xyz=0.032 -0.0 -0.1374 rpy=-0.0 0.0 -0.0 -> xyz=0.032 -0.0 -0.1374 rpy=0.0 0.0 0.0

File: tron2/SF_TRON2A/urdf/robot_rl.urdf (robot description, URDF)
Before this commit: robot bipedal_robot, 11 links, 10 joints
Links:
- added link base_imu, mass 0.01
Joints:
- added joint base_imu_Joint: type fixed, parent base_Link, child base_imu, origin xyz=0.0 0.0 0.0 rpy=0.0 0.0 0.0
- joint ankle_pitch_R_Joint: origin xyz=-0.004 0.06775 -0.35 rpy=-0.0 0.0 -0.0 -> xyz=-0.004 0.06775 -0.35 rpy=0.0 0.0 0.0
- joint knee_R_Joint: origin xyz=0.004 -0.032 -0.2126 rpy=-0.0 0.0 -0.0 -> xyz=0.004 -0.032 -0.2126 rpy=0.0 0.0 0.0
- joint proximal_pitch_L_Joint: axis 0.0 0.9961947268929313 -0.0871554135479712 -> 0.0 0.996194726892931 -0.0871554135479712
- joint proximal_pitch_R_Joint: axis 0.0 0.9961947268929313 0.0871554135479712 -> 0.0 0.996194726892931 0.0871554135479712
- joint proximal_roll_L_Joint: limit lower=-0.2617993877991494 upper=3.19395248 effort=150.0 velocity=18.3 -> lower=-0.2617993877991494 upper=3.1939524787897455 effort=150.0 velocity=18.3
- joint proximal_roll_R_Joint: limit lower=-3.19395248 upper=0.2617993877991494 effort=150.0 velocity=18.3 -> lower=-3.1939524787897455 upper=0.2617993877991494 effort=150.0 velocity=18.3; origin xyz=-0.032 -0.0758 -0.00663 rpy=-0.0 0.0 -0.0 -> xyz=-0.032 -0.0758 -0.00663 rpy=0.0 0.0 0.0
- joint proximal_yaw_R_Joint: origin xyz=0.032 -0.0 -0.1374 rpy=-0.0 0.0 -0.0 -> xyz=0.032 -0.0 -0.1374 rpy=0.0 0.0 0.0
