Commit message: feat(SFYG_TRON2A): align xacro with piper-x URDF
The piper-x rewrite (commit 54f0a7c) reshaped SFYG: legs received the
yaw_180 rotation, ankles gained 12 collision primitives (1 box + 11
spheres), the 7-DOF arm + flange was replaced by a 6-DOF arm linked
directly to the gripper base, and antenna_L/R, camera_mount, and radar
peripherals were added.

robot.urdf.xacro:
- Apply leg yaw_180 (mirrors the SF change).
- Replace the single-mesh ankle collision with 12 primitives.
- Add transition, arm_base, arm1..arm6, gripper_base, gripper1/2,
  antenna_L/R, camera_mount, and radar links/joints.
- Add gazebo friction/material blocks for every new link.
- Refresh proximal_roll limits and proximal_pitch axis precision.

macros.xacro:
- Add ROS1 transmissions for arm1..arm6 and gripper1/2.
- Add matching ros2_control joint blocks.

Co-Authored-By: Claude Opus 4.7 (1M context) <noreply@anthropic.com>

File: tron2/SFYG_TRON2A/xacro/macros.xacro (robot description, xacro)
@@ -156,4 +156,84 @@
       </actuator>
     </transmission>
+    <transmission name="arm1_Joint_trans">
+      <type>transmission_interface/SimpleTransmission</type>
+      <joint name="arm1_Joint">
+        <hardwareInterface>hardware_interface/EffortJointInterface</hardwareInterface>
+      </joint>
+      <actuator name="arm1_Joint_motor">
+        <hardwareInterface>hardware_interface/EffortJointInterface</hardwareInterface>
+        <mechanicalReduction>1</mechanicalReduction>
+      </actuator>
+    </transmission>
+    <transmission name="arm2_Joint_trans">
+      <type>transmission_interface/SimpleTransmission</type>
+      <joint name="arm2_Joint">
+        <hardwareInterface>hardware_interface/EffortJointInterface</hardwareInterface>
+      </joint>
+      <actuator name="arm2_Joint_motor">
+        <hardwareInterface>hardware_interface/EffortJointInterface</hardwareInterface>
+        <mechanicalReduction>1</mechanicalReduction>
+      </actuator>
+    </transmission>
+    <transmission name="arm3_Joint_trans">
+      <type>transmission_interface/SimpleTransmission</type>
+      <joint name="arm3_Joint">
+        <hardwareInterface>hardware_interface/EffortJointInterface</hardwareInterface>
+      </joint>
+      <actuator name="arm3_Joint_motor">
+        <hardwareInterface>hardware_interface/EffortJointInterface</hardwareInterface>
+        <mechanicalReduction>1</mechanicalReduction>
+      </actuator>
+    </transmission>
+    <transmission name="arm4_Joint_trans">
+      <type>transmission_interface/SimpleTransmission</type>
+      <joint name="arm4_Joint">
+        <hardwareInterface>hardware_interface/EffortJointInterface</hardwareInterface>
+      </joint>
+      <actuator name="arm4_Joint_motor">
+        <hardwareInterface>hardware_interface/EffortJointInterface</hardwareInterface>
+        <mechanicalReduction>1</mechanicalReduction>
+      </actuator>
+    </transmission>
+    <transmission name="arm5_Joint_trans">
+      <type>transmission_interface/SimpleTransmission</type>
+      <joint name="arm5_Joint">
+        <hardwareInterface>hardware_interface/EffortJointInterface</hardwareInterface>
+      </joint>
+      <actuator name="arm5_Joint_motor">
+        <hardwareInterface>hardware_interface/EffortJointInterface</hardwareInterface>
+        <mechanicalReduction>1</mechanicalReduction>
+      </actuator>
+    </transmission>
+    <transmission name="arm6_Joint_trans">
+      <type>transmission_interface/SimpleTransmission</type>
+      <joint name="arm6_Joint">
+        <hardwareInterface>hardware_interface/EffortJointInterface</hardwareInterface>
+      </joint>
+      <actuator name="arm6_Joint_motor">
+        <hardwareInterface>hardware_interface/EffortJointInterface</hardwareInterface>
+        <mechanicalReduction>1</mechanicalReduction>
+      </actuator>
+    </transmission>
+    <transmission name="gripper1_Joint_trans">
+      <type>transmission_interface/SimpleTransmission</type>
+      <joint name="gripper1_Joint">
+        <hardwareInterface>hardware_interface/EffortJointInterface</hardwareInterface>
+      </joint>
+      <actuator name="gripper1_Joint_motor">
+        <hardwareInterface>hardware_interface/EffortJointInterface</hardwareInterface>
+        <mechanicalReduction>1</mechanicalReduction>
+      </actuator>
+    </transmission>
+    <transmission name="gripper2_Joint_trans">
+      <type>transmission_interface/SimpleTransmission</type>
+      <joint name="gripper2_Joint">
+        <hardwareInterface>hardware_interface/EffortJointInterface</hardwareInterface>
+      </joint>
+      <actuator name="gripper2_Joint_motor">
+        <hardwareInterface>hardware_interface/EffortJointInterface</hardwareInterface>
+        <mechanicalReduction>1</mechanicalReduction>
+      </actuator>
+    </transmission>
   </xacro:macro>
   <!-- ==================== ROS2 Gazebo Macro ==================== -->
@@ -243,4 +323,68 @@
       </joint>
       <joint name="ankle_pitch_R_Joint">
+        <command_interface name="position" />
+        <command_interface name="velocity" />
+        <command_interface name="effort" />
+        <state_interface name="position" />
+        <state_interface name="velocity" />
+        <state_interface name="effort" />
+      </joint>
+      <joint name="arm1_Joint">
+        <command_interface name="position" />
+        <command_interface name="velocity" />
+        <command_interface name="effort" />
+        <state_interface name="position" />
+        <state_interface name="velocity" />
+        <state_interface name="effort" />
+      </joint>
+      <joint name="arm2_Joint">
+        <command_interface name="position" />
+        <command_interface name="velocity" />
+        <command_interface name="effort" />
+        <state_interface name="position" />
+        <state_interface name="velocity" />
+        <state_interface name="effort" />
+      </joint>
+      <joint name="arm3_Joint">
+        <command_interface name="position" />
+        <command_interface name="velocity" />
+        <command_interface name="effort" />
+        <state_interface name="position" />
+        <state_interface name="velocity" />
+        <state_interface name="effort" />
+      </joint>
+      <joint name="arm4_Joint">
+        <command_interface name="position" />
+        <command_interface name="velocity" />
+        <command_interface name="effort" />
+        <state_interface name="position" />
+        <state_interface name="velocity" />
+        <state_interface name="effort" />
+      </joint>
+      <joint name="arm5_Joint">
+        <command_interface name="position" />
+        <command_interface name="velocity" />
+        <command_interface name="effort" />
+        <state_interface name="position" />
+        <state_interface name="velocity" />
+        <state_interface name="effort" />
+      </joint>
+      <joint name="arm6_Joint">
+        <command_interface name="position" />
+        <command_interface name="velocity" />
+        <command_interface name="effort" />
+        <state_interface name="position" />
+        <state_interface name="velocity" />
+        <state_interface name="effort" />
+      </joint>
+      <joint name="gripper1_Joint">
+        <command_interface name="position" />
+        <command_interface name="velocity" />
+        <command_interface name="effort" />
+        <state_interface name="position" />
+        <state_interface name="velocity" />
+        <state_interface name="effort" />
+      </joint>
+      <joint name="gripper2_Joint">
         <command_interface name="position" />
         <command_interface name="velocity" />

File: tron2/SFYG_TRON2A/xacro/robot.urdf.xacro (robot description, xacro)
@@ -103,8 +103,8 @@
   <link name="proximal_yaw_L_Link">
     <inertial>
-      <origin xyz="2.76E-03 -1.64E-03 -111.48E-03" rpy="0 0 0" />
+      <origin xyz="-2.76E-03 1.64E-03 -111.48E-03" rpy="0 0 0" />
       <mass value="1.56" />
-      <inertia ixx="15039.66E-06" ixy="-3.86E-06" ixz="-266.64E-06"
-        iyy="14341.41E-06" iyz="-65.94E-06" izz="3757.85E-06" />
+      <inertia ixx="15039.66E-06" ixy="-3.86E-06" ixz="266.64E-06"
+        iyy="14341.41E-06" iyz="65.94E-06" izz="3757.85E-06" />
     </inertial>
     <visual>
@@ -124,8 +124,8 @@
   <link name="knee_L_Link">
     <inertial>
-      <origin xyz="2.17E-03 29.64E-03 -128.34E-03" rpy="0 0 0" />
+      <origin xyz="-2.17E-03 -29.64E-03 -128.34E-03" rpy="0 0 0" />
       <mass value="4.25" />
-      <inertia ixx="96150.17E-06" ixy="-37.46E-06" ixz="927.79E-06"
-        iyy="96994.26E-06" iyz="2867.36E-06" izz="5286.18E-06" />
+      <inertia ixx="96150.17E-06" ixy="-37.45E-06" ixz="-927.74E-06"
+        iyy="96994.27E-06" iyz="-2867.36E-06" izz="5286.18E-06" />
     </inertial>
     <visual>
@@ -145,8 +145,8 @@
   <link name="ankle_pitch_L_Link">
     <inertial>
-      <origin xyz="15.25E-03 -35.42E-03 -46.68E-03" rpy="0 0 0" />
+      <origin xyz="-15.25E-03 35.42E-03 -46.68E-03" rpy="0 0 0" />
       <mass value="1.02" />
-      <inertia ixx="1443.30E-06" ixy="35.45E-06" ixz="145.15E-06"
-        iyy="3461.81E-06" iyz="-68.35E-06" izz="3941.99E-06" />
+      <inertia ixx="1443.30E-06" ixy="35.45E-06" ixz="-145.15E-06"
+        iyy="3461.81E-06" iyz="68.35E-06" izz="3941.99E-06" />
     </inertial>
     <visual>
@@ -158,7 +158,67 @@
     </visual>
     <collision>
-      <origin xyz="0 0 0" rpy="0 0 0" />
-      <geometry>
-        <mesh filename="package://robot_description/tron2/SF_TRON2A/meshes/ankle_pitch_L_Link.STL" />
+      <origin rpy="0 0 0" xyz="-0.014425463037384678 0.035848761272903706 -0.05027431354942169" />
+      <geometry>
+        <box size="0.14 0.06 0.025" />
+      </geometry>
+    </collision>
+    <collision>
+      <origin rpy="0 0 0" xyz="-0.11909570195246066 0.06354314585176701 -0.07124" />
+      <geometry>
+        <sphere radius="0.0025" />
+      </geometry>
+    </collision>
+    <collision>
+      <origin rpy="0 0 0" xyz="-0.10049390971791083 0.0038735829813696387 -0.07124" />
+      <geometry>
+        <sphere radius="0.0025" />
+      </geometry>
+    </collision>
+    <collision>
+      <origin rpy="0 0 0" xyz="0.07502612984116563 0.011635070405830783 -0.07123754260807935" />
+      <geometry>
+        <sphere radius="0.0025" />
+      </geometry>
+    </collision>
+    <collision>
+      <origin rpy="0 0 0" xyz="0.07502612984116541 0.06270942031820081 -0.07124" />
+      <geometry>
+        <sphere radius="0.0025" />
+      </geometry>
+    </collision>
+    <collision>
+      <origin rpy="0 0 0" xyz="-0.08472274114731804 0.07904998982922917 -0.06424918850744032" />
+      <geometry>
+        <sphere radius="0.0025" />
+      </geometry>
+    </collision>
+    <collision>
+      <origin rpy="0 0 0" xyz="0.03564470406430653 0.07627499491461442 -0.06424918850744032" />
+      <geometry>
+        <sphere radius="0.0025" />
+      </geometry>
+    </collision>
+    <collision>
+      <origin rpy="0 0 0" xyz="-0.08472274114731826 -0.007719774188539752 -0.06424918850744032" />
+      <geometry>
+        <sphere radius="0.0025" />
+      </geometry>
+    </collision>
+    <collision>
+      <origin rpy="0 0 0" xyz="0.03564470406430653 -0.0051139227977490265 -0.06424918850744032" />
+      <geometry>
+        <sphere radius="0.0025" />
+      </geometry>
+    </collision>
+    <collision>
+      <origin rpy="0 0 0" xyz="-0.12805773805226417 0.0355 -0.06424607954803907" />
+      <geometry>
+        <sphere radius="0.0025" />
+      </geometry>
+    </collision>
+    <collision>
+      <origin rpy="0 0 0" xyz="0.08868077416023412 0.03550000000000009 -0.06424607954803907" />
+      <geometry>
+        <sphere radius="0.0025" />
       </geometry>
     </collision>
@@ -208,8 +268,8 @@
   <link name="proximal_yaw_R_Link">
     <inertial>
-      <origin xyz="0.00276 0.00164 -0.11148" rpy="0 0 0" />
+      <origin xyz="-0.00276 -0.00164 -0.11148" rpy="0 0 0" />
       <mass value="1.56" />
-      <inertia ixx="0.01503966" ixy="3.86e-06" ixz="-0.00026664"
-        iyy="0.01434141" iyz="6.594e-05" izz="0.00375785" />
+      <inertia ixx="0.01503966" ixy="3.86e-06" ixz="0.00026664"
+        iyy="0.01434141" iyz="-6.594e-05" izz="0.00375785" />
     </inertial>
     <visual>
@@ -229,8 +289,8 @@
   <link name="knee_R_Link">
     <inertial>
-      <origin xyz="0.00217 -0.02964 -0.12834" rpy="0 0 0" />
+      <origin xyz="-0.00217 0.02964 -0.12834" rpy="0 0 0" />
       <mass value="4.25" />
-      <inertia ixx="0.09615017" ixy="3.746e-05" ixz="0.00092779"
-        iyy="0.09699426" iyz="-0.00286736" izz="0.00528618" />
+      <inertia ixx="0.09615017" ixy="3.745e-05" ixz="-0.00092774"
+        iyy="0.09699427" iyz="0.00286736" izz="0.00528618" />
     </inertial>
     <visual>
@@ -248,10 +308,362 @@
     </collision>
   </link>
+  <!-- Arm + Gripper + Peripherals (piper-x) -->
+  <link name="transition_Link">
+    <inertial>
+      <origin xyz="-0.111727 0.000317 0.014516" rpy="0 0 0" />
+      <mass value="1.117" />
+      <inertia ixx="0.002739303" ixy="6.6427e-05" ixz="0.000914255"
+        iyy="0.006871988" iyz="-2.0809e-05" izz="0.007888835" />
+    </inertial>
+    <visual>
+      <origin xyz="0 0 0" rpy="0 0 0" />
+      <geometry>
+        <mesh filename="package://robot_description/tron2/SFYG_TRON2A/meshes/transition_Link.STL" />
+      </geometry>
+      <material name="white" />
+    </visual>
+    <collision>
+      <origin xyz="0 0 0" rpy="0 0 0" />
+      <geometry>
+        <mesh filename="package://robot_description/tron2/SFYG_TRON2A/meshes/transition_Link_collision.STL" />
+      </geometry>
+    </collision>
+  </link>
+  <link name="arm_base_Link">
+    <inertial>
+      <origin xyz="-0.004736412 2.5683e-05 0.041451518" rpy="0 0 0" />
+      <mass value="1.02" />
+      <inertia ixx="0.00267433" ixy="-7.3e-07" ixz="-0.00017389"
+        iyy="0.00282612" iyz="4e-07" izz="0.00089624" />
+    </inertial>
+    <visual>
+      <origin xyz="0 0 0" rpy="0 0 0" />
+      <geometry>
+        <mesh filename="package://robot_description/tron2/SFYG_TRON2A/meshes/arm_base_Link.STL" />
+      </geometry>
+      <material name="grey" />
+    </visual>
+    <collision>
+      <origin xyz="0 0 0" rpy="0 0 0" />
+      <geometry>
+        <mesh filename="package://robot_description/tron2/SFYG_TRON2A/meshes/arm_base_Link.STL" />
+      </geometry>
+    </collision>
+  </link>
+  <link name="arm1_Link">
+    <inertial>
+      <origin xyz="0.00053 -0.00039 -0.00315" rpy="0 0 0" />
+      <mass value="0.71" />
+      <inertia ixx="0.00050027" ixy="7.8e-07" ixz="6.26e-06"
+        iyy="0.00040879" iyz="4.62e-06" izz="0.00045802" />
+    </inertial>
+    <visual>
+      <origin xyz="0 0 0" rpy="0 0 0" />
+      <geometry>
+        <mesh filename="package://robot_description/tron2/SFYG_TRON2A/meshes/arm1_Link.STL" />
+      </geometry>
+      <material name="grey" />
+    </visual>
+    <collision>
+      <origin xyz="0 0 0" rpy="0 0 0" />
+      <geometry>
+        <mesh filename="package://robot_description/tron2/SFYG_TRON2A/meshes/arm1_Link.STL" />
+      </geometry>
+    </collision>
+  </link>
+  <link name="arm2_Link">
+    <inertial>
+      <origin xyz="0.21856 -0.00859 0.00227" rpy="0 0 0" />
+      <mass value="1.16" />
+      <inertia ixx="0.00111915" ixy="0.00182916" ixz="0.00019233"
+        iyy="0.06763251" iyz="7.67e-06" izz="0.067559" />
+    </inertial>
+    <visual>
+      <origin xyz="0 0 0" rpy="0 0 0" />
+      <geometry>
+        <mesh filename="package://robot_description/tron2/SFYG_TRON2A/meshes/arm2_Link.STL" />
+      </geometry>
+      <material name="grey" />
+    </visual>
+    <collision>
+      <origin xyz="0 0 0" rpy="0 0 0" />
+      <geometry>
+        <mesh filename="package://robot_description/tron2/SFYG_TRON2A/meshes/arm2_Link_collision1.STL" />
+      </geometry>
+    </collision>
+    <collision>
+      <origin xyz="0 0 0" rpy="0 0 0" />
+      <geometry>
+        <mesh filename="package://robot_description/tron2/SFYG_TRON2A/meshes/arm2_Link_collision2.STL" />
+      </geometry>
+    </collision>
+  </link>
+  <link name="arm3_Link">
+    <inertial>
+      <origin xyz="0.2014 -0.00418 -0.00141" rpy="0 0 0" />
+      <mass value="0.67" />
+      <inertia ixx="0.00033471" ixy="0.00026891" ixz="0.00013918"
+        iyy="0.03360411" iyz="5.2e-07" izz="0.03356941" />
+    </inertial>
+    <visual>
+      <origin xyz="0 0 0" rpy="0 0 0" />
+      <geometry>
+        <mesh filename="package://robot_description/tron2/SFYG_TRON2A/meshes/arm3_Link.STL" />
+      </geometry>
+      <material name="grey" />
+    </visual>
+    <collision>
+      <origin xyz="0 0 0" rpy="0 0 0" />
+      <geometry>
+        <mesh filename="package://robot_description/tron2/SFYG_TRON2A/meshes/arm3_Link_collision1.STL" />
+      </geometry>
+    </collision>
+    <collision>
+      <origin xyz="0 0 0" rpy="0 0 0" />
+      <geometry>
+        <mesh filename="package://robot_description/tron2/SFYG_TRON2A/meshes/arm3_Link_collision2.STL" />
+      </geometry>
+    </collision>
+  </link>
+  <link name="arm4_Link">
+    <inertial>
+      <origin xyz="0.059 -0.05831 0.002" rpy="0 0 0" />
+      <mass value="0.39" />
+      <inertia ixx="0.00120173" ixy="0.00138165" ixz="1.187e-05"
+        iyy="0.00209324" iyz="2.17e-06" izz="0.00307814" />
+    </inertial>
+    <visual>
+      <origin xyz="0 0 0" rpy="0 0 0" />
+      <geometry>
+        <mesh filename="package://robot_description/tron2/SFYG_TRON2A/meshes/arm4_Link.STL" />
+      </geometry>
+      <material name="grey" />
+    </visual>
+    <collision>
+      <origin xyz="0 0 0" rpy="0 0 0" />
+      <geometry>
+        <mesh filename="package://robot_description/tron2/SFYG_TRON2A/meshes/arm4_Link_collision1.STL" />
+      </geometry>
+    </collision>
+    <collision>
+      <origin xyz="0 0 0" rpy="0 0 0" />
+      <geometry>
+        <mesh filename="package://robot_description/tron2/SFYG_TRON2A/meshes/arm4_Link_collision2.STL" />
+      </geometry>
+    </collision>
+  </link>
+  <link name="arm5_Link">
+    <inertial>
+      <origin xyz="5e-05 -0.01282 -0.00429" rpy="0 0 0" />
+      <mass value="0.35" />
+      <inertia ixx="0.0002266" ixy="1.9e-07" ixz="5e-08"
+        iyy="0.0001774" iyz="8.5e-07" izz="0.00019425" />
+    </inertial>
+    <visual>
+      <origin xyz="0 0 0" rpy="0 0 0" />
+      <geometry>
+        <mesh filename="package://robot_description/tron2/SFYG_TRON2A/meshes/arm5_Link.STL" />
+      </geometry>
+      <material name="grey" />
+    </visual>
+    <collision>
+      <origin xyz="0 0 0" rpy="0 0 0" />
+      <geometry>
+        <mesh filename="package://robot_description/tron2/SFYG_TRON2A/meshes/arm5_Link.STL" />
+      </geometry>
+    </collision>
+  </link>
+  <link name="arm6_Link">
+    <inertial>
+      <origin xyz="0.0 0.0 -0.0035" rpy="0 0 0" />
+      <mass value="0.007" />
+      <inertia ixx="0.00152112" ixy="2.02e-06" ixz="2.61e-06"
+        iyy="0.00138626" iyz="2e-08" izz="0.00031152" />
+    </inertial>
+    <visual>
+      <origin xyz="0 0 0" rpy="0 0 0" />
+      <geometry>
+        <mesh filename="package://robot_description/tron2/SFYG_TRON2A/meshes/arm6_Link.STL" />
+      </geometry>
+      <material name="grey" />
+    </visual>
+    <collision>
+      <origin xyz="0 0 0" rpy="0 0 0" />
+      <geometry>
+        <mesh filename="package://robot_description/tron2/SFYG_TRON2A/meshes/arm6_Link.STL" />
+      </geometry>
+    </collision>
+  </link>
+  <link name="gripper_base_Link">
+    <inertial>
+      <origin xyz="-0.000183807 8.0503e-05 0.032143669" rpy="0 0 0" />
+      <mass value="0.45" />
+      <inertia ixx="0.00092934" ixy="3.4e-07" ixz="-7.38e-06"
+        iyy="0.00071447" iyz="5e-08" izz="0.00039442" />
+    </inertial>
+    <visual>
+      <origin xyz="0 0 0" rpy="0 0 0" />
+      <geometry>
+        <mesh filename="package://robot_description/tron2/SFYG_TRON2A/meshes/gripper_base_Link.STL" />
+      </geometry>
+      <material name="grey" />
+    </visual>
+    <collision>
+      <origin xyz="0 0 0" rpy="0 0 0" />
+      <geometry>
+        <mesh filename="package://robot_description/tron2/SFYG_TRON2A/meshes/gripper_base_Link_collision1.STL" />
+      </geometry>
+    </collision>
+    <collision>
+      <origin xyz="0 0 0" rpy="0 0 0" />
+      <geometry>
+        <mesh filename="package://robot_description/tron2/SFYG_TRON2A/meshes/gripper_base_Link_collision2.STL" />
+      </geometry>
+    </collision>
+  </link>
+  <link name="gripper1_Link">
+    <inertial>
+      <origin xyz="0.000651232 -0.049192987 0.009722588" rpy="0 0 0" />
+      <mass value="0.025" />
+      <inertia ixx="7.371e-05" ixy="-1.13e-06" ixz="2.1e-07"
+        iyy="7.81e-06" iyz="-1.372e-05" izz="7.47e-05" />
+    </inertial>
+    <visual>
+      <origin xyz="0 0 0" rpy="0 0 0" />
+      <geometry>
+        <mesh filename="package://robot_description/tron2/SFYG_TRON2A/meshes/gripper1_Link.STL" />
+      </geometry>
+      <material name="grey" />
+    </visual>
+    <collision>
+      <origin xyz="0 0 0" rpy="0 0 0" />
+      <geometry>
+        <mesh filename="package://robot_description/tron2/SFYG_TRON2A/meshes/gripper1_Link.STL" />
+      </geometry>
+    </collision>
+  </link>
+  <link name="gripper2_Link">
+    <inertial>
+      <origin xyz="0.000651232 -0.049192987 0.009722588" rpy="0 0 0" />
+      <mass value="0.025" />
+      <inertia ixx="7.371e-05" ixy="-1.13e-06" ixz="2.1e-07"
+        iyy="7.81e-06" iyz="-1.372e-05" izz="7.47e-05" />
+    </inertial>
+    <visual>
+      <origin xyz="0 0 0" rpy="0 0 0" />
+      <geometry>
+        <mesh filename="package://robot_description/tron2/SFYG_TRON2A/meshes/gripper2_Link.STL" />
+      </geometry>
+      <material name="grey" />
+    </visual>
+    <collision>
+      <origin xyz="0 0 0" rpy="0 0 0" />
+      <geometry>
+        <mesh filename="package://robot_description/tron2/SFYG_TRON2A/meshes/gripper2_Link.STL" />
+      </geometry>
+    </collision>
+  </link>
+  <link name="antenna_L_Link">
+    <inertial>
+      <origin xyz="-2.7e-05 -0.028426 0.013784" rpy="0 0 0" />
+      <mass value="0.231" />
+      <inertia ixx="0.000424493" ixy="-1.15e-07" ixz="-1.18e-07"
+        iyy="0.000169977" iyz="3.0807e-05" izz="0.00039175" />
+    </inertial>
+    <visual>
+      <origin xyz="0 0 0" rpy="0 0 0" />
+      <geometry>
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