Commit message: refactor: rename limx_imu to base_imu across SF/SFYG/WF/WFYG xacros
Update the IMU link, joint, gazebo references, and ros2_control sensor
name uniformly across the four configurations. Each robot.urdf.xacro
gets the link/joint/gazebo joint reference renamed (and the d435_joint
parent for SF/SFYG); each macros.xacro gets the ros2_control sensor
name and the gazebo IMU sensor block renamed.

Tron2HWSim resolves the IMU by sensor name, so renaming the
ros2_control entry together with the gazebo <sensor name> keeps the
binding intact.

Note: urdf/robot.urdf and tron2/*/xml/robot.xml still carry the
limx_imu name; consumers loading those directly (instead of expanding
the xacro) keep the old TF frame.

Co-Authored-By: Claude Opus 4.7 (1M context) <noreply@anthropic.com>

File: tron2/SFYG_TRON2A/xacro/macros.xacro (robot description, xacro)
@@ -394,5 +394,5 @@
         <state_interface name="effort" />
       </joint>
-      <sensor name="limx_imu_sensor">
+      <sensor name="base_imu_sensor">
         <state_interface name="orientation.x" />
         <state_interface name="orientation.y" />
@@ -408,6 +408,6 @@
     </ros2_control>
     <!-- IMU Gazebo sensor plugin (ROS2) -->
-    <gazebo reference="limx_imu">
-      <sensor type="imu" name="limx_imu_sensor">
+    <gazebo reference="base_imu">
+      <sensor type="imu" name="base_imu_sensor">
         <always_on>true</always_on>
         <update_rate>100</update_rate>

File: tron2/SFYG_TRON2A/xacro/robot.urdf.xacro (robot description, xacro)
@@ -15,10 +15,10 @@
   </material>
   <!-- IMU Link -->
-  <joint name="limx_imu_joint" type="fixed">
+  <joint name="base_imu_joint" type="fixed">
     <origin rpy="0. 0. 0." xyz="0. 0. 0." />
     <parent link="base_Link" />
-    <child link="limx_imu" />
-  </joint>
-  <link name="limx_imu">
+    <child link="base_imu" />
+  </joint>
+  <link name="base_imu">
     <inertial>
       <mass value="0.01" />
@@ -34,5 +34,5 @@
     </visual>
   </link>
-  <gazebo reference="limx_imu_joint">
+  <gazebo reference="base_imu_joint">
     <disableFixedJointLumping>true</disableFixedJointLumping>
   </gazebo>
@@ -755,5 +755,5 @@
   <joint name="d435_joint" type="fixed">
     <origin rpy="0 1.063778179 0" xyz="0.12213 0.01759 0.00599" />
-    <parent link="limx_imu" />
+    <parent link="base_imu" />
     <child link="d435_Link" />
   </joint>

File: tron2/SF_TRON2A/xacro/macros.xacro (robot description, xacro)
@@ -250,5 +250,5 @@
         <state_interface name="effort" />
       </joint>
-      <sensor name="limx_imu_sensor">
+      <sensor name="base_imu_sensor">
         <state_interface name="orientation.x" />
         <state_interface name="orientation.y" />
@@ -264,6 +264,6 @@
     </ros2_control>
     <!-- IMU Gazebo sensor plugin (ROS2) -->
-    <gazebo reference="limx_imu">
-      <sensor type="imu" name="limx_imu_sensor">
+    <gazebo reference="base_imu">
+      <sensor type="imu" name="base_imu_sensor">
         <always_on>true</always_on>
         <update_rate>100</update_rate>

File: tron2/SF_TRON2A/xacro/robot.urdf.xacro (robot description, xacro)
@@ -15,10 +15,10 @@
   </material>
   <!-- IMU Link -->
-  <joint name="limx_imu_joint" type="fixed">
+  <joint name="base_imu_joint" type="fixed">
     <origin rpy="0. 0. 0." xyz="0. 0. 0." />
     <parent link="base_Link" />
-    <child link="limx_imu" />
-  </joint>
-  <link name="limx_imu">
+    <child link="base_imu" />
+  </joint>
+  <link name="base_imu">
     <inertial>
       <mass value="0.01" />
@@ -34,5 +34,5 @@
     </visual>
   </link>
-  <gazebo reference="limx_imu_joint">
+  <gazebo reference="base_imu_joint">
     <disableFixedJointLumping>true</disableFixedJointLumping>
   </gazebo>
@@ -283,5 +283,5 @@
   <joint name="d435_joint" type="fixed">
     <origin rpy="0 1.063778179 0" xyz="0.12213 0.01759 0.00599" />
-    <parent link="limx_imu" />
+    <parent link="base_imu" />
     <child link="d435_Link" />
   </joint>

File: tron2/WFYG_TRON2A/xacro/macros.xacro (robot description, xacro)
@@ -236,5 +236,5 @@
         <state_interface name="effort" />
       </joint>
-      <sensor name="limx_imu_sensor">
+      <sensor name="base_imu_sensor">
         <state_interface name="orientation.x" />
         <state_interface name="orientation.y" />
@@ -250,6 +250,6 @@
     </ros2_control>
     <!-- IMU Gazebo sensor plugin (ROS2) -->
-    <gazebo reference="limx_imu">
-      <sensor type="imu" name="limx_imu_sensor">
+    <gazebo reference="base_imu">
+      <sensor type="imu" name="base_imu_sensor">
         <always_on>true</always_on>
         <update_rate>100</update_rate>

File: tron2/WFYG_TRON2A/xacro/robot.urdf.xacro (robot description, xacro)
@@ -17,10 +17,10 @@
   </material>
   <!-- IMU Link -->
-  <joint name="limx_imu_joint" type="fixed">
+  <joint name="base_imu_joint" type="fixed">
     <origin rpy="0. 0. 0." xyz="0. 0. 0." />
     <parent link="base_Link" />
-    <child link="limx_imu" />
-  </joint>
-  <link name="limx_imu">
+    <child link="base_imu" />
+  </joint>
+  <link name="base_imu">
     <inertial>
       <mass value="0.01" />
@@ -36,5 +36,5 @@
     </visual>
   </link>
-  <gazebo reference="limx_imu_joint">
+  <gazebo reference="base_imu_joint">
     <disableFixedJointLumping>true</disableFixedJointLumping>
   </gazebo>
