Commit message: feat(WFYG_TRON2A): align legs to URDF and re-point meshes to WFYG_TRON2A
The WFYG xacro was forked from WF and never re-tuned. Bring the legs
in line with WFYG/urdf/robot.urdf:

- Joint effort: 150 -> 200 for proximal_pitch/roll/knee, 60 -> 70 for
  proximal_yaw, matching the WFYG hardware (WF kept its sim2real-tuned
  150/60).
- proximal_roll limits: +/-3.19395248 -> +/-3.2288591161895095.
- wheel limit precision: 1745329.2519943293 -> 1745329.2519943295.
- proximal_pitch axis lifted to URDF full precision.
- Re-point all 56 leg/wheel mesh references from tron2/WF_TRON2A/meshes
  to tron2/WFYG_TRON2A/meshes (the meshes already live there).

Co-Authored-By: Claude Opus 4.7 (1M context) <noreply@anthropic.com>

File: tron2/WFYG_TRON2A/xacro/robot.urdf.xacro (robot description, xacro)
@@ -50,10 +50,10 @@
       <origin xyz="0 0 0" rpy="0 0 0" />
       <geometry>
-        <mesh filename="package://robot_description/tron2/WF_TRON2A/meshes/base_Link.STL" />
-      </geometry>
-      <material name="grey" />
-    </visual>
-    <xacro:unless value="${use_primitive}">
-      <xacro:collision_mesh mesh_filename="package://robot_description/tron2/WF_TRON2A/meshes/base_Link.STL" />
+        <mesh filename="package://robot_description/tron2/WFYG_TRON2A/meshes/base_Link.STL" />
+      </geometry>
+      <material name="grey" />
+    </visual>
+    <xacro:unless value="${use_primitive}">
+      <xacro:collision_mesh mesh_filename="package://robot_description/tron2/WFYG_TRON2A/meshes/base_Link.STL" />
     </xacro:unless>
     <xacro:if value="${use_primitive}">
@@ -74,10 +74,10 @@
       <origin xyz="0 0 0" rpy="0 0 0" />
       <geometry>
-        <mesh filename="package://robot_description/tron2/WF_TRON2A/meshes/proximal_pitch_L_Link.STL" />
-      </geometry>
-      <material name="grey" />
-    </visual>
-    <xacro:unless value="${use_primitive}">
-      <xacro:collision_mesh mesh_filename="package://robot_description/tron2/WF_TRON2A/meshes/proximal_pitch_L_Link.STL" />
+        <mesh filename="package://robot_description/tron2/WFYG_TRON2A/meshes/proximal_pitch_L_Link.STL" />
+      </geometry>
+      <material name="grey" />
+    </visual>
+    <xacro:unless value="${use_primitive}">
+      <xacro:collision_mesh mesh_filename="package://robot_description/tron2/WFYG_TRON2A/meshes/proximal_pitch_L_Link.STL" />
     </xacro:unless>
     <xacro:if value="${use_primitive}">
@@ -98,10 +98,10 @@
       <origin xyz="0 0 0" rpy="0 0 0" />
       <geometry>
-        <mesh filename="package://robot_description/tron2/WF_TRON2A/meshes/proximal_roll_L_Link.STL" />
-      </geometry>
-      <material name="grey" />
-    </visual>
-    <xacro:unless value="${use_primitive}">
-      <xacro:collision_mesh mesh_filename="package://robot_description/tron2/WF_TRON2A/meshes/proximal_roll_L_Link.STL" />
+        <mesh filename="package://robot_description/tron2/WFYG_TRON2A/meshes/proximal_roll_L_Link.STL" />
+      </geometry>
+      <material name="grey" />
+    </visual>
+    <xacro:unless value="${use_primitive}">
+      <xacro:collision_mesh mesh_filename="package://robot_description/tron2/WFYG_TRON2A/meshes/proximal_roll_L_Link.STL" />
     </xacro:unless>
     <xacro:if value="${use_primitive}">
@@ -122,10 +122,10 @@
       <origin xyz="0 0 0" rpy="0 0 0" />
       <geometry>
-        <mesh filename="package://robot_description/tron2/WF_TRON2A/meshes/proximal_yaw_L_Link.STL" />
-      </geometry>
-      <material name="grey" />
-    </visual>
-    <xacro:unless value="${use_primitive}">
-      <xacro:collision_mesh mesh_filename="package://robot_description/tron2/WF_TRON2A/meshes/proximal_yaw_L_Link.STL" />
+        <mesh filename="package://robot_description/tron2/WFYG_TRON2A/meshes/proximal_yaw_L_Link.STL" />
+      </geometry>
+      <material name="grey" />
+    </visual>
+    <xacro:unless value="${use_primitive}">
+      <xacro:collision_mesh mesh_filename="package://robot_description/tron2/WFYG_TRON2A/meshes/proximal_yaw_L_Link.STL" />
     </xacro:unless>
     <xacro:if value="${use_primitive}">
@@ -146,10 +146,10 @@
       <origin xyz="0 0 0" rpy="0 0 0" />
       <geometry>
-        <mesh filename="package://robot_description/tron2/WF_TRON2A/meshes/knee_L_Link.STL" />
-      </geometry>
-      <material name="grey" />
-    </visual>
-    <xacro:unless value="${use_primitive}">
-      <xacro:collision_mesh mesh_filename="package://robot_description/tron2/WF_TRON2A/meshes/knee_L_Link.STL" />
+        <mesh filename="package://robot_description/tron2/WFYG_TRON2A/meshes/knee_L_Link.STL" />
+      </geometry>
+      <material name="grey" />
+    </visual>
+    <xacro:unless value="${use_primitive}">
+      <xacro:collision_mesh mesh_filename="package://robot_description/tron2/WFYG_TRON2A/meshes/knee_L_Link.STL" />
     </xacro:unless>
     <xacro:if value="${use_primitive}">
@@ -170,5 +170,5 @@
       <origin xyz="0 0 0" rpy="0 0 0" />
       <geometry>
-        <mesh filename="package://robot_description/tron2/WF_TRON2A/meshes/wheel_L_Link.STL" />
+        <mesh filename="package://robot_description/tron2/WFYG_TRON2A/meshes/wheel_L_Link.STL" />
       </geometry>
       <material name="grey" />
@@ -191,10 +191,10 @@
       <origin xyz="0 0 0" rpy="0 0 0" />
       <geometry>
-        <mesh filename="package://robot_description/tron2/WF_TRON2A/meshes/proximal_pitch_R_Link.STL" />
-      </geometry>
-      <material name="grey" />
-    </visual>
-    <xacro:unless value="${use_primitive}">
-      <xacro:collision_mesh mesh_filename="package://robot_description/tron2/WF_TRON2A/meshes/proximal_pitch_R_Link.STL" />
+        <mesh filename="package://robot_description/tron2/WFYG_TRON2A/meshes/proximal_pitch_R_Link.STL" />
+      </geometry>
+      <material name="grey" />
+    </visual>
+    <xacro:unless value="${use_primitive}">
+      <xacro:collision_mesh mesh_filename="package://robot_description/tron2/WFYG_TRON2A/meshes/proximal_pitch_R_Link.STL" />
     </xacro:unless>
     <xacro:if value="${use_primitive}">
@@ -215,10 +215,10 @@
       <origin xyz="0 0 0" rpy="0 0 0" />
       <geometry>
-        <mesh filename="package://robot_description/tron2/WF_TRON2A/meshes/proximal_roll_R_Link.STL" />
-      </geometry>
-      <material name="grey" />
-    </visual>
-    <xacro:unless value="${use_primitive}">
-      <xacro:collision_mesh mesh_filename="package://robot_description/tron2/WF_TRON2A/meshes/proximal_roll_R_Link.STL" />
+        <mesh filename="package://robot_description/tron2/WFYG_TRON2A/meshes/proximal_roll_R_Link.STL" />
+      </geometry>
+      <material name="grey" />
+    </visual>
+    <xacro:unless value="${use_primitive}">
+      <xacro:collision_mesh mesh_filename="package://robot_description/tron2/WFYG_TRON2A/meshes/proximal_roll_R_Link.STL" />
     </xacro:unless>
     <xacro:if value="${use_primitive}">
@@ -239,10 +239,10 @@
       <origin xyz="0 0 0" rpy="0 0 0" />
       <geometry>
-        <mesh filename="package://robot_description/tron2/WF_TRON2A/meshes/proximal_yaw_R_Link.STL" />
-      </geometry>
-      <material name="grey" />
-    </visual>
-    <xacro:unless value="${use_primitive}">
-      <xacro:collision_mesh mesh_filename="package://robot_description/tron2/WF_TRON2A/meshes/proximal_yaw_R_Link.STL" />
+        <mesh filename="package://robot_description/tron2/WFYG_TRON2A/meshes/proximal_yaw_R_Link.STL" />
+      </geometry>
+      <material name="grey" />
+    </visual>
+    <xacro:unless value="${use_primitive}">
+      <xacro:collision_mesh mesh_filename="package://robot_description/tron2/WFYG_TRON2A/meshes/proximal_yaw_R_Link.STL" />
     </xacro:unless>
     <xacro:if value="${use_primitive}">
@@ -263,10 +263,10 @@
       <origin xyz="0 0 0" rpy="0 0 0" />
       <geometry>
-        <mesh filename="package://robot_description/tron2/WF_TRON2A/meshes/knee_R_Link.STL" />
-      </geometry>
-      <material name="grey" />
-    </visual>
-    <xacro:unless value="${use_primitive}">
-      <xacro:collision_mesh mesh_filename="package://robot_description/tron2/WF_TRON2A/meshes/knee_R_Link.STL" />
+        <mesh filename="package://robot_description/tron2/WFYG_TRON2A/meshes/knee_R_Link.STL" />
+      </geometry>
+      <material name="grey" />
+    </visual>
+    <xacro:unless value="${use_primitive}">
+      <xacro:collision_mesh mesh_filename="package://robot_description/tron2/WFYG_TRON2A/meshes/knee_R_Link.STL" />
     </xacro:unless>
     <xacro:if value="${use_primitive}">
@@ -287,5 +287,5 @@
       <origin xyz="0 0 0" rpy="0 0 0" />
       <geometry>
-        <mesh filename="package://robot_description/tron2/WF_TRON2A/meshes/wheel_R_Link.STL" />
+        <mesh filename="package://robot_description/tron2/WFYG_TRON2A/meshes/wheel_R_Link.STL" />
       </geometry>
       <material name="grey" />
@@ -303,6 +303,6 @@
     <parent link="base_Link" />
     <child link="proximal_pitch_L_Link" />
-    <axis xyz="0 0.99619 -0.087155" />
-    <limit lower="-3.141592653589793" upper="2.600540585471551" effort="150" velocity="18.3" />
+    <axis xyz="0.0 0.996194726892931 -0.0871554135479712" />
+    <limit lower="-3.141592653589793" upper="2.600540585471551" effort="200" velocity="18.3" />
   </joint>
   <joint name="proximal_roll_L_Joint" type="revolute">
@@ -311,5 +311,5 @@
     <child link="proximal_roll_L_Link" />
     <axis xyz="1 0 0" />
-    <limit lower="-0.2617993877991494" upper="3.19395248" effort="150" velocity="18.3" />
+    <limit lower="-0.2617993877991494" upper="3.2288591161895095" effort="200" velocity="18.3" />
   </joint>
   <joint name="proximal_yaw_L_Joint" type="revolute">
@@ -318,5 +318,5 @@
     <child link="proximal_yaw_L_Link" />
     <axis xyz="0 0 1" />
-    <limit lower="-3.6651914291880923" upper="1.4835298641951802" effort="60" velocity="22.52" />
+    <limit lower="-3.6651914291880923" upper="1.4835298641951802" effort="70" velocity="22.52" />
   </joint>
   <joint name="knee_L_Joint" type="revolute">
@@ -325,5 +325,5 @@
     <child link="knee_L_Link" />
     <axis xyz="0 1 0" />
-    <limit lower="-2.6179938779914944" upper="0.2617993877991494" effort="150" velocity="18.3" />
+    <limit lower="-2.6179938779914944" upper="0.2617993877991494" effort="200" velocity="18.3" />
   </joint>
   <joint name="wheel_L_Joint" type="revolute">
@@ -332,5 +332,5 @@
     <child link="wheel_L_Link" />
     <axis xyz="0 1 0" />
-    <limit lower="-1745329.2519943293" upper="1745329.2519943293" effort="22" velocity="41.89" />
+    <limit lower="-1745329.2519943295" upper="1745329.2519943295" effort="22" velocity="41.89" />
   </joint>
   <joint name="proximal_pitch_R_Joint" type="revolute">
@@ -338,6 +338,6 @@
     <parent link="base_Link" />
     <child link="proximal_pitch_R_Link" />
-    <axis xyz="0 0.99619 0.087155" />
-    <limit lower="-3.141592653589793" upper="2.600540585471551" effort="150" velocity="18.3" />
+    <axis xyz="-0.0 0.996194726892931 0.0871554135479712" />
+    <limit lower="-3.141592653589793" upper="2.600540585471551" effort="200" velocity="18.3" />
   </joint>
   <joint name="proximal_roll_R_Joint" type="revolute">
@@ -346,5 +346,5 @@
     <child link="proximal_roll_R_Link" />
     <axis xyz="1 0 0" />
-    <limit lower="-3.19395248" upper="0.2617993877991494" effort="150" velocity="18.3" />
+    <limit lower="-3.2288591161895095" upper="0.2617993877991494" effort="200" velocity="18.3" />
   </joint>
   <joint name="proximal_yaw_R_Joint" type="revolute">
@@ -353,5 +353,5 @@
     <child link="proximal_yaw_R_Link" />
     <axis xyz="0 0 1" />
-    <limit lower="-1.4835298641951802" upper="3.6651914291880923" effort="60" velocity="22.52" />
+    <limit lower="-1.4835298641951802" upper="3.6651914291880923" effort="70" velocity="22.52" />
   </joint>
   <joint name="knee_R_Joint" type="revolute">
@@ -360,5 +360,5 @@
     <child link="knee_R_Link" />
     <axis xyz="0 1 0" />
-    <limit lower="-2.6179938779914944" upper="0.2617993877991494" effort="150" velocity="18.3" />
+    <limit lower="-2.6179938779914944" upper="0.2617993877991494" effort="200" velocity="18.3" />
   </joint>
   <joint name="wheel_R_Joint" type="revolute">
@@ -367,5 +367,5 @@
     <child link="wheel_R_Link" />
     <axis xyz="0 1 0" />
-    <limit lower="-1745329.2519943293" upper="1745329.2519943293" effort="22" velocity="41.89" />
+    <limit lower="-1745329.2519943295" upper="1745329.2519943295" effort="22" velocity="41.89" />
   </joint>
   <!-- Gazebo Material / Friction (shared) -->
