Commit message: feat(WFYG_TRON2A): add piper-x arm, gripper, peripherals, d435
Bring the WFYG xacro up to the piper-x URDF (commit ccd9239). The
URDF added a 6-DOF arm linked to a gripper, plus antennas, a camera
mount, and a radar block; the xacro was still a copy of WF.

robot.urdf.xacro:
- Add transition, arm_base, arm1..arm6, gripper_base, gripper1/2,
  antenna_L/R, camera_mount, radar links and joints.
- Add d435_Link, d435_optical_frame, and the d435 fixed joints
  (parent base_imu).
- Add gazebo friction/material blocks for every new link.

macros.xacro:
- ROS1: add transmissions for arm1..arm6 and gripper1/2; add the
  D435 ROS1 plugin (split into camera + depth_camera sensors per the
  same fix applied to SF/SFYG, which avoids the openni_kinect /
  gazebo_ros_control deadlock).
- ROS2: add the eight matching ros2_control joint blocks and the
  D435 ROS2 plugin (libgazebo_ros_camera.so).

Co-Authored-By: Claude Opus 4.7 (1M context) <noreply@anthropic.com>

File: tron2/WFYG_TRON2A/xacro/robot.urdf.xacro (robot description, xacro)
@@ -298,4 +298,379 @@
     </collision>
   </link>
+  <!-- Arm + Gripper + Peripherals (piper-x) -->
+  <link name="transition_Link">
+    <inertial>
+      <origin xyz="-0.111727 0.000317 0.014516" rpy="0 0 0" />
+      <mass value="1.117" />
+      <inertia ixx="0.002739303" ixy="6.6427e-05" ixz="0.000914255"
+        iyy="0.006871988" iyz="-2.0809e-05" izz="0.007888835" />
+    </inertial>
+    <visual>
+      <origin xyz="0 0 0" rpy="0 0 0" />
+      <geometry>
+        <mesh filename="package://robot_description/tron2/WFYG_TRON2A/meshes/transition_Link.STL" />
+      </geometry>
+      <material name="white" />
+    </visual>
+    <collision>
+      <origin xyz="0 0 0" rpy="0 0 0" />
+      <geometry>
+        <mesh filename="package://robot_description/tron2/WFYG_TRON2A/meshes/transition_Link_collision.STL" />
+      </geometry>
+    </collision>
+  </link>
+  <link name="arm_base_Link">
+    <inertial>
+      <origin xyz="-0.004736412 2.5683e-05 0.041451518" rpy="0 0 0" />
+      <mass value="1.02" />
+      <inertia ixx="0.00267433" ixy="-7.3e-07" ixz="-0.00017389"
+        iyy="0.00282612" iyz="4e-07" izz="0.00089624" />
+    </inertial>
+    <visual>
+      <origin xyz="0 0 0" rpy="0 0 0" />
+      <geometry>
+        <mesh filename="package://robot_description/tron2/WFYG_TRON2A/meshes/arm_base_Link.STL" />
+      </geometry>
+      <material name="grey" />
+    </visual>
+    <collision>
+      <origin xyz="0 0 0" rpy="0 0 0" />
+      <geometry>
+        <mesh filename="package://robot_description/tron2/WFYG_TRON2A/meshes/arm_base_Link.STL" />
+      </geometry>
+    </collision>
+  </link>
+  <link name="arm1_Link">
+    <inertial>
+      <origin xyz="0.00053 -0.00039 -0.00315" rpy="0 0 0" />
+      <mass value="0.71" />
+      <inertia ixx="0.00050027" ixy="7.8e-07" ixz="6.26e-06"
+        iyy="0.00040879" iyz="4.62e-06" izz="0.00045802" />
+    </inertial>
+    <visual>
+      <origin xyz="0 0 0" rpy="0 0 0" />
+      <geometry>
+        <mesh filename="package://robot_description/tron2/WFYG_TRON2A/meshes/arm1_Link.STL" />
+      </geometry>
+      <material name="grey" />
+    </visual>
+    <collision>
+      <origin xyz="0 0 0" rpy="0 0 0" />
+      <geometry>
+        <mesh filename="package://robot_description/tron2/WFYG_TRON2A/meshes/arm1_Link.STL" />
+      </geometry>
+    </collision>
+  </link>
+  <link name="arm2_Link">
+    <inertial>
+      <origin xyz="0.21856 -0.00859 0.00227" rpy="0 0 0" />
+      <mass value="1.16" />
+      <inertia ixx="0.00111915" ixy="0.00182916" ixz="0.00019233"
+        iyy="0.06763251" iyz="7.67e-06" izz="0.067559" />
+    </inertial>
+    <visual>
+      <origin xyz="0 0 0" rpy="0 0 0" />
+      <geometry>
+        <mesh filename="package://robot_description/tron2/WFYG_TRON2A/meshes/arm2_Link.STL" />
+      </geometry>
+      <material name="grey" />
+    </visual>
+    <collision>
+      <origin xyz="0 0 0" rpy="0 0 0" />
+      <geometry>
+        <mesh filename="package://robot_description/tron2/WFYG_TRON2A/meshes/arm2_Link_collision1.STL" />
+      </geometry>
+    </collision>
+    <collision>
+      <origin xyz="0 0 0" rpy="0 0 0" />
+      <geometry>
+        <mesh filename="package://robot_description/tron2/WFYG_TRON2A/meshes/arm2_Link_collision2.STL" />
+      </geometry>
+    </collision>
+  </link>
+  <link name="arm3_Link">
+    <inertial>
+      <origin xyz="0.2014 -0.00418 -0.00141" rpy="0 0 0" />
+      <mass value="0.67" />
+      <inertia ixx="0.00033471" ixy="0.00026891" ixz="0.00013918"
+        iyy="0.03360411" iyz="5.2e-07" izz="0.03356941" />
+    </inertial>
+    <visual>
+      <origin xyz="0 0 0" rpy="0 0 0" />
+      <geometry>
+        <mesh filename="package://robot_description/tron2/WFYG_TRON2A/meshes/arm3_Link.STL" />
+      </geometry>
+      <material name="grey" />
+    </visual>
+    <collision>
+      <origin xyz="0 0 0" rpy="0 0 0" />
+      <geometry>
+        <mesh filename="package://robot_description/tron2/WFYG_TRON2A/meshes/arm3_Link_collision1.STL" />
+      </geometry>
+    </collision>
+    <collision>
+      <origin xyz="0 0 0" rpy="0 0 0" />
+      <geometry>
+        <mesh filename="package://robot_description/tron2/WFYG_TRON2A/meshes/arm3_Link_collision2.STL" />
+      </geometry>
+    </collision>
+  </link>
+  <link name="arm4_Link">
+    <inertial>
+      <origin xyz="0.059 -0.05831 0.002" rpy="0 0 0" />
+      <mass value="0.39" />
+      <inertia ixx="0.00120173" ixy="0.00138165" ixz="1.187e-05"
+        iyy="0.00209324" iyz="2.17e-06" izz="0.00307814" />
+    </inertial>
+    <visual>
+      <origin xyz="0 0 0" rpy="0 0 0" />
+      <geometry>
+        <mesh filename="package://robot_description/tron2/WFYG_TRON2A/meshes/arm4_Link.STL" />
+      </geometry>
+      <material name="grey" />
+    </visual>
+    <collision>
+      <origin xyz="0 0 0" rpy="0 0 0" />
+      <geometry>
+        <mesh filename="package://robot_description/tron2/WFYG_TRON2A/meshes/arm4_Link_collision1.STL" />
+      </geometry>
+    </collision>
+    <collision>
+      <origin xyz="0 0 0" rpy="0 0 0" />
+      <geometry>
+        <mesh filename="package://robot_description/tron2/WFYG_TRON2A/meshes/arm4_Link_collision2.STL" />
+      </geometry>
+    </collision>
+  </link>
+  <link name="arm5_Link">
+    <inertial>
+      <origin xyz="5e-05 -0.01282 -0.00429" rpy="0 0 0" />
+      <mass value="0.35" />
+      <inertia ixx="0.0002266" ixy="1.9e-07" ixz="5e-08"
+        iyy="0.0001774" iyz="8.5e-07" izz="0.00019425" />
+    </inertial>
+    <visual>
+      <origin xyz="0 0 0" rpy="0 0 0" />
+      <geometry>
+        <mesh filename="package://robot_description/tron2/WFYG_TRON2A/meshes/arm5_Link.STL" />
+      </geometry>
+      <material name="grey" />
+    </visual>
+    <collision>
+      <origin xyz="0 0 0" rpy="0 0 0" />
+      <geometry>
+        <mesh filename="package://robot_description/tron2/WFYG_TRON2A/meshes/arm5_Link.STL" />
+      </geometry>
+    </collision>
+  </link>
+  <link name="arm6_Link">
+    <inertial>
+      <origin xyz="0.0 0.0 -0.0035" rpy="0 0 0" />
+      <mass value="0.007" />
+      <inertia ixx="0.00152112" ixy="2.02e-06" ixz="2.61e-06"
+        iyy="0.00138626" iyz="2e-08" izz="0.00031152" />
+    </inertial>
+    <visual>
+      <origin xyz="0 0 0" rpy="0 0 0" />
+      <geometry>
+        <mesh filename="package://robot_description/tron2/WFYG_TRON2A/meshes/arm6_Link.STL" />
+      </geometry>
+      <material name="grey" />
+    </visual>
+    <collision>
+      <origin xyz="0 0 0" rpy="0 0 0" />
+      <geometry>
+        <mesh filename="package://robot_description/tron2/WFYG_TRON2A/meshes/arm6_Link.STL" />
+      </geometry>
+    </collision>
+  </link>
+  <link name="gripper_base_Link">
+    <inertial>
+      <origin xyz="-0.000183807 8.0503e-05 0.032143669" rpy="0 0 0" />
+      <mass value="0.45" />
+      <inertia ixx="0.00092934" ixy="3.4e-07" ixz="-7.38e-06"
+        iyy="0.00071447" iyz="5e-08" izz="0.00039442" />
+    </inertial>
+    <visual>
+      <origin xyz="0 0 0" rpy="0 0 0" />
+      <geometry>
+        <mesh filename="package://robot_description/tron2/WFYG_TRON2A/meshes/gripper_base_Link.STL" />
+      </geometry>
+      <material name="grey" />
+    </visual>
+    <collision>
+      <origin xyz="0 0 0" rpy="0 0 0" />
+      <geometry>
+        <mesh filename="package://robot_description/tron2/WFYG_TRON2A/meshes/gripper_base_Link_collision1.STL" />
+      </geometry>
+    </collision>
+    <collision>
+      <origin xyz="0 0 0" rpy="0 0 0" />
+      <geometry>
+        <mesh filename="package://robot_description/tron2/WFYG_TRON2A/meshes/gripper_base_Link_collision2.STL" />
+      </geometry>
+    </collision>
+  </link>
+  <link name="gripper1_Link">
+    <inertial>
+      <origin xyz="0.000651232 -0.049192987 0.009722588" rpy="0 0 0" />
+      <mass value="0.025" />
+      <inertia ixx="7.371e-05" ixy="-1.13e-06" ixz="2.1e-07"
+        iyy="7.81e-06" iyz="-1.372e-05" izz="7.47e-05" />
+    </inertial>
+    <visual>
+      <origin xyz="0 0 0" rpy="0 0 0" />
+      <geometry>
+        <mesh filename="package://robot_description/tron2/WFYG_TRON2A/meshes/gripper1_Link.STL" />
+      </geometry>
+      <material name="grey" />
+    </visual>
+    <collision>
+      <origin xyz="0 0 0" rpy="0 0 0" />
+      <geometry>
+        <mesh filename="package://robot_description/tron2/WFYG_TRON2A/meshes/gripper1_Link.STL" />
+      </geometry>
+    </collision>
+  </link>
+  <link name="gripper2_Link">
+    <inertial>
+      <origin xyz="0.000651232 -0.049192987 0.009722588" rpy="0 0 0" />
+      <mass value="0.025" />
+      <inertia ixx="7.371e-05" ixy="-1.13e-06" ixz="2.1e-07"
+        iyy="7.81e-06" iyz="-1.372e-05" izz="7.47e-05" />
+    </inertial>
+    <visual>
+      <origin xyz="0 0 0" rpy="0 0 0" />
+      <geometry>
+        <mesh filename="package://robot_description/tron2/WFYG_TRON2A/meshes/gripper2_Link.STL" />
+      </geometry>
+      <material name="grey" />
+    </visual>
+    <collision>
+      <origin xyz="0 0 0" rpy="0 0 0" />
+      <geometry>
+        <mesh filename="package://robot_description/tron2/WFYG_TRON2A/meshes/gripper2_Link.STL" />
+      </geometry>
+    </collision>
+  </link>
+  <link name="antenna_L_Link">
+    <inertial>
+      <origin xyz="-2.7e-05 -0.028426 0.013784" rpy="0 0 0" />
+      <mass value="0.231" />
+      <inertia ixx="0.000424493" ixy="-1.15e-07" ixz="-1.18e-07"
+        iyy="0.000169977" iyz="3.0807e-05" izz="0.00039175" />
+    </inertial>
+    <visual>
+      <origin xyz="0 0 0" rpy="0 0 0" />
+      <geometry>
+        <mesh filename="package://robot_description/tron2/WFYG_TRON2A/meshes/antenna_L_Link.STL" />
+      </geometry>
+      <material name="white" />
+    </visual>
+    <collision>
+      <origin xyz="0 0 0" rpy="0 0 0" />
+      <geometry>
+        <mesh filename="package://robot_description/tron2/WFYG_TRON2A/meshes/antenna_L_Link_collision1.STL" />
+      </geometry>
+    </collision>
+    <collision>
+      <origin xyz="0 0 0" rpy="0 0 0" />
+      <geometry>
+        <mesh filename="package://robot_description/tron2/WFYG_TRON2A/meshes/antenna_L_Link_collision2.STL" />
+      </geometry>
+    </collision>
+  </link>
+  <link name="antenna_R_Link">
+    <inertial>
+      <origin xyz="2.7e-05 0.028426 0.013784" rpy="0 0 0" />
+      <mass value="0.231" />
+      <inertia ixx="0.000424493" ixy="-1.15e-07" ixz="1.17e-07"
+        iyy="0.000169977" iyz="-3.0808e-05" izz="0.000391749" />
+    </inertial>
+    <visual>
+      <origin xyz="0 0 0" rpy="0 0 0" />
+      <geometry>
+        <mesh filename="package://robot_description/tron2/WFYG_TRON2A/meshes/antenna_R_Link.STL" />
+      </geometry>
+      <material name="white" />
+    </visual>
+    <collision>
+      <origin xyz="0 0 0" rpy="0 0 0" />
+      <geometry>
+        <mesh filename="package://robot_description/tron2/WFYG_TRON2A/meshes/antenna_R_Link_collision1.STL" />
+      </geometry>
+    </collision>
+    <collision>
+      <origin xyz="0 0 0" rpy="0 0 0" />
+      <geometry>
+        <mesh filename="package://robot_description/tron2/WFYG_TRON2A/meshes/antenna_R_Link_collision2.STL" />
+      </geometry>
+    </collision>
+  </link>
+  <link name="camera_mount_Link">
+    <inertial>
+      <origin xyz="0.002536 0.000321 -0.060392" rpy="0 0 0" />
+      <mass value="0.381" />
+      <inertia ixx="0.001630905" ixy="-3.911e-06" ixz="-0.000204624"
+        iyy="0.001504517" iyz="-3.269e-06" izz="0.000548227" />
+    </inertial>
+    <visual>
+      <origin xyz="0 0 0" rpy="0 0 0" />
+      <geometry>
+        <mesh filename="package://robot_description/tron2/WFYG_TRON2A/meshes/camera_mount_Link.STL" />
+      </geometry>
+      <material name="white" />
+    </visual>
+    <collision>
+      <origin xyz="0 0 0" rpy="0 0 0" />
+      <geometry>
+        <mesh filename="package://robot_description/tron2/WFYG_TRON2A/meshes/camera_mount_Link_collision.STL" />
+      </geometry>
+    </collision>
+  </link>
+  <link name="radar_Link">
+    <inertial>
+      <origin xyz="-4.8e-05 8.4e-05 0.03502" rpy="0 0 0" />
+      <mass value="0.394" />
+      <inertia ixx="0.000308871" ixy="6.27e-07" ixz="-4.96e-07"
+        iyy="0.000308088" iyz="8.62e-07" izz="0.000305305" />
+    </inertial>
+    <visual>
+      <origin xyz="0 0 0" rpy="0 0 0" />
+      <geometry>
+        <mesh filename="package://robot_description/tron2/WFYG_TRON2A/meshes/radar_Link.STL" />
+      </geometry>
+      <material name="white" />
+    </visual>
+    <collision>
+      <origin xyz="0 0 0" rpy="0 0 0" />
+      <geometry>
+        <mesh filename="package://robot_description/tron2/WFYG_TRON2A/meshes/radar_Link.STL" />
+      </geometry>
+    </collision>
+  </link>
+  <!-- D435 Camera Links -->
+  <link name="d435_Link">
+    <visual>
+      <origin rpy="1.5707963267948966 0 1.5707963267948966" xyz="0.0 -0.0 0" />
+      <geometry>
+        <box size="0.01 0.01 0.001" />
+      </geometry>
+      <material name="camera_red">
+        <color rgba="1.0 0.0 0.0 1.0" />
+      </material>
+    </visual>
+  </link>
+  <joint name="d435_joint" type="fixed">
+    <origin rpy="0 1.063778179 0" xyz="0.12213 0.01759 0.00599" />
+    <parent link="base_imu" />
+    <child link="d435_Link" />
+  </joint>
+  <joint name="d435_optical_joint" type="fixed">
+    <origin rpy="-1.5707963267948966 0 -1.5707963267948966" xyz="0 0 0" />
+    <parent link="d435_Link" />
+    <child link="d435_optical_frame" />
+  </joint>
+  <link name="d435_optical_frame" />
   <!-- Joints -->
   <joint name="proximal_pitch_L_Joint" type="revolute">
@@ -369,4 +744,96 @@
     <limit lower="-1745329.2519943295" upper="1745329.2519943295" effort="22" velocity="41.89" />
   </joint>
+  <!-- Arm + Gripper + Peripherals joints (piper-x) -->
+  <joint name="transition_Joint" type="fixed">
+    <origin xyz="0.01 0.0 0.26915" rpy="0 0 0" />
+    <parent link="base_Link" />
+    <child link="transition_Link" />
+  </joint>
+  <joint name="arm_base_Joint" type="fixed">
+    <origin xyz="0.006 0.0 0.0" rpy="0 0 0" />
+    <parent link="transition_Link" />
+    <child link="arm_base_Link" />
+  </joint>
+  <joint name="arm1_Joint" type="revolute">
+    <origin xyz="0.0 0.0 0.123" rpy="0.0 0.0 3.1415926" />
+    <parent link="arm_base_Link" />
+    <child link="arm1_Link" />
+    <axis xyz="0 0 1" />
+    <limit lower="-2.6179938081783245" upper="2.6179938081783245" effort="100.0" velocity="5.0" />
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