Commit message: Feature/tron2 v5 0224

File: tron2/DA_TRON2A/urdf/robot.urdf (robot description, URDF)
Before this commit: robot bipedal_robot, 23 links, 22 joints
Links:
- removed link L_ee_Link
- removed link R_ee_Link
- removed link abad_L_Link
- removed link abad_R_Link
- removed link hip_L_Link
- removed link hip_R_Link
- removed link knee_L_Link
- removed link knee_R_Link
- removed link world
- removed link yaw_L_Link
- removed link yaw_R_Link
- added link elbow_L_Link, mass 1.11; collision mesh filename=package://robot_description/tron2/DA_TRON2A/meshes/elbow_L_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; visual mesh filename=package://robot_description/tron2/DA_TRON2A/meshes/elbow_L_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
- added link elbow_R_Link, mass 1.11; collision mesh filename=package://robot_description/tron2/DA_TRON2A/meshes/elbow_R_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; visual mesh filename=package://robot_description/tron2/DA_TRON2A/meshes/elbow_R_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
- added link proximal_pitch_L_Link, mass 2.07; collision mesh filename=package://robot_description/tron2/DA_TRON2A/meshes/proximal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; visual mesh filename=package://robot_description/tron2/DA_TRON2A/meshes/proximal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
- added link proximal_pitch_R_Link, mass 2.07; collision mesh filename=package://robot_description/tron2/DA_TRON2A/meshes/proximal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; visual mesh filename=package://robot_description/tron2/DA_TRON2A/meshes/proximal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
- added link proximal_roll_L_Link, mass 1.74; collision mesh filename=package://robot_description/tron2/DA_TRON2A/meshes/proximal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; visual mesh filename=package://robot_description/tron2/DA_TRON2A/meshes/proximal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
- added link proximal_roll_R_Link, mass 1.74; collision mesh filename=package://robot_description/tron2/DA_TRON2A/meshes/proximal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; visual mesh filename=package://robot_description/tron2/DA_TRON2A/meshes/proximal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
- added link proximal_yaw_L_Link, mass 1.15; collision mesh filename=package://robot_description/tron2/DA_TRON2A/meshes/proximal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; visual mesh filename=package://robot_description/tron2/DA_TRON2A/meshes/proximal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
- added link proximal_yaw_R_Link, mass 1.15; collision mesh filename=package://robot_description/tron2/DA_TRON2A/meshes/proximal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; visual mesh filename=package://robot_description/tron2/DA_TRON2A/meshes/proximal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
- link base_2_Link: mass 0.1 -> 0; geometry collision mesh filename=package://robot_description/tron2/DA_TRON2A/meshes/base_2_L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; visual mesh filename=package://robot_description/tron2/DA_TRON2A/meshes/base_2_L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
- link base_3_Link: mass 0.1 -> 0; geometry collision mesh filename=package://robot_description/tron2/DA_TRON2A/meshes/base_3_L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; visual mesh filename=package://robot_description/tron2/DA_TRON2A/meshes/base_3_L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
- link base_Link: mass 10.92 -> 11.07; geometry collision mesh filename=package://robot_description/tron2/DA_TRON2A/meshes/base_Lin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; visual mesh filename=package://robot_description/tron2/DA_TRON2A/meshes/base_Lin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
- link grasper_L_Link: mass 0.66 -> 0.53; geometry collision mesh filename=package://robot_description/tron2/DA_TRON2A/meshes/grasper_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; visual mesh filename=package://robot_description/tron2/DA_TRON2A/meshes/grasper_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
- link grasper_R_Link: mass 0.66 -> 0.53; geometry collision mesh filename=package://robot_description/tron2/DA_TRON2A/meshes/grasper_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; visual mesh filename=package://robot_description/tron2/DA_TRON2A/meshes/grasper_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
- link wrist_pitch_L_Link: mass 0.70 -> 0.44; geometry collision mesh filename=package://robot_description/tron2/DA_TRON2A/meshes/wrist_pi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; visual mesh filename=package://robot_description/tron2/DA_TRON2A/meshes/wrist_pi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
- link wrist_pitch_R_Link: mass 0.70 -> 0.44; geometry collision mesh filename=package://robot_description/tron2/DA_TRON2A/meshes/wrist_pi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; visual mesh filename=package://robot_description/tron2/DA_TRON2A/meshes/wrist_pi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
- link wrist_roll_L_Link: mass 0.26 -> 0.24; geometry collision mesh filename=package://robot_description/tron2/DA_TRON2A/meshes/wrist_ro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; visual mesh filename=package://robot_description/tron2/DA_TRON2A/meshes/wrist_ro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
- link wrist_roll_R_Link: mass 0.26 -> 0.24; geometry collision mesh filename=package://robot_description/tron2/DA_TRON2A/meshes/wrist_ro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; visual mesh filename=package://robot_description/tron2/DA_TRON2A/meshes/wrist_ro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
- link wrist_yaw_L_Link: mass 0.90 -> 1.15; geometry collision mesh filename=package://robot_description/tron2/DA_TRON2A/meshes/wrist_ya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; visual mesh filename=package://robot_description/tron2/DA_TRON2A/meshes/wrist_ya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
- link wrist_yaw_R_Link: mass 0.90 -> 1.15; geometry collision mesh filename=package://robot_description/tron2/DA_TRON2A/meshes/wrist_ya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; visual mesh filename=package://robot_description/tron2/DA_TRON2A/meshes/wrist_ya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
Joints:
- removed joint L_ee_Joint
- removed joint R_ee_Joint
- removed joint abad_L_Joint
- removed joint abad_R_Joint
- removed joint base_3_joint
- removed joint base_fixed_joint
- removed joint grasper_L_joint
- removed joint hip_L_Joint
- removed joint hip_R_Joint
- removed joint knee_L_Joint
- removed joint knee_R_Joint
- removed joint yaw_L_Joint
- removed joint yaw_R_Joint
- added joint base_3_Joint: type fixed, parent base_2_Link, child base_3_Link, origin xyz=0.0 0.0 -0.9295 rpy=0 0 0
- added joint elbow_L_Joint: type revolute, parent proximal_yaw_L_Link, child elbow_L_Link, origin xyz=0.004 0.02972 -0.2126 rpy=0 0 0, axis 0 1 0, limit lower=-2.6179938779914944 upper=0.5235987755982988 effort=70 velocity=22.52
- added joint elbow_R_Joint: type revolute, parent proximal_yaw_R_Link, child elbow_R_Link, origin xyz=0.004 -0.02972 -0.2126 rpy=0 0 0, axis 0 1 0, limit lower=-2.6179938779914944 upper=0.5235987755982988 effort=70 velocity=22.52
- added joint grasper_L_Joint: type fixed, parent wrist_roll_L_Link, child grasper_L_Link, origin xyz=-0.0317 0.0 -0.0812 rpy=0 0 0
- added joint proximal_pitch_L_Joint: type revolute, parent base_Link, child proximal_pitch_L_Link, origin xyz=-0.00044 0.09178 0.05474 rpy=0 0 0, axis 0 0.99619 -0.087155, limit lower=-3.141592653589793 upper=2.600540585471551 effort=200 velocity=18.3
- added joint proximal_pitch_R_Joint: type revolute, parent base_Link, child proximal_pitch_R_Link, origin xyz=-0.00044 -0.09178 0.05474 rpy=0 0 0, axis 0 0.99619 0.087155, limit lower=-3.141592653589793 upper=2.600540585471551 effort=200 velocity=18.3
- added joint proximal_roll_L_Joint: type revolute, parent proximal_pitch_L_Link, child proximal_roll_L_Link, origin xyz=-0.032 0.0758 -0.00663 rpy=0 0 0, axis 1 0 0, limit lower=-0.2617993877991494 upper=3.2288591161895095 effort=200 velocity=18.3
- added joint proximal_roll_R_Joint: type revolute, parent proximal_pitch_R_Link, child proximal_roll_R_Link, origin xyz=-0.032 -0.0758 -0.00663 rpy=0 0 0, axis 1 0 0, limit lower=-3.2288591161895095 upper=0.2617993877991494 effort=200 velocity=18.3
- added joint proximal_yaw_L_Joint: type revolute, parent proximal_roll_L_Link, child proximal_yaw_L_Link, origin xyz=0.032 0.0 -0.1374 rpy=0 0 0, axis 0 0 1, limit lower=-3.6651914291880923 upper=1.4835298641951802 effort=70 velocity=22.52
- added joint proximal_yaw_R_Joint: type revolute, parent proximal_roll_R_Link, child proximal_yaw_R_Link, origin xyz=0.032 -0.0 -0.1374 rpy=0 0 0, axis 0 0 1, limit lower=-1.4835298641951802 upper=3.6651914291880923 effort=70 velocity=22.52
- joint base_2_Joint: origin xyz=0.0048 9e-05 -0.09005 rpy=0 0 0 -> xyz=0.00056 -9e-05 -0.07285 rpy=0 0 0
- joint grasper_R_Joint: origin xyz=-0.0338 0 -0.0825 rpy=0 0 0 -> xyz=-0.0317 -0.0 -0.0812 rpy=0 0 0
- joint wrist_pitch_L_Joint: origin xyz=0.0 0.0307 -0.1231 rpy=0 0 0 -> xyz=0.0 0.0367 -0.1743 rpy=0 0 0
- joint wrist_pitch_R_Joint: origin xyz=0 -0.0307 -0.1231 rpy=0 0 0 -> xyz=0.0 -0.0367 -0.1743 rpy=0 0 0
- joint wrist_roll_L_Joint: limit lower=-1.7453292519943295 upper=1.7453292519943295 effort=20 velocity=17.8 -> lower=-1.5707963267948966 upper=1.5707963267948966 effort=20 velocity=17.8; origin xyz=0.0338 -0.0304 0.0 rpy=0 0 0 -> xyz=0.0317 -0.0367 0.0 rpy=0 0 0
- joint wrist_roll_R_Joint: limit lower=-1.7453292519943295 upper=1.7453292519943295 effort=20 velocity=17.8 -> lower=-1.5707963267948966 upper=1.5707963267948966 effort=20 velocity=17.8; origin xyz=0.0338 0.0304 0 rpy=0 0 0 -> xyz=0.0317 0.0367 0.0 rpy=0 0 0
- joint wrist_yaw_L_Joint: limit lower=-2.356194490192345 upper=0.7853981633974483 effort=20 velocity=17.8 -> lower=-1.7453292519943295 upper=1.3962634015954636 effort=20 velocity=17.8; origin xyz=0.0 -0.0305 -0.1912 rpy=0 0 0 -> xyz=-0.004 -0.02972 -0.0685 rpy=0 0 0; parent knee_L_Link -> elbow_L_Link
- joint wrist_yaw_R_Joint: limit lower=-0.7853981633974483 upper=2.356194490192345 effort=20 velocity=17.8 -> lower=-1.3962634015954636 upper=1.7453292519943295 effort=20 velocity=17.8; origin xyz=0 0.0305 -0.1912 rpy=0 0 0 -> xyz=-0.004 0.02972 -0.0685 rpy=0 0 0; parent knee_R_Link -> elbow_R_Link

Commit message: Feat/tron2 v5 ros2

File: tron2/DA_TRON2A/urdf/robot.urdf (robot description, URDF)
Before this commit: robot bipedal_robot, 20 links, 19 joints
Links:
- link base_2_Link: geometry collision mesh filename=../meshes/base_2_Link.STL; visual mesh filename=../meshes/base_2_Link.STL
- link base_3_Link: geometry collision mesh filename=../meshes/base_3_Link.STL; visual mesh filename=../meshes/base_3_Link.STL
- link base_Link: geometry collision mesh filename=../meshes/base_Link.STL; visual mesh filename=../meshes/base_Link.STL
- link elbow_L_Link: geometry collision mesh filename=../meshes/elbow_L_Link.STL; visual mesh filename=../meshes/elbow_L_Link.STL
- link elbow_R_Link: geometry collision mesh filename=../meshes/elbow_R_Link.STL; visual mesh filename=../meshes/elbow_R_Link.STL
- link grasper_L_Link: geometry collision mesh filename=../meshes/grasper_L_Link.STL; visual mesh filename=../meshes/grasper_L_Link.STL
- link grasper_R_Link: geometry collision mesh filename=../meshes/grasper_R_Link.STL; visual mesh filename=../meshes/grasper_R_Link.STL
- link proximal_pitch_L_Link: geometry collision mesh filename=../meshes/proximal_pitch_L_Link.STL; visual mesh filename=../meshes/proximal_pitch_L_Link.STL
- link proximal_pitch_R_Link: geometry collision mesh filename=../meshes/proximal_pitch_R_Link.STL; visual mesh filename=../meshes/proximal_pitch_R_Link.STL
- link proximal_roll_L_Link: geometry collision mesh filename=../meshes/proximal_roll_L_Link.STL; visual mesh filename=../meshes/proximal_roll_L_Link.STL
- link proximal_roll_R_Link: geometry collision mesh filename=../meshes/proximal_roll_R_Link.STL; visual mesh filename=../meshes/proximal_roll_R_Link.STL
- link proximal_yaw_L_Link: geometry collision mesh filename=../meshes/proximal_yaw_L_Link.STL; visual mesh filename=../meshes/proximal_yaw_L_Link.STL
- link proximal_yaw_R_Link: geometry collision mesh filename=../meshes/proximal_yaw_R_Link.STL; visual mesh filename=../meshes/proximal_yaw_R_Link.STL
- link wrist_pitch_L_Link: geometry collision mesh filename=../meshes/wrist_pitch_L_Link.STL; visual mesh filename=../meshes/wrist_pitch_L_Link.STL
- link wrist_pitch_R_Link: geometry collision mesh filename=../meshes/wrist_pitch_R_Link.STL; visual mesh filename=../meshes/wrist_pitch_R_Link.STL
- link wrist_roll_L_Link: geometry collision mesh filename=../meshes/wrist_roll_L_Link.STL; visual mesh filename=../meshes/wrist_roll_L_Link.STL
- link wrist_roll_R_Link: geometry collision mesh filename=../meshes/wrist_roll_R_Link.STL; visual mesh filename=../meshes/wrist_roll_R_Link.STL
- link wrist_yaw_L_Link: geometry collision mesh filename=../meshes/wrist_yaw_L_Link.STL; visual mesh filename=../meshes/wrist_yaw_L_Link.STL
- link wrist_yaw_R_Link: geometry collision mesh filename=../meshes/wrist_yaw_R_Link.STL; visual mesh filename=../meshes/wrist_yaw_R_Link.STL

File: tron2/SF_TRON2A/urdf/robot.urdf (robot description, URDF)
Before this commit: robot bipedal_robot, 12 links, 11 joints
Links:
- added link d435_Link; visual box size=0.01 0.01 0.001
- added link d435_optical_frame
Joints:
- added joint d435_joint: type fixed, parent limx_imu, child d435_Link, origin xyz=0.12213 0.01759 0.00599 rpy=0 1.063778179 0
- added joint d435_optical_joint: type fixed, parent d435_Link, child d435_optical_frame, origin xyz=0 0 0 rpy=-1.5707963267948966 0 -1.5707963267948966
- joint ankle_pitch_R_Joint: axis 0 0.99619 0.087155 -> 0 1 0
- joint proximal_pitch_R_Joint: axis 0 1 0 -> 0 0.99619 0.087155

File: tron2/WF_TRON2A/urdf/robot.urdf (robot description, URDF)
Before this commit: robot bipedal_robot, 12 links, 11 joints
Links:
- link wheel_L_Link: geometry collision cylinder length=0.045 radius=0.1; visual mesh filename=package://robot_description/tron2/WF_TRON2A/meshes/wheel_L_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
- link wheel_R_Link: geometry collision cylinder length=0.045 radius=0.1; visual mesh filename=package://robot_description/tron2/WF_TRON2A/meshes/wheel_R_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

Commit message: feat: regenerate DA_TRON2A

File: tron2/DA_TRON2A/urdf/robot.urdf (robot description, URDF)
Before this commit: robot bipedal_robot, 20 links, 19 joints
Links:
- added link base_imu, mass 0.01
- added link d435_Link; visual box size=0.01 0.01 0.001
- added link d435_optical_frame
- link base_2_Link: mass 0 -> 0.001; geometry collision mesh filename=package://bipedal_robot/meshes/base_2_Link.STL; visual mesh filename=package://bipedal_robot/meshes/base_2_Link.STL
- link base_3_Link: mass 0 -> 0.001; geometry collision mesh filename=package://bipedal_robot/meshes/base_3_Link.STL; visual mesh filename=package://bipedal_robot/meshes/base_3_Link.STL
- link base_Link: geometry collision mesh filename=package://bipedal_robot/meshes/base_Link.STL; visual mesh filename=package://bipedal_robot/meshes/base_Link.STL
- link elbow_L_Link: geometry collision mesh filename=package://bipedal_robot/meshes/elbow_L_Link.STL; visual mesh filename=package://bipedal_robot/meshes/elbow_L_Link.STL
- link elbow_R_Link: geometry collision mesh filename=package://bipedal_robot/meshes/elbow_R_Link.STL; visual mesh filename=package://bipedal_robot/meshes/elbow_R_Link.STL
- link grasper_L_Link: geometry collision mesh filename=package://bipedal_robot/meshes/grasper_L_Link.STL; visual mesh filename=package://bipedal_robot/meshes/grasper_L_Link.STL
- link grasper_R_Link: geometry collision mesh filename=package://bipedal_robot/meshes/grasper_R_Link.STL; visual mesh filename=package://bipedal_robot/meshes/grasper_R_Link.STL
- link proximal_pitch_L_Link: geometry collision mesh filename=package://bipedal_robot/meshes/proximal_pitch_L_Link.STL; visual mesh filename=package://bipedal_robot/meshes/proximal_pitch_L_Link.STL
- link proximal_pitch_R_Link: geometry collision mesh filename=package://bipedal_robot/meshes/proximal_pitch_R_Link.STL; visual mesh filename=package://bipedal_robot/meshes/proximal_pitch_R_Link.STL
- link proximal_roll_L_Link: geometry collision mesh filename=package://bipedal_robot/meshes/proximal_roll_L_Link.STL; visual mesh filename=package://bipedal_robot/meshes/proximal_roll_L_Link.STL
- link proximal_roll_R_Link: geometry collision mesh filename=package://bipedal_robot/meshes/proximal_roll_R_Link.STL; visual mesh filename=package://bipedal_robot/meshes/proximal_roll_R_Link.STL
- link proximal_yaw_L_Link: geometry collision mesh filename=package://bipedal_robot/meshes/proximal_yaw_L_Link_collisio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; visual mesh filename=package://bipedal_robot/meshes/proximal_yaw_L_Link.STL
- link proximal_yaw_R_Link: geometry collision mesh filename=package://bipedal_robot/meshes/proximal_yaw_R_Link_collisio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; visual mesh filename=package://bipedal_robot/meshes/proximal_yaw_R_Link.STL
- link wrist_pitch_L_Link: geometry collision mesh filename=package://bipedal_robot/meshes/wrist_pitch_L_Link.STL; visual mesh filename=package://bipedal_robot/meshes/wrist_pitch_L_Link.STL
- link wrist_pitch_R_Link: geometry collision mesh filename=package://bipedal_robot/meshes/wrist_pitch_R_Link.STL; visual mesh filename=package://bipedal_robot/meshes/wrist_pitch_R_Link.STL
- link wrist_roll_L_Link: geometry collision mesh filename=package://bipedal_robot/meshes/wrist_roll_L_Link_collision.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; visual mesh filename=package://bipedal_robot/meshes/wrist_roll_L_Link.STL
- link wrist_roll_R_Link: geometry collision mesh filename=package://bipedal_robot/meshes/wrist_roll_R_Link_collision.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; visual mesh filename=package://bipedal_robot/meshes/wrist_roll_R_Link.STL
- link wrist_yaw_L_Link: geometry collision mesh filename=package://bipedal_robot/meshes/wrist_yaw_L_Link.STL; visual mesh filename=package://bipedal_robot/meshes/wrist_yaw_L_Link.STL
- link wrist_yaw_R_Link: geometry collision mesh filename=package://bipedal_robot/meshes/wrist_yaw_R_Link.STL; visual mesh filename=package://bipedal_robot/meshes/wrist_yaw_R_Link.STL
Joints:
- added joint base_imu_Joint: type fixed, parent base_Link, child base_imu, origin xyz=0.0 0.0 0.0 rpy=0.0 0.0 0.0
- added joint d435_joint: type fixed, parent limx_imu, child d435_Link, origin xyz=0.12213 0.01759 0.00599 rpy=0.0 1.063778179 0.0
- added joint d435_optical_joint: type fixed, parent d435_Link, child d435_optical_frame, origin xyz=0 0 0 rpy=-1.5707963267948966 0 -1.5707963267948966
- joint base_2_Joint: origin xyz=0.00056 -9e-05 -0.07285 rpy=0 0 0 -> xyz=0.00056 -9e-05 -0.07285 rpy=0.0 0.0 0.0
- joint base_3_Joint: origin xyz=0.0 0.0 -0.9295 rpy=0 0 0 -> xyz=0.0 0.0 -0.9295 rpy=0.0 0.0 0.0
- joint elbow_L_Joint: axis 0 1 0 -> 0.0 1.0 0.0; limit lower=-2.6179938779914944 upper=0.5235987755982988 effort=70 velocity=22.52 -> lower=-2.6179938779914944 upper=0.5235987755982988 effort=70.0 velocity=22.52; origin xyz=0.004 0.02972 -0.2126 rpy=0 0 0 -> xyz=0.004 0.02972 -0.2126 rpy=0.0 0.0 0.0
- joint elbow_R_Joint: axis 0 1 0 -> 0.0 1.0 0.0; limit lower=-2.6179938779914944 upper=0.5235987755982988 effort=70 velocity=22.52 -> lower=-2.6179938779914944 upper=0.5235987755982988 effort=70.0 velocity=22.52; origin xyz=0.004 -0.02972 -0.2126 rpy=0 0 0 -> xyz=0.004 -0.02972 -0.2126 rpy=0.0 0.0 0.0
- joint grasper_L_Joint: origin xyz=-0.0317 0.0 -0.0812 rpy=0 0 0 -> xyz=-0.0317 0.0 -0.0812 rpy=0.0 0.0 0.0
- joint grasper_R_Joint: origin xyz=-0.0317 -0.0 -0.0812 rpy=0 0 0 -> xyz=-0.0317 -0.0 -0.0812 rpy=0.0 0.0 0.0
- joint limx_imu_joint: origin xyz=0. 0. 0. rpy=0. 0. 0. -> xyz=0.0 0.0 0.0 rpy=0.0 0.0 0.0
- joint proximal_pitch_L_Joint: axis 0 0.99619 -0.087155 -> 0.0 0.9961947268929313 -0.0871554135479712; limit lower=-3.141592653589793 upper=2.600540585471551 effort=150 velocity=18.3 -> lower=-3.141592653589793 upper=2.600540585471551 effort=150.0 velocity=18.3; origin xyz=-0.00044 0.09178 0.05474 rpy=0 0 0 -> xyz=-0.00044 0.09178 0.05474 rpy=0.0 0.0 0.0
- joint proximal_pitch_R_Joint: axis 0 0.99619 0.087155 -> 0.0 0.9961947268929313 0.0871554135479712; limit lower=-3.141592653589793 upper=2.600540585471551 effort=150 velocity=18.3 -> lower=-3.141592653589793 upper=2.600540585471551 effort=150.0 velocity=18.3; origin xyz=-0.00044 -0.09178 0.05474 rpy=0 0 0 -> xyz=-0.00044 -0.09178 0.05474 rpy=0.0 0.0 0.0
- joint proximal_roll_L_Joint: axis 1 0 0 -> 1.0 0.0 0.0; limit lower=-0.2617993877991494 upper=3.19395248 effort=150 velocity=18.3 -> lower=-0.2617993877991494 upper=3.1939524787897455 effort=150.0 velocity=18.3; origin xyz=-0.032 0.0758 -0.00663 rpy=0 0 0 -> xyz=-0.032 0.0758 -0.00663 rpy=0.0 0.0 0.0
- joint proximal_roll_R_Joint: axis 1 0 0 -> 1.0 0.0 0.0; limit lower=-3.19395248 upper=0.2617993877991494 effort=150 velocity=18.3 -> lower=-3.1939524787897455 upper=0.2617993877991494 effort=150.0 velocity=18.3; origin xyz=-0.032 -0.0758 -0.00663 rpy=0 0 0 -> xyz=-0.032 -0.0758 -0.00663 rpy=0.0 0.0 0.0
- joint proximal_yaw_L_Joint: axis 0 0 1 -> 0.0 0.0 1.0; limit lower=-3.6651914291880923 upper=1.4835298641951802 effort=60 velocity=22.52 -> lower=-3.6651914291880923 upper=1.4835298641951802 effort=60.0 velocity=22.52; origin xyz=0.032 0.0 -0.1374 rpy=0 0 0 -> xyz=0.032 0.0 -0.1374 rpy=0.0 0.0 0.0
- joint proximal_yaw_R_Joint: axis 0 0 1 -> 0.0 0.0 1.0; limit lower=-1.4835298641951802 upper=3.6651914291880923 effort=60 velocity=22.52 -> lower=-1.4835298641951802 upper=3.6651914291880923 effort=60.0 velocity=22.52; origin xyz=0.032 -0.0 -0.1374 rpy=0 0 0 -> xyz=0.032 -0.0 -0.1374 rpy=0.0 0.0 0.0
- joint wrist_pitch_L_Joint: axis 0 1 0 -> 0.0 1.0 0.0; limit lower=-0.7853981633974483 upper=0.7853981633974483 effort=20 velocity=17.8 -> lower=-0.7853981633974483 upper=0.7853981633974483 effort=20.0 velocity=17.8; origin xyz=0.0 0.0367 -0.1743 rpy=0 0 0 -> xyz=0.0 0.0367 -0.1743 rpy=0.0 0.0 0.0
- joint wrist_pitch_R_Joint: axis 0 1 0 -> 0.0 1.0 0.0; limit lower=-0.7853981633974483 upper=0.7853981633974483 effort=20 velocity=17.8 -> lower=-0.7853981633974483 upper=0.7853981633974483 effort=20.0 velocity=17.8; origin xyz=0.0 -0.0367 -0.1743 rpy=0 0 0 -> xyz=0.0 -0.0367 -0.1743 rpy=0.0 0.0 0.0
- joint wrist_roll_L_Joint: axis 1 0 0 -> 1.0 0.0 0.0; limit lower=-1.5707963267948966 upper=1.5707963267948966 effort=20 velocity=17.8 -> lower=-1.5707963267948966 upper=1.5707963267948966 effort=20.0 velocity=17.8; origin xyz=0.0317 -0.0367 0.0 rpy=0 0 0 -> xyz=0.0317 -0.0367 0.0 rpy=0.0 0.0 0.0
- joint wrist_roll_R_Joint: axis 1 0 0 -> 1.0 0.0 0.0; limit lower=-1.5707963267948966 upper=1.5707963267948966 effort=20 velocity=17.8 -> lower=-1.5707963267948966 upper=1.5707963267948966 effort=20.0 velocity=17.8; origin xyz=0.0317 0.0367 0.0 rpy=0 0 0 -> xyz=0.0317 0.0367 0.0 rpy=0.0 0.0 0.0
- joint wrist_yaw_L_Joint: axis 0 0 1 -> 0.0 0.0 1.0; limit lower=-1.7453292519943295 upper=1.3962634015954636 effort=20 velocity=17.8 -> lower=-1.7453292519943295 upper=1.3962634015954636 effort=20.0 velocity=17.8; origin xyz=-0.004 -0.02972 -0.0685 rpy=0 0 0 -> xyz=-0.004 -0.02972 -0.0685 rpy=0.0 0.0 0.0
- joint wrist_yaw_R_Joint: axis 0 0 1 -> 0.0 0.0 1.0; limit lower=-1.3962634015954636 upper=1.7453292519943295 effort=20 velocity=17.8 -> lower=-1.3962634015954636 upper=1.7453292519943295 effort=20.0 velocity=17.8; origin xyz=-0.004 0.02972 -0.0685 rpy=0 0 0 -> xyz=-0.004 0.02972 -0.0685 rpy=0.0 0.0 0.0
