Commit message: feat: add d435 link & remove gazebo info & fixed DA base

File: tron2/DA_TRON2A/urdf/robot.urdf (robot description, URDF)
Before this commit: robot bipedal_robot, 23 links, 22 joints
Links:
- removed link limx_imu
- link d435_Link: mass None -> 0.001; geometry visual box size=0.005 0.005 0.005
- link d435_optical_frame: mass None -> 0.001
Joints:
- removed joint d435_joint
- removed joint d435_optical_joint
- removed joint limx_imu_joint
- added joint d435_Joint: type fixed, parent base_Link, child d435_Link, origin xyz=0.0968 0.01759 -0.00409 rpy=0 2.7227 0
- added joint d435_optical_Joint: type fixed, parent d435_Link, child d435_optical_frame, origin xyz=0 0 0 rpy=-1.5707963267948966 0 -1.5707963267948966

File: tron2/DA_TRON2A/urdf/robot_rl.urdf (robot description, URDF)
Before this commit: robot bipedal_robot, 20 links, 19 joints
Links:
- added link d435_Link, mass 0.001; visual box size=0.005 0.005 0.005
- added link d435_optical_frame, mass 0.001
Joints:
- added joint d435_Joint: type fixed, parent base_Link, child d435_Link, origin xyz=0.0968 0.01759 -0.00409 rpy=0 2.7227 0
- added joint d435_optical_Joint: type fixed, parent d435_Link, child d435_optical_frame, origin xyz=0 0 0 rpy=-1.5707963267948966 0 -1.5707963267948966

File: tron2/SFYG_TRON2A/urdf/robot.urdf (robot description, URDF)
Before this commit: robot bipedal_robot, 29 links, 28 joints
Links:
- removed link limx_imu
- link d435_Link: mass None -> 0.001; geometry visual box size=0.005 0.005 0.005
- link d435_optical_frame: mass None -> 0.001
Joints:
- removed joint d435_joint
- removed joint d435_optical_joint
- removed joint limx_imu_joint
- added joint d435_Joint: type fixed, parent base_Link, child d435_Link, origin xyz=0.0968 0.01759 -0.00409 rpy=0 2.7227 0
- added joint d435_optical_Joint: type fixed, parent d435_Link, child d435_optical_frame, origin xyz=0 0 0 rpy=-1.5707963267948966 0 -1.5707963267948966

File: tron2/SFYG_TRON2A/urdf/robot_rl.urdf (robot description, URDF)
Before this commit: robot bipedal_robot, 27 links, 26 joints
Links:
- added link d435_Link, mass 0.001; visual box size=0.005 0.005 0.005
- added link d435_optical_frame, mass 0.001
Joints:
- added joint d435_Joint: type fixed, parent base_Link, child d435_Link, origin xyz=0.0968 0.01759 -0.00409 rpy=0 2.7227 0
- added joint d435_optical_Joint: type fixed, parent d435_Link, child d435_optical_frame, origin xyz=0 0 0 rpy=-1.5707963267948966 0 -1.5707963267948966

File: tron2/SF_TRON2A/urdf/robot.urdf (robot description, URDF)
Before this commit: robot bipedal_robot, 15 links, 14 joints
Links:
- link d435_Link: mass None -> 0.001; geometry visual box size=0.005 0.005 0.005
- link d435_optical_frame: mass None -> 0.001
Joints:
- removed joint d435_joint
- removed joint d435_optical_joint
- added joint d435_Joint: type fixed, parent base_Link, child d435_Link, origin xyz=0.0968 0.01759 -0.00409 rpy=0 2.7227 0
- added joint d435_optical_Joint: type fixed, parent d435_Link, child d435_optical_frame, origin xyz=0 0 0 rpy=-1.5707963267948966 0 -1.5707963267948966

File: tron2/SF_TRON2A/urdf/robot_rl.urdf (robot description, URDF)
Before this commit: robot bipedal_robot, 12 links, 11 joints
Links:
- added link d435_Link, mass 0.001; visual box size=0.005 0.005 0.005
- added link d435_optical_frame, mass 0.001
Joints:
- added joint d435_Joint: type fixed, parent base_Link, child d435_Link, origin xyz=0.0968 0.01759 -0.00409 rpy=0 2.7227 0
- added joint d435_optical_Joint: type fixed, parent d435_Link, child d435_optical_frame, origin xyz=0 0 0 rpy=-1.5707963267948966 0 -1.5707963267948966

File: tron2/WFYG_TRON2A/urdf/robot.urdf (robot description, URDF)
Before this commit: robot bipedal_robot, 29 links, 28 joints
Links:
- removed link limx_imu
- link d435_Link: mass None -> 0.001; geometry visual box size=0.005 0.005 0.005
- link d435_optical_frame: mass None -> 0.001
Joints:
- removed joint d435_joint
- removed joint d435_optical_joint
- removed joint limx_imu_joint
- added joint d435_Joint: type fixed, parent base_Link, child d435_Link, origin xyz=0.0968 0.01759 -0.00409 rpy=0 2.7227 0
- added joint d435_optical_Joint: type fixed, parent d435_Link, child d435_optical_frame, origin xyz=0 0 0 rpy=-1.5707963267948966 0 -1.5707963267948966

File: tron2/WFYG_TRON2A/urdf/robot_rl.urdf (robot description, URDF)
Before this commit: robot bipedal_robot, 27 links, 26 joints
Links:
- added link d435_Link, mass 0.001; visual box size=0.005 0.005 0.005
- added link d435_optical_frame, mass 0.001
Joints:
- added joint d435_Joint: type fixed, parent base_Link, child d435_Link, origin xyz=0.0968 0.01759 -0.00409 rpy=0 2.7227 0
- added joint d435_optical_Joint: type fixed, parent d435_Link, child d435_optical_frame, origin xyz=0 0 0 rpy=-1.5707963267948966 0 -1.5707963267948966

File: tron2/WF_TRON2A/urdf/robot.urdf (robot description, URDF)
Before this commit: robot bipedal_robot, 15 links, 14 joints
Links:
- removed link limx_imu
- link d435_Link: mass None -> 0.001; geometry visual box size=0.005 0.005 0.005
- link d435_optical_frame: mass None -> 0.001
Joints:
- removed joint d435_joint
- removed joint d435_optical_joint
- removed joint limx_imu_joint
- added joint d435_Joint: type fixed, parent base_Link, child d435_Link, origin xyz=0.0968 0.01759 -0.00409 rpy=0 2.7227 0
- added joint d435_optical_Joint: type fixed, parent d435_Link, child d435_optical_frame, origin xyz=0 0 0 rpy=-1.5707963267948966 0 -1.5707963267948966

File: tron2/WF_TRON2A/urdf/robot_rl.urdf (robot description, URDF)
Before this commit: robot bipedal_robot, 12 links, 11 joints
Links:
- added link d435_Link, mass 0.001; visual box size=0.005 0.005 0.005
- added link d435_optical_frame, mass 0.001
Joints:
- added joint d435_Joint: type fixed, parent base_Link, child d435_Link, origin xyz=0.0968 0.01759 -0.00409 rpy=0 2.7227 0
- added joint d435_optical_Joint: type fixed, parent d435_Link, child d435_optical_frame, origin xyz=0 0 0 rpy=-1.5707963267948966 0 -1.5707963267948966

Commit message: feat: regenerate DACH_TRON2A & fix DA_TRON2A base_2&3 inertial and collision

File: tron2/DA_TRON2A/urdf/robot.urdf (robot description, URDF)
Before this commit: robot bipedal_robot, 22 links, 21 joints
Links:
- link base_2_Link: mass 0.001 -> 10; geometry collision box size=0.118 0.085 0.98; visual mesh filename=package://bipedal_robot/meshes/base_2_Link.STL
- link base_3_Link: mass 0.001 -> 20

File: tron2/DA_TRON2A/urdf/robot_rl.urdf (robot description, URDF)
Before this commit: robot bipedal_robot, 22 links, 21 joints
Links:
- link base_2_Link: mass 0.001 -> 10; geometry collision box size=0.118 0.085 0.98; visual mesh filename=../meshes/base_2_Link.STL
- link base_3_Link: mass 0.001 -> 20
