Commit message: feat: SFYG, arm=piper-x

File: tron2/SFYG_TRON2A/urdf/robot.urdf (robot description, URDF)
Before this commit: robot bipedal_robot, 27 links, 26 joints
Links:
- removed link arm7_Link
- removed link gripper_flange_Link
- added link antenna_L_Link, mass 0.231; collision mesh filename=package://bipedal_robot/meshes/antenna_L_Link_collision1.STL; collision mesh filename=package://bipedal_robot/meshes/antenna_L_Link_collision2.STL
- added link antenna_R_Link, mass 0.231; collision mesh filename=package://bipedal_robot/meshes/antenna_R_Link_collision1.STL; collision mesh filename=package://bipedal_robot/meshes/antenna_R_Link_collision2.STL
- added link camera_mount_Link, mass 0.381; collision mesh filename=package://bipedal_robot/meshes/camera_mount_Link_collision.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; visual mesh filename=package://bipedal_robot/meshes/camera_mount_Link.STL
- added link radar_Link, mass 0.394; collision mesh filename=package://bipedal_robot/meshes/radar_Link.STL; visual mesh filename=package://bipedal_robot/meshes/radar_Link.STL
- link ankle_pitch_L_Link: geometry collision box size=0.14 0.06 0.025; collision sphere radius=0.0025
- link ankle_pitch_R_Link: geometry collision box size=0.14 0.06 0.025; collision sphere radius=0.0025
- link arm1_Link: mass 0.77 -> 0.71
- link arm2_Link: mass 0.69 -> 1.16; geometry collision mesh filename=package://bipedal_robot/meshes/arm2_Link_collision1.STL; collision mesh filename=package://bipedal_robot/meshes/arm2_Link_collision2.STL
- link arm3_Link: geometry collision mesh filename=package://bipedal_robot/meshes/arm3_Link_collision1.STL; collision mesh filename=package://bipedal_robot/meshes/arm3_Link_collision2.STL
- link arm4_Link: mass 0.48 -> 0.39; geometry collision mesh filename=package://bipedal_robot/meshes/arm4_Link_collision1.STL; collision mesh filename=package://bipedal_robot/meshes/arm4_Link_collision2.STL
- link arm5_Link: mass 0.58 -> 0.35; geometry collision mesh filename=package://bipedal_robot/meshes/arm5_Link.STL; visual mesh filename=package://bipedal_robot/meshes/arm5_Link.STL
- link arm6_Link: mass 0.31 -> 0.007
- link arm_base_Link: mass 1.06 -> 1.02
- link gripper1_Link: mass 0.03 -> 0.025
- link gripper2_Link: mass 0.03 -> 0.025
- link transition_Link: mass 0.3 -> 1.117; geometry collision mesh filename=package://bipedal_robot/meshes/transition_Link_collision.STL; visual mesh filename=package://bipedal_robot/meshes/transition_Link.STL
Joints:
- removed joint arm7_Joint
- removed joint gripper_flange_Joint
- added joint antenna_L_Joint: type fixed, parent base_Link, child antenna_L_Link, origin xyz=-0.0025 0.16692 0.211 rpy=0.0 0.0 0.0
- added joint antenna_R_Joint: type fixed, parent base_Link, child antenna_R_Link, origin xyz=-0.0025 -0.16692 0.211 rpy=0.0 0.0 0.0
- added joint camera_mount_Joint: type fixed, parent base_Link, child camera_mount_Link, origin xyz=0.18058 0.0 0.23876 rpy=0.0 0.0 0.0
- added joint radar_Joint: type fixed, parent camera_mount_Link, child radar_Link, origin xyz=0.0 0.0 0.0 rpy=0.0 0.0 0.0
- joint ankle_pitch_L_Joint: limit lower=-1.6231562043547265 upper=1.6231562043547265 effort=60 velocity=22.52 -> lower=-1.6231562043547265 upper=1.6231562043547265 effort=60.0 velocity=22.52; origin xyz=0.004 0.06775 -0.35 rpy=0.0 0.0 0.0 -> xyz=-0.004 -0.06775 -0.35 rpy=0.0 0.0 0.0
- joint ankle_pitch_R_Joint: limit lower=-1.6231562043547265 upper=1.6231562043547265 effort=60 velocity=22.52 -> lower=-1.6231562043547265 upper=1.6231562043547265 effort=60.0 velocity=22.52; origin xyz=0.004 -0.06775 -0.35 rpy=-0.0 0.0 -0.0 -> xyz=-0.004 0.06775 -0.35 rpy=-0.0 0.0 -0.0
- joint arm1_Joint: limit lower=-2.705260340591211 upper=2.705260340591211 effort=100.0 velocity=5.0 -> lower=-2.6179938081783245 upper=2.6179938081783245 effort=100.0 velocity=5.0; origin xyz=0.0 0.0 0.138 rpy=0.0 0.0 0.0 -> xyz=0.0 0.0 0.123 rpy=0.0 0.0 3.1415926
- joint arm2_Joint: limit lower=-1.739918731313147 upper=1.739918731313147 effort=100.0 velocity=5.0 -> lower=0.0 upper=3.141592601229916 effort=100.0 velocity=5.0; origin xyz=0.0 0.0 0.0 rpy=1.5707963 3.1415926 0.0 -> xyz=0.0 0.0 0.0 rpy=-1.5707963 -3.005806 -3.1415926
- joint arm3_Joint: limit lower=-2.7499407694422655 upper=2.7499407694422655 effort=100.0 velocity=5.0 -> lower=-2.967059693483775 upper=0.0 effort=100.0 velocity=5.0; origin xyz=0.0 -0.31 0.0 rpy=-1.5707963 0.0 3.1415926926 -> xyz=0.28503 0.0 0.0 rpy=0.0 0.0 2.8380798
- joint arm4_Joint: limit lower=-1.0100220381291185 upper=2.1399481958702475 effort=100.0 velocity=5.0 -> lower=-1.5533429993683683 upper=1.5533429993683683 effort=100.0 velocity=5.0; origin xyz=0.0 0.0 0.0 rpy=-1.5707963 0.0 3.1415926926 -> xyz=0.27364 0.0 0.0 rpy=0.0 0.0 0.0806342
- joint arm5_Joint: limit lower=-2.7499407694422655 upper=2.7499407694422655 effort=100.0 velocity=5.0 -> lower=-1.5533429993683683 upper=1.5533429993683683 effort=100.0 velocity=5.0; origin xyz=0.0 -0.27001 0.0 rpy=1.5707963 -1.5707963 0.0 -> xyz=0.07466 0.0 0.0 rpy=-1.5707963 1.5707963 0.0
- joint arm6_Joint: limit lower=-0.730071226109228 upper=0.9499827118605135 effort=100.0 velocity=5.0 -> lower=-2.0943951023931953 upper=2.0943951023931953 effort=100.0 velocity=5.0; origin xyz=0.0 0.0 0.0 rpy=1.5707963 -1.5707963 0.0 -> xyz=0.0 -0.035 0.0 rpy=1.5707963 0.0 0.0
- joint gripper1_Joint: limit lower=0.0 upper=0.04991641660703782 effort=10.0 velocity=3.0 -> lower=0.0 upper=0.050000000424915834 effort=10.0 velocity=3.0; origin xyz=0.0 0.0 0.1358 rpy=1.5707963 0.0 3.1415926 -> xyz=0.0 0.0 0.1358 rpy=1.5707963 0.0 0.0
- joint gripper2_Joint: limit lower=-0.04991641660703782 upper=0.0 effort=10.0 velocity=3.0 -> lower=-0.0 upper=0.050000000424915834 effort=10.0 velocity=3.0; origin xyz=0.0 0.0 0.1358 rpy=1.5707963 0.0 0.0 -> xyz=0.0 0.0 0.1358 rpy=1.5707963 0.0 -3.1415926
- joint gripper_base_Joint: origin xyz=0.0 0.0 0.0055 rpy=0.0 0.0 0.0 -> xyz=0.0 0.0 0.0 rpy=0.0 0.0 1.5707963; parent gripper_flange_Link -> arm6_Link
- joint knee_L_Joint: limit lower=-0.2617993877991494 upper=2.6179938779914944 effort=150 velocity=18.3 -> lower=-2.6179938779914944 upper=0.2617993877991494 effort=150.0 velocity=18.3; origin xyz=-0.004 -0.032 -0.2126 rpy=0.0 0.0 0.0 -> xyz=0.004 0.032 -0.2126 rpy=0.0 0.0 0.0
- joint knee_R_Joint: limit lower=-0.2617993877991494 upper=2.6179938779914944 effort=150 velocity=18.3 -> lower=-2.6179938779914944 upper=0.2617993877991494 effort=150.0 velocity=18.3; origin xyz=-0.004 0.032 -0.2126 rpy=-0.0 0.0 -0.0 -> xyz=0.004 -0.032 -0.2126 rpy=-0.0 0.0 -0.0
- joint proximal_pitch_L_Joint: axis 0.0 0.9961947268929313 -0.0871554135479712 -> 0.0 0.996194726892931 -0.0871554135479712; limit lower=-3.141592653589793 upper=2.600540585471551 effort=150 velocity=18.3 -> lower=-3.141592653589793 upper=2.600540585471551 effort=150.0 velocity=18.3
- joint proximal_pitch_R_Joint: axis -0.0 0.9961947268929313 0.0871554135479712 -> -0.0 0.996194726892931 0.0871554135479712; limit lower=-3.141592653589793 upper=2.600540585471551 effort=150 velocity=18.3 -> lower=-3.141592653589793 upper=2.600540585471551 effort=150.0 velocity=18.3
- joint proximal_roll_L_Joint: limit lower=-0.2617993877991494 upper=3.19395248 effort=150 velocity=18.3 -> lower=-0.2617993877991494 upper=3.1939524787897455 effort=150.0 velocity=18.3
- joint proximal_roll_R_Joint: limit lower=-3.19395248 upper=0.2617993877991494 effort=150 velocity=18.3 -> lower=-3.1939524787897455 upper=0.2617993877991494 effort=150.0 velocity=18.3
- joint proximal_yaw_L_Joint: limit lower=-0.5235987755982988 upper=4.625122517784973 effort=60 velocity=22.52 -> lower=-3.6651914291880923 upper=1.4835298641951802 effort=60.0 velocity=22.52
- joint proximal_yaw_R_Joint: limit lower=-4.625122517784973 upper=0.5235987755982988 effort=60 velocity=22.52 -> lower=-1.4835298641951802 upper=3.6651914291880923 effort=60.0 velocity=22.52
- joint transition_Joint: origin xyz=0.0055 0.0 0.26897 rpy=0.0 0.0 3.1415926 -> xyz=0.01 0.0 0.26915 rpy=0.0 0.0 0.0

File: tron2/SFYG_TRON2A/urdf/robot_rl.urdf (robot description, URDF)
Before this commit: robot bipedal_robot, 25 links, 24 joints
Links:
- removed link arm7_Link
- removed link gripper_flange_Link
- removed link limx_imu
- added link antenna_L_Link, mass 0.231; collision mesh filename=../meshes/antenna_L_Link_collision1.STL; collision mesh filename=../meshes/antenna_L_Link_collision2.STL
- added link antenna_R_Link, mass 0.231; collision mesh filename=../meshes/antenna_R_Link_collision1.STL; collision mesh filename=../meshes/antenna_R_Link_collision2.STL
- added link camera_mount_Link, mass 0.381; collision mesh filename=../meshes/camera_mount_Link_collision.STL; visual mesh filename=../meshes/camera_mount_Link.STL
- added link radar_Link, mass 0.394; collision mesh filename=../meshes/radar_Link.STL; visual mesh filename=../meshes/radar_Link.STL
- link ankle_pitch_L_Link: geometry collision box size=0.14 0.06 0.025; collision sphere radius=0.0025
- link ankle_pitch_R_Link: geometry collision box size=0.14 0.06 0.025; collision sphere radius=0.0025
- link arm1_Link: mass 0.77 -> 0.71
- link arm2_Link: mass 0.69 -> 1.16; geometry collision mesh filename=../meshes/arm2_Link_collision1.STL; collision mesh filename=../meshes/arm2_Link_collision2.STL
- link arm3_Link: geometry collision mesh filename=../meshes/arm3_Link_collision1.STL; collision mesh filename=../meshes/arm3_Link_collision2.STL
- link arm4_Link: mass 0.48 -> 0.39; geometry collision mesh filename=../meshes/arm4_Link_collision1.STL; collision mesh filename=../meshes/arm4_Link_collision2.STL
- link arm5_Link: mass 0.58 -> 0.35; geometry collision mesh filename=../meshes/arm5_Link.STL; visual mesh filename=../meshes/arm5_Link.STL
- link arm6_Link: mass 0.31 -> 0.007
- link arm_base_Link: mass 1.06 -> 1.02
- link gripper1_Link: mass 0.03 -> 0.025
- link gripper2_Link: mass 0.03 -> 0.025
- link transition_Link: mass 0.3 -> 1.117; geometry collision mesh filename=../meshes/transition_Link_collision.STL; visual mesh filename=../meshes/transition_Link.STL
Joints:
- removed joint arm7_Joint
- removed joint gripper_flange_Joint
- removed joint limx_imu_joint
- added joint antenna_L_Joint: type fixed, parent base_Link, child antenna_L_Link, origin xyz=-0.0025 0.16692 0.211 rpy=0.0 0.0 0.0
- added joint antenna_R_Joint: type fixed, parent base_Link, child antenna_R_Link, origin xyz=-0.0025 -0.16692 0.211 rpy=0.0 0.0 0.0
- added joint camera_mount_Joint: type fixed, parent base_Link, child camera_mount_Link, origin xyz=0.18058 0.0 0.23876 rpy=0.0 0.0 0.0
- added joint radar_Joint: type fixed, parent camera_mount_Link, child radar_Link, origin xyz=0.0 0.0 0.0 rpy=0.0 0.0 0.0
- joint ankle_pitch_L_Joint: limit lower=-1.6231562043547265 upper=1.6231562043547265 effort=60 velocity=22.52 -> lower=-1.6231562043547265 upper=1.6231562043547265 effort=60.0 velocity=22.52; origin xyz=0.004 0.06775 -0.35 rpy=0.0 0.0 0.0 -> xyz=-0.004 -0.06775 -0.35 rpy=0.0 0.0 0.0
- joint ankle_pitch_R_Joint: limit lower=-1.6231562043547265 upper=1.6231562043547265 effort=60 velocity=22.52 -> lower=-1.6231562043547265 upper=1.6231562043547265 effort=60.0 velocity=22.52; origin xyz=0.004 -0.06775 -0.35 rpy=-0.0 0.0 -0.0 -> xyz=-0.004 0.06775 -0.35 rpy=-0.0 0.0 -0.0
- joint arm1_Joint: limit lower=-2.705260340591211 upper=2.705260340591211 effort=100.0 velocity=5.0 -> lower=-2.6179938081783245 upper=2.6179938081783245 effort=100.0 velocity=5.0; origin xyz=0.0 0.0 0.138 rpy=0.0 0.0 0.0 -> xyz=0.0 0.0 0.123 rpy=0.0 0.0 3.1415926
- joint arm2_Joint: limit lower=-1.739918731313147 upper=1.739918731313147 effort=100.0 velocity=5.0 -> lower=0.0 upper=3.141592601229916 effort=100.0 velocity=5.0; origin xyz=0.0 0.0 0.0 rpy=1.5707963 3.1415926 0.0 -> xyz=0.0 0.0 0.0 rpy=-1.5707963 -3.005806 -3.1415926
- joint arm3_Joint: limit lower=-2.7499407694422655 upper=2.7499407694422655 effort=100.0 velocity=5.0 -> lower=-2.967059693483775 upper=0.0 effort=100.0 velocity=5.0; origin xyz=0.0 -0.31 0.0 rpy=-1.5707963 0.0 3.1415926926 -> xyz=0.28503 0.0 0.0 rpy=0.0 0.0 2.8380798
- joint arm4_Joint: limit lower=-1.0100220381291185 upper=2.1399481958702475 effort=100.0 velocity=5.0 -> lower=-1.5533429993683683 upper=1.5533429993683683 effort=100.0 velocity=5.0; origin xyz=0.0 0.0 0.0 rpy=-1.5707963 0.0 3.1415926926 -> xyz=0.27364 0.0 0.0 rpy=0.0 0.0 0.0806342
- joint arm5_Joint: limit lower=-2.7499407694422655 upper=2.7499407694422655 effort=100.0 velocity=5.0 -> lower=-1.5533429993683683 upper=1.5533429993683683 effort=100.0 velocity=5.0; origin xyz=0.0 -0.27001 0.0 rpy=1.5707963 -1.5707963 0.0 -> xyz=0.07466 0.0 0.0 rpy=-1.5707963 1.5707963 0.0
- joint arm6_Joint: limit lower=-0.730071226109228 upper=0.9499827118605135 effort=100.0 velocity=5.0 -> lower=-2.0943951023931953 upper=2.0943951023931953 effort=100.0 velocity=5.0; origin xyz=0.0 0.0 0.0 rpy=1.5707963 -1.5707963 0.0 -> xyz=0.0 -0.035 0.0 rpy=1.5707963 0.0 0.0
- joint gripper1_Joint: limit lower=0.0 upper=0.04991641660703782 effort=10.0 velocity=3.0 -> lower=0.0 upper=0.050000000424915834 effort=10.0 velocity=3.0; origin xyz=0.0 0.0 0.1358 rpy=1.5707963 0.0 3.1415926 -> xyz=0.0 0.0 0.1358 rpy=1.5707963 0.0 0.0
- joint gripper2_Joint: limit lower=-0.04991641660703782 upper=0.0 effort=10.0 velocity=3.0 -> lower=-0.050000000424915834 upper=0.0 effort=10.0 velocity=3.0; origin xyz=0.0 0.0 0.1358 rpy=1.5707963 0.0 0.0 -> xyz=0.0 0.0 0.1358 rpy=1.5707963 0.0 -3.1415926
- joint gripper_base_Joint: origin xyz=0.0 0.0 0.0055 rpy=0.0 0.0 0.0 -> xyz=0.0 0.0 0.0 rpy=0.0 0.0 1.5707963; parent gripper_flange_Link -> arm6_Link
- joint knee_L_Joint: limit lower=-0.2617993877991494 upper=2.6179938779914944 effort=150 velocity=18.3 -> lower=-2.6179938779914944 upper=0.2617993877991494 effort=150.0 velocity=18.3; origin xyz=-0.004 -0.032 -0.2126 rpy=0.0 0.0 0.0 -> xyz=0.004 0.032 -0.2126 rpy=0.0 0.0 0.0
- joint knee_R_Joint: limit lower=-0.2617993877991494 upper=2.6179938779914944 effort=150 velocity=18.3 -> lower=-2.6179938779914944 upper=0.2617993877991494 effort=150.0 velocity=18.3; origin xyz=-0.004 0.032 -0.2126 rpy=-0.0 0.0 -0.0 -> xyz=0.004 -0.032 -0.2126 rpy=-0.0 0.0 -0.0
- joint proximal_pitch_L_Joint: axis 0.0 0.9961947268929313 -0.0871554135479712 -> 0.0 0.996194726892931 -0.0871554135479712; limit lower=-3.141592653589793 upper=2.600540585471551 effort=150 velocity=18.3 -> lower=-3.141592653589793 upper=2.600540585471551 effort=150.0 velocity=18.3
- joint proximal_pitch_R_Joint: axis -0.0 0.9961947268929313 0.0871554135479712 -> -0.0 0.996194726892931 0.0871554135479712; limit lower=-3.141592653589793 upper=2.600540585471551 effort=150 velocity=18.3 -> lower=-3.141592653589793 upper=2.600540585471551 effort=150.0 velocity=18.3
- joint proximal_roll_L_Joint: limit lower=-0.2617993877991494 upper=3.19395248 effort=150 velocity=18.3 -> lower=-0.2617993877991494 upper=3.1939524787897455 effort=150.0 velocity=18.3
- joint proximal_roll_R_Joint: limit lower=-3.19395248 upper=0.2617993877991494 effort=150 velocity=18.3 -> lower=-3.1939524787897455 upper=0.2617993877991494 effort=150.0 velocity=18.3
- joint proximal_yaw_L_Joint: limit lower=-0.5235987755982988 upper=4.625122517784973 effort=60 velocity=22.52 -> lower=-3.6651914291880923 upper=1.4835298641951802 effort=60.0 velocity=22.52
- joint proximal_yaw_R_Joint: limit lower=-4.625122517784973 upper=0.5235987755982988 effort=60 velocity=22.52 -> lower=-1.4835298641951802 upper=3.6651914291880923 effort=60.0 velocity=22.52
- joint transition_Joint: origin xyz=0.0055 0.0 0.26897 rpy=0.0 0.0 3.1415926 -> xyz=0.01 0.0 0.26915 rpy=0.0 0.0 0.0

Commit message: fix(SFYG&WFYG): prevent self collision between arm5 and gripper_base

File: tron2/SFYG_TRON2A/urdf/robot.urdf (robot description, URDF)
Before this commit: robot bipedal_robot, 28 links, 27 joints
Links:
- link arm6_Link: geometry visual mesh filename=package://bipedal_robot/meshes/arm6_Link.STL

File: tron2/SFYG_TRON2A/urdf/robot_rl.urdf (robot description, URDF)
Before this commit: robot bipedal_robot, 29 links, 28 joints
Links:
- link arm6_Link: geometry visual mesh filename=../meshes/arm6_Link.STL

File: tron2/WFYG_TRON2A/urdf/robot.urdf (robot description, URDF)
Before this commit: robot bipedal_robot, 28 links, 27 joints
Links:
- link arm6_Link: geometry visual mesh filename=package://bipedal_robot/meshes/arm6_Link.STL

File: tron2/WFYG_TRON2A/urdf/robot_rl.urdf (robot description, URDF)
Before this commit: robot bipedal_robot, 29 links, 28 joints
Links:
- link arm6_Link: geometry visual mesh filename=../meshes/arm6_Link.STL
