Commit message: feat: regenerate SFYG_TRON2A

File: tron2/SFYG_TRON2A/urdf/robot_rl.urdf (robot description, URDF)
Before this commit: robot bipedal_robot, 26 links, 25 joints
Links:
- added link base_imu, mass 0.01
Joints:
- added joint base_imu_Joint: type fixed, parent base_Link, child base_imu, origin xyz=0.0 0.0 0.0 rpy=0.0 0.0 0.0

Commit message: feat(SFYG&WFYG): add gripper pick link in USD

File: tron2/SFYG_TRON2A/urdf/robot_rl.urdf (robot description, URDF)
Before this commit: robot bipedal_robot, 29 links, 28 joints
Links:
- added link gripper_pick, mass 0.001; visual box size=0.0025 0.0025 0.0025
Joints:
- added joint gripper_pick_Joint: type fixed, parent gripper_base_Link, child gripper_pick, origin xyz=0.00118 0.0 0.13544 rpy=0.0 -1.5707963 0.0

File: tron2/WFYG_TRON2A/urdf/robot_rl.urdf (robot description, URDF)
Before this commit: robot bipedal_robot, 29 links, 28 joints
Links:
- added link gripper_pick, mass 0.001; visual box size=0.0025 0.0025 0.0025
Joints:
- added joint gripper_pick_Joint: type fixed, parent gripper_base_Link, child gripper_pick, origin xyz=0.00118 0.0 0.13544 rpy=0.0 -1.5707963 0.0
