Commit message: feat: 为WF_TRON2A在Gazebo和MuJoco下增加深度相机支持，SF_TRON2A增加MuJoco深度相机支持

File: tron2/WF_TRON2A/xacro/macros.xacro (robot description, xacro)
@@ -41,4 +41,71 @@
       </plugin>
     </gazebo>
+    <!-- D435 Camera ROS1 Plugin: split into two sensors instead of using
+         libgazebo_ros_openni_kinect.so. The openni_kinect plugin deadlocks
+         with gazebo_ros_control on Load() and prevents Tron2HWSim::initSim
+         from being called. -->
+    <gazebo reference="d435_Link">
+      <sensor type="camera" name="d435_color_sensor">
+        <pose>0 0 0 0 0 0</pose>
+        <update_rate>60</update_rate>
+        <visualize>false</visualize>
+        <camera>
+          <horizontal_fov>1.5177</horizontal_fov>
+          <image>
+            <format>B8G8R8</format>
+            <width>64</width>
+            <height>48</height>
+          </image>
+          <clip>
+            <near>0.1</near>
+            <far>1.8</far>
+          </clip>
+        </camera>
+        <plugin name="d435_color_controller" filename="libgazebo_ros_camera.so">
+          <robotNamespace>d435</robotNamespace>
+          <cameraName>color</cameraName>
+          <imageTopicName>image_raw</imageTopicName>
+          <cameraInfoTopicName>camera_info</cameraInfoTopicName>
+          <frameName>d435_optical_frame</frameName>
+        </plugin>
+      </sensor>
+      <sensor type="depth" name="d435_depth_sensor">
+        <pose>0 0 0 0 0 0</pose>
+        <update_rate>60</update_rate>
+        <visualize>false</visualize>
+        <camera>
+          <horizontal_fov>1.5177</horizontal_fov>
+          <image>
+            <format>R8G8B8</format>
+            <width>64</width>
+            <height>48</height>
+          </image>
+          <clip>
+            <near>0.1</near>
+            <far>1.8</far>
+          </clip>
+        </camera>
+        <plugin name="d435_depth_controller" filename="libgazebo_ros_depth_camera.so">
+          <robotNamespace>d435</robotNamespace>
+          <!-- cameraName must differ from the color sensor; otherwise both
+               plugins share the same set_camera_info / set_parameters
+               services and Gazebo logs "Tried to advertise a service that
+               is already advertised" on the second one. -->
+          <cameraName>depth</cameraName>
+          <!-- imageTopicName / cameraInfoTopicName publish the IR/grayscale
+               frame from libgazebo_ros_depth_camera.so. Route them under
+               infra/ so they don't collide with depthImageTopicName /
+               depthImageCameraInfoTopicName (the real depth stream). -->
+          <imageTopicName>infra/image_raw</imageTopicName>
+          <cameraInfoTopicName>infra/camera_info</cameraInfoTopicName>
+          <depthImageTopicName>image_raw</depthImageTopicName>
+          <depthImageCameraInfoTopicName>camera_info</depthImageCameraInfoTopicName>
+          <pointCloudTopicName>points</pointCloudTopicName>
+          <frameName>d435_optical_frame</frameName>
+          <pointCloudCutoff>0.1</pointCloudCutoff>
+          <pointCloudCutoffMax>1.8</pointCloudCutoffMax>
+        </plugin>
+      </sensor>
+    </gazebo>
     <!-- Transmissions (ROS1) -->
     <transmission name="proximal_pitch_L_Joint_trans">
@@ -278,4 +345,33 @@
       </plugin>
     </gazebo>
+    <!-- D435 Camera ROS2 Plugin -->
+    <gazebo reference="d435_Link">
+      <sensor type="depth" name="d435_camera_sensor">
+        <pose>0 0 0 0 0 0</pose>
+        <update_rate>60</update_rate>
+        <visualize>false</visualize>
+        <camera>
+          <horizontal_fov>1.5177</horizontal_fov>
+          <image>
+            <format>B8G8R8</format>
+            <width>64</width>
+            <height>48</height>
+          </image>
+          <clip>
+            <near>0.1</near>
+            <far>1.8</far>
+          </clip>
+        </camera>
+        <plugin name="camera_controller" filename="libgazebo_ros_camera.so">
+          <ros>
+            <namespace>d435</namespace>
+          </ros>
+          <camera_name>d435_camera</camera_name>
+          <frame_name>d435_optical_frame</frame_name>
+          <min_depth>0.1</min_depth>
+          <max_depth>1.8</max_depth>
+        </plugin>
+      </sensor>
+    </gazebo>
   </xacro:macro>
 </robot>

File: tron2/WF_TRON2A/xacro/robot.urdf.xacro (robot description, xacro)
@@ -432,4 +432,27 @@
     <kd value="100.0" />
   </gazebo>
+  <!-- D435 Camera Links -->
+  <link name="d435_Link">
+    <visual>
+      <origin rpy="1.5707963267948966 0 1.5707963267948966" xyz="0.0 -0.0 0" />
+      <geometry>
+        <box size="0.01 0.01 0.001" />
+      </geometry>
+      <material name="camera_red">
+        <color rgba="1.0 0.0 0.0 1.0" />
+      </material>
+    </visual>
+  </link>
+  <joint name="d435_joint" type="fixed">
+    <origin rpy="0 1.063778179 0" xyz="0.12213 0.01759 0.00599" />
+    <parent link="base_imu" />
+    <child link="d435_Link" />
+  </joint>
+  <joint name="d435_optical_joint" type="fixed">
+    <origin rpy="-1.5707963267948966 0 -1.5707963267948966" xyz="0 0 0" />
+    <parent link="d435_Link" />
+    <child link="d435_optical_frame" />
+  </joint>
+  <link name="d435_optical_frame" />
   <!-- Conditional ROS version -->
   <xacro:if value="${ros_version == 1}">
