Commit message: fix: fixed DACH_TRON2A joint efforts and armatures

File: tron2/DACH_TRON2A/urdf/robot.urdf (robot description, URDF)
Before this commit: robot bipedal_robot, 25 links, 24 joints
Joints:
- joint head_pitch_Joint: limit lower=-0.7853981633974483 upper=1.0471975511965976 effort=0.0 velocity=0.0 -> lower=-0.7853981633974483 upper=1.0471975511965976 effort=20.0 velocity=17.8
- joint head_yaw_Joint: limit lower=-1.5707963267948966 upper=1.5707963267948966 effort=0.0 velocity=0.0 -> lower=-1.5707963267948966 upper=1.5707963267948966 effort=20.0 velocity=17.8
- joint proximal_pitch_L_Joint: limit lower=-3.141592653589793 upper=2.600540585471551 effort=200.0 velocity=18.3 -> lower=-3.141592653589793 upper=2.600540585471551 effort=150.0 velocity=18.3
- joint proximal_pitch_R_Joint: limit lower=-3.141592653589793 upper=2.600540585471551 effort=200.0 velocity=18.3 -> lower=-3.141592653589793 upper=2.600540585471551 effort=150.0 velocity=18.3
- joint proximal_roll_L_Joint: limit lower=-0.2617993877991494 upper=3.193952531149623 effort=200.0 velocity=18.3 -> lower=-0.2617993877991494 upper=3.193952531149623 effort=150.0 velocity=18.3
- joint proximal_roll_R_Joint: limit lower=-3.193952531149623 upper=0.2617993877991494 effort=200.0 velocity=18.3 -> lower=-3.193952531149623 upper=0.2617993877991494 effort=150.0 velocity=18.3
- joint proximal_yaw_L_Joint: limit lower=-3.6651914291880923 upper=1.4835298641951802 effort=70.0 velocity=22.52 -> lower=-3.6651914291880923 upper=1.4835298641951802 effort=60.0 velocity=22.52
- joint proximal_yaw_R_Joint: limit lower=-1.4835298641951802 upper=3.6651914291880923 effort=70.0 velocity=22.52 -> lower=-1.4835298641951802 upper=3.6651914291880923 effort=60.0 velocity=22.52

File: tron2/DACH_TRON2A/urdf/robot_rl.urdf (robot description, URDF)
Before this commit: robot bipedal_robot, 25 links, 24 joints
Joints:
- joint head_pitch_Joint: limit lower=-0.7853981633974483 upper=1.0471975511965976 effort=0.0 velocity=0.0 -> lower=-0.7853981633974483 upper=1.0471975511965976 effort=20.0 velocity=17.8
- joint head_yaw_Joint: limit lower=-1.5707963267948966 upper=1.5707963267948966 effort=0.0 velocity=0.0 -> lower=-1.5707963267948966 upper=1.5707963267948966 effort=20.0 velocity=17.8
- joint proximal_pitch_L_Joint: limit lower=-3.141592653589793 upper=2.600540585471551 effort=200.0 velocity=18.3 -> lower=-3.141592653589793 upper=2.600540585471551 effort=150.0 velocity=18.3
- joint proximal_pitch_R_Joint: limit lower=-3.141592653589793 upper=2.600540585471551 effort=200.0 velocity=18.3 -> lower=-3.141592653589793 upper=2.600540585471551 effort=150.0 velocity=18.3
- joint proximal_roll_L_Joint: limit lower=-0.2617993877991494 upper=3.193952531149623 effort=200.0 velocity=18.3 -> lower=-0.2617993877991494 upper=3.193952531149623 effort=150.0 velocity=18.3
- joint proximal_roll_R_Joint: limit lower=-3.193952531149623 upper=0.2617993877991494 effort=200.0 velocity=18.3 -> lower=-3.193952531149623 upper=0.2617993877991494 effort=150.0 velocity=18.3
- joint proximal_yaw_L_Joint: limit lower=-3.6651914291880923 upper=1.4835298641951802 effort=70.0 velocity=22.52 -> lower=-3.6651914291880923 upper=1.4835298641951802 effort=60.0 velocity=22.52
- joint proximal_yaw_R_Joint: limit lower=-1.4835298641951802 upper=3.6651914291880923 effort=70.0 velocity=22.52 -> lower=-1.4835298641951802 upper=3.6651914291880923 effort=60.0 velocity=22.52

Commit message: Feat: 创建DA/DACH_TRON2A xacro文件，并修复urdf中的package方法的mesh解析路径

File: tron2/DACH_TRON2A/urdf/robot.urdf (robot description, URDF)
Before this commit: robot bipedal_robot, 25 links, 24 joints
Links:
- link base_2_Link: geometry collision box size=0.118 0.085 0.98; visual mesh filename=package://robot_description/tron2/DACH_TRON2A/meshes/base_2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
- link base_3_Link: geometry collision mesh filename=package://robot_description/tron2/DACH_TRON2A/meshes/base_3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; visual mesh filename=package://robot_description/tron2/DACH_TRON2A/meshes/base_3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
- link base_Link: geometry collision mesh filename=package://robot_description/tron2/DACH_TRON2A/meshes/base_L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; visual mesh filename=package://robot_description/tron2/DACH_TRON2A/meshes/base_L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
- link elbow_L_Link: geometry collision mesh filename=package://robot_description/tron2/DACH_TRON2A/meshes/elbow_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; visual mesh filename=package://robot_description/tron2/DACH_TRON2A/meshes/elbow_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
- link elbow_R_Link: geometry collision mesh filename=package://robot_description/tron2/DACH_TRON2A/meshes/elbow_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; visual mesh filename=package://robot_description/tron2/DACH_TRON2A/meshes/elbow_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
- link grasper_L_Link: geometry collision mesh filename=package://robot_description/tron2/DACH_TRON2A/meshes/graspe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; visual mesh filename=package://robot_description/tron2/DACH_TRON2A/meshes/graspe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
- link grasper_R_Link: geometry collision mesh filename=package://robot_description/tron2/DACH_TRON2A/meshes/graspe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; visual mesh filename=package://robot_description/tron2/DACH_TRON2A/meshes/graspe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
- link head_base_Link: geometry visual mesh filename=package://robot_description/tron2/DACH_TRON2A/meshes/head_b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
- link head_pitch_Link: geometry collision mesh filename=package://robot_description/tron2/DACH_TRON2A/meshes/head_p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; visual mesh filename=package://robot_description/tron2/DACH_TRON2A/meshes/head_p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
- link head_yaw_Link: geometry collision mesh filename=package://robot_description/tron2/DACH_TRON2A/meshes/head_y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; visual mesh filename=package://robot_description/tron2/DACH_TRON2A/meshes/head_y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
- link proximal_pitch_L_Link: geometry collision mesh filename=package://robot_description/tron2/DACH_TRON2A/meshes/proxim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; visual mesh filename=package://robot_description/tron2/DACH_TRON2A/meshes/proxim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
- link proximal_pitch_R_Link: geometry collision mesh filename=package://robot_description/tron2/DACH_TRON2A/meshes/proxim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; visual mesh filename=package://robot_description/tron2/DACH_TRON2A/meshes/proxim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
- link proximal_roll_L_Link: geometry collision mesh filename=package://robot_description/tron2/DACH_TRON2A/meshes/proxim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; visual mesh filename=package://robot_description/tron2/DACH_TRON2A/meshes/proxim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
- link proximal_roll_R_Link: geometry collision mesh filename=package://robot_description/tron2/DACH_TRON2A/meshes/proxim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; visual mesh filename=package://robot_description/tron2/DACH_TRON2A/meshes/proxim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
- link proximal_yaw_L_Link: geometry collision mesh filename=package://robot_description/tron2/DACH_TRON2A/meshes/proxim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; visual mesh filename=package://robot_description/tron2/DACH_TRON2A/meshes/proxim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
- link proximal_yaw_R_Link: geometry collision mesh filename=package://robot_description/tron2/DACH_TRON2A/meshes/proxim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; visual mesh filename=package://robot_description/tron2/DACH_TRON2A/meshes/proxim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
- link wrist_pitch_L_Link: geometry collision mesh filename=package://robot_description/tron2/DACH_TRON2A/meshes/wrist_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; visual mesh filename=package://robot_description/tron2/DACH_TRON2A/meshes/wrist_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
- link wrist_pitch_R_Link: geometry collision mesh filename=package://robot_description/tron2/DACH_TRON2A/meshes/wrist_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; visual mesh filename=package://robot_description/tron2/DACH_TRON2A/meshes/wrist_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
- link wrist_roll_L_Link: geometry collision mesh filename=package://robot_description/tron2/DACH_TRON2A/meshes/wrist_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; visual mesh filename=package://robot_description/tron2/DACH_TRON2A/meshes/wrist_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
- link wrist_roll_R_Link: geometry collision mesh filename=package://robot_description/tron2/DACH_TRON2A/meshes/wrist_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; visual mesh filename=package://robot_description/tron2/DACH_TRON2A/meshes/wrist_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
- link wrist_yaw_L_Link: geometry collision mesh filename=package://robot_description/tron2/DACH_TRON2A/meshes/wrist_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; visual mesh filename=package://robot_description/tron2/DACH_TRON2A/meshes/wrist_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
- link wrist_yaw_R_Link: geometry collision mesh filename=package://robot_description/tron2/DACH_TRON2A/meshes/wrist_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; visual mesh filename=package://robot_description/tron2/DACH_TRON2A/meshes/wrist_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

File: tron2/DA_TRON2A/urdf/robot.urdf (robot description, URDF)
Before this commit: robot bipedal_robot, 22 links, 21 joints
Links:
- link base_2_Link: geometry collision box size=0.118 0.085 0.98; visual mesh filename=package://robot_description/tron2/DA_TRON2A/meshes/base_2_L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
- link base_3_Link: geometry collision mesh filename=package://robot_description/tron2/DA_TRON2A/meshes/base_3_L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; visual mesh filename=package://robot_description/tron2/DA_TRON2A/meshes/base_3_L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
- link base_Link: geometry collision mesh filename=package://robot_description/tron2/DA_TRON2A/meshes/base_Lin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; visual mesh filename=package://robot_description/tron2/DA_TRON2A/meshes/base_Lin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
- link elbow_L_Link: geometry collision mesh filename=package://robot_description/tron2/DA_TRON2A/meshes/elbow_L_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; visual mesh filename=package://robot_description/tron2/DA_TRON2A/meshes/elbow_L_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
- link elbow_R_Link: geometry collision mesh filename=package://robot_description/tron2/DA_TRON2A/meshes/elbow_R_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; visual mesh filename=package://robot_description/tron2/DA_TRON2A/meshes/elbow_R_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
- link grasper_L_Link: geometry collision mesh filename=package://robot_description/tron2/DA_TRON2A/meshes/grasper_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; visual mesh filename=package://robot_description/tron2/DA_TRON2A/meshes/grasper_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
- link grasper_R_Link: geometry collision mesh filename=package://robot_description/tron2/DA_TRON2A/meshes/grasper_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; visual mesh filename=package://robot_description/tron2/DA_TRON2A/meshes/grasper_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
- link proximal_pitch_L_Link: geometry collision mesh filename=package://robot_description/tron2/DA_TRON2A/meshes/proximal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; visual mesh filename=package://robot_description/tron2/DA_TRON2A/meshes/proximal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
- link proximal_pitch_R_Link: geometry collision mesh filename=package://robot_description/tron2/DA_TRON2A/meshes/proximal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; visual mesh filename=package://robot_description/tron2/DA_TRON2A/meshes/proximal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
- link proximal_roll_L_Link: geometry collision mesh filename=package://robot_description/tron2/DA_TRON2A/meshes/proximal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; visual mesh filename=package://robot_description/tron2/DA_TRON2A/meshes/proximal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
- link proximal_roll_R_Link: geometry collision mesh filename=package://robot_description/tron2/DA_TRON2A/meshes/proximal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; visual mesh filename=package://robot_description/tron2/DA_TRON2A/meshes/proximal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
- link proximal_yaw_L_Link: geometry collision mesh filename=package://robot_description/tron2/DA_TRON2A/meshes/proximal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; visual mesh filename=package://robot_description/tron2/DA_TRON2A/meshes/proximal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
- link proximal_yaw_R_Link: geometry collision mesh filename=package://robot_description/tron2/DA_TRON2A/meshes/proximal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; visual mesh filename=package://robot_description/tron2/DA_TRON2A/meshes/proximal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
- link wrist_pitch_L_Link: geometry collision mesh filename=package://robot_description/tron2/DA_TRON2A/meshes/wrist_pi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; visual mesh filename=package://robot_description/tron2/DA_TRON2A/meshes/wrist_pi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
- link wrist_pitch_R_Link: geometry collision mesh filename=package://robot_description/tron2/DA_TRON2A/meshes/wrist_pi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; visual mesh filename=package://robot_description/tron2/DA_TRON2A/meshes/wrist_pi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
- link wrist_roll_L_Link: geometry collision mesh filename=package://robot_description/tron2/DA_TRON2A/meshes/wrist_ro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; visual mesh filename=package://robot_description/tron2/DA_TRON2A/meshes/wrist_ro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
- link wrist_roll_R_Link: geometry collision mesh filename=package://robot_description/tron2/DA_TRON2A/meshes/wrist_ro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; visual mesh filename=package://robot_description/tron2/DA_TRON2A/meshes/wrist_ro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
- link wrist_yaw_L_Link: geometry collision mesh filename=package://robot_description/tron2/DA_TRON2A/meshes/wrist_ya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; visual mesh filename=package://robot_description/tron2/DA_TRON2A/meshes/wrist_ya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
- link wrist_yaw_R_Link: geometry collision mesh filename=package://robot_description/tron2/DA_TRON2A/meshes/wrist_ya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; visual mesh filename=package://robot_description/tron2/DA_TRON2A/meshes/wrist_ya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
