Commit message: chore(TRON2A): sync latest internal fixes from develop
- DACH_TRON2A: align robot_grasper mass/inertia with robot.urdf/xml
- SFYG_TRON2A / WFYG_TRON2A: switch to updated sensor-mast meshes
  (rename *_collision1/2 -> *_collision_1/2, refreshed antenna/camera/
  radar/transition STL geometry) and regenerate URDF/xacro/MJCF/USD
- DASF_TRON2A / DASF2_TRON2A: refreshed USD physics/sensor configuration

Note: the newly added TRON2B robot family (21 commits on internal
develop) is intentionally excluded from this push. ASSETS.md does not
yet document its license/provenance status, which per this repo's own
policy blocks public release; two of its USD files also exceed
GitHub's 100MB limit. TRON2B remains on the internal develop branch
pending review.

File: tron2a/DACH_TRON2A/urdf/robot_grasper.urdf (robot description, URDF)
Before this commit: robot robot_description/tron2/DACH_TRON2A, 45 links, 44 joints
Links:
- link grasper_base_L_Link: mass 0.04219468 -> 0.49169168
- link grasper_base_R_Link: mass 0.04219468 -> 0.49169168

File: tron2a/SFYG_TRON2A/urdf/robot.urdf (robot description, URDF)
Before this commit: robot bipedal_robot, 29 links, 28 joints
Links:
- link antenna_L_Link: mass 0.231 -> 0.073; geometry collision mesh filename=package://bipedal_robot/meshes/antenna_L_Link_collision_1.S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; collision mesh filename=package://bipedal_robot/meshes/antenna_L_Link_collision_2.S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
- link antenna_R_Link: mass 0.231 -> 0.073; geometry collision mesh filename=package://bipedal_robot/meshes/antenna_R_Link_collision_1.S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; collision mesh filename=package://bipedal_robot/meshes/antenna_R_Link_collision_2.S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
- link camera_mount_Link: mass 0.381 -> 0.288; geometry collision mesh filename=package://bipedal_robot/meshes/camera_mount_Link.STL; visual mesh filename=package://bipedal_robot/meshes/camera_mount_Link.STL
- link radar_Link: mass 0.394 -> 0.406
- link transition_Link: geometry collision mesh filename=package://bipedal_robot/meshes/transition_Link_collision_1.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; collision mesh filename=package://bipedal_robot/meshes/transition_Link_collision_2.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
Joints:
- joint antenna_L_Joint: origin xyz=-0.0025 0.16692 0.211 rpy=0.0 0.0 0.0 -> xyz=-0.04365 0.1535 0.23765 rpy=0.0 0.0 0.0
- joint antenna_R_Joint: origin xyz=-0.0025 -0.16692 0.211 rpy=0.0 0.0 0.0 -> xyz=-0.04365 -0.1535 0.23765 rpy=0.0 0.0 0.0
- joint arm_base_Joint: origin xyz=0.006 0.0 0.0 rpy=0.0 0.0 0.0 -> xyz=0.0 0.0 0.0 rpy=0.0 0.0 0.0
- joint radar_Joint: origin xyz=0.0 0.0 0.0 rpy=0.0 0.0 0.0 -> xyz=0.18058 0.0 0.23876 rpy=0.0 0.0 0.0; parent camera_mount_Link -> base_Link

File: tron2a/SFYG_TRON2A/urdf/robot_rl.urdf (robot description, URDF)
Before this commit: robot bipedal_robot, 30 links, 29 joints
Links:
- link antenna_L_Link: mass 0.231 -> 0.073; geometry collision mesh filename=../meshes/antenna_L_Link_collision_1.STL; collision mesh filename=../meshes/antenna_L_Link_collision_2.STL
- link antenna_R_Link: mass 0.231 -> 0.073; geometry collision mesh filename=../meshes/antenna_R_Link_collision_1.STL; collision mesh filename=../meshes/antenna_R_Link_collision_2.STL
- link camera_mount_Link: mass 0.381 -> 0.288; geometry collision mesh filename=../meshes/camera_mount_Link.STL; visual mesh filename=../meshes/camera_mount_Link.STL
- link radar_Link: mass 0.394 -> 0.406
- link transition_Link: geometry collision mesh filename=../meshes/transition_Link_collision_1.STL; collision mesh filename=../meshes/transition_Link_collision_2.STL
Joints:
- joint antenna_L_Joint: origin xyz=-0.0025 0.16692 0.211 rpy=0.0 0.0 0.0 -> xyz=-0.04365 0.1535 0.23765 rpy=0.0 0.0 0.0
- joint antenna_R_Joint: origin xyz=-0.0025 -0.16692 0.211 rpy=0.0 0.0 0.0 -> xyz=-0.04365 -0.1535 0.23765 rpy=0.0 0.0 0.0
- joint arm_base_Joint: origin xyz=0.006 0.0 0.0 rpy=0.0 0.0 0.0 -> xyz=0.0 0.0 0.0 rpy=0.0 0.0 0.0
- joint radar_Joint: origin xyz=0.0 0.0 0.0 rpy=0.0 0.0 0.0 -> xyz=0.18058 0.0 0.23876 rpy=0.0 0.0 0.0; parent camera_mount_Link -> base_Link

File: tron2a/SFYG_TRON2A/xacro/robot.urdf.xacro (robot description, xacro)
@@ -313,8 +313,8 @@
   <link name="transition_Link">
     <inertial>
-      <origin xyz="-0.111727 0.000317 0.014516" rpy="0 0 0" />
+      <origin xyz="-0.109866 -0.002238 0.012131" rpy="0 0 0" />
       <mass value="1.117" />
-      <inertia ixx="0.002739303" ixy="6.6427e-05" ixz="0.000914255"
-        iyy="0.006871988" iyz="-2.0809e-05" izz="0.007888835" />
+      <inertia ixx="0.002748897" ixy="-0.000172411" ixz="0.00101041"
+        iyy="0.007134041" iyz="3.8511e-05" izz="0.008548272" />
     </inertial>
     <visual>
@@ -328,5 +328,11 @@
       <origin xyz="0 0 0" rpy="0 0 0" />
       <geometry>
-        <mesh filename="package://robot_description/tron2/SFYG_TRON2A/meshes/transition_Link_collision.STL" />
+        <mesh filename="package://robot_description/tron2/SFYG_TRON2A/meshes/transition_Link_collision_1.STL" />
+      </geometry>
+    </collision>
+    <collision>
+      <origin xyz="0 0 0" rpy="0 0 0" />
+      <geometry>
+        <mesh filename="package://robot_description/tron2/SFYG_TRON2A/meshes/transition_Link_collision_2.STL" />
       </geometry>
     </collision>
@@ -568,8 +574,8 @@
   <link name="antenna_L_Link">
     <inertial>
-      <origin xyz="-2.7e-05 -0.028426 0.013784" rpy="0 0 0" />
-      <mass value="0.231" />
-      <inertia ixx="0.000424493" ixy="-1.15e-07" ixz="-1.18e-07"
-        iyy="0.000169977" iyz="3.0807e-05" izz="0.00039175" />
+      <origin xyz="0.0 -0.025937 0.00756" rpy="0 0 0" />
+      <mass value="0.073" />
+      <inertia ixx="9.4062e-05" ixy="-1e-09" ixz="0.0"
+        iyy="2.8597e-05" iyz="-2.91e-07" izz="7.7585e-05" />
     </inertial>
     <visual>
@@ -583,11 +589,11 @@
       <origin xyz="0 0 0" rpy="0 0 0" />
       <geometry>
-        <mesh filename="package://robot_description/tron2/SFYG_TRON2A/meshes/antenna_L_Link_collision1.STL" />
-      </geometry>
-    </collision>
-    <collision>
-      <origin xyz="0 0 0" rpy="0 0 0" />
-      <geometry>
-        <mesh filename="package://robot_description/tron2/SFYG_TRON2A/meshes/antenna_L_Link_collision2.STL" />
+        <mesh filename="package://robot_description/tron2/SFYG_TRON2A/meshes/antenna_L_Link_collision_1.STL" />
+      </geometry>
+    </collision>
+    <collision>
+      <origin xyz="0 0 0" rpy="0 0 0" />
+      <geometry>
+        <mesh filename="package://robot_description/tron2/SFYG_TRON2A/meshes/antenna_L_Link_collision_2.STL" />
       </geometry>
     </collision>
@@ -595,8 +601,8 @@
   <link name="antenna_R_Link">
     <inertial>
-      <origin xyz="2.7e-05 0.028426 0.013784" rpy="0 0 0" />
-      <mass value="0.231" />
-      <inertia ixx="0.000424493" ixy="-1.15e-07" ixz="1.17e-07"
-        iyy="0.000169977" iyz="-3.0808e-05" izz="0.000391749" />
+      <origin xyz="0.0 0.025937 0.00756" rpy="0 0 0" />
+      <mass value="0.073" />
+      <inertia ixx="9.4062e-05" ixy="-1e-09" ixz="0.0"
+        iyy="2.8597e-05" iyz="2.9e-07" izz="7.7584e-05" />
     </inertial>
     <visual>
@@ -610,11 +616,11 @@
       <origin xyz="0 0 0" rpy="0 0 0" />
       <geometry>
-        <mesh filename="package://robot_description/tron2/SFYG_TRON2A/meshes/antenna_R_Link_collision1.STL" />
-      </geometry>
-    </collision>
-    <collision>
-      <origin xyz="0 0 0" rpy="0 0 0" />
-      <geometry>
-        <mesh filename="package://robot_description/tron2/SFYG_TRON2A/meshes/antenna_R_Link_collision2.STL" />
+        <mesh filename="package://robot_description/tron2/SFYG_TRON2A/meshes/antenna_R_Link_collision_1.STL" />
+      </geometry>
+    </collision>
+    <collision>
+      <origin xyz="0 0 0" rpy="0 0 0" />
+      <geometry>
+        <mesh filename="package://robot_description/tron2/SFYG_TRON2A/meshes/antenna_R_Link_collision_2.STL" />
       </geometry>
     </collision>
@@ -622,8 +628,8 @@
   <link name="camera_mount_Link">
     <inertial>
-      <origin xyz="0.002536 0.000321 -0.060392" rpy="0 0 0" />
-      <mass value="0.381" />
-      <inertia ixx="0.001630905" ixy="-3.911e-06" ixz="-0.000204624"
-        iyy="0.001504517" iyz="-3.269e-06" izz="0.000548227" />
+      <origin xyz="-0.019708 0.000381 -0.010581" rpy="0 0 0" />
+      <mass value="0.288" />
+      <inertia ixx="0.000766135" ixy="-6.264e-06" ixz="0.000325236"
+        iyy="0.001331301" iyz="-1.455e-06" izz="0.001742907" />
     </inertial>
     <visual>
@@ -637,5 +643,5 @@
       <origin xyz="0 0 0" rpy="0 0 0" />
       <geometry>
-        <mesh filename="package://robot_description/tron2/SFYG_TRON2A/meshes/camera_mount_Link_collision.STL" />
+        <mesh filename="package://robot_description/tron2/SFYG_TRON2A/meshes/camera_mount_Link.STL" />
       </geometry>
     </collision>
@@ -643,8 +649,8 @@
   <link name="radar_Link">
     <inertial>
-      <origin xyz="-4.8e-05 8.4e-05 0.03502" rpy="0 0 0" />
-      <mass value="0.394" />
-      <inertia ixx="0.000308871" ixy="6.27e-07" ixz="-4.96e-07"
-        iyy="0.000308088" iyz="8.62e-07" izz="0.000305305" />
+      <origin xyz="-0.001188 1e-06 0.037286" rpy="0 0 0" />
+      <mass value="0.406" />
+      <inertia ixx="0.000379149" ixy="5.2e-08" ixz="1.011e-06"
+        iyy="0.00036962" iyz="-3e-09" izz="0.000353387" />
     </inertial>
     <visual>
@@ -844,5 +850,5 @@
   </joint>
   <joint name="arm_base_Joint" type="fixed">
-    <origin xyz="0.006 0.0 0.0" rpy="0 0 0" />
+    <origin xyz="0.0 0.0 0.0" rpy="0 0 0" />
     <parent link="transition_Link" />
     <child link="arm_base_Link" />
@@ -910,10 +916,10 @@
   </joint>
   <joint name="antenna_L_Joint" type="fixed">
-    <origin xyz="-0.0025 0.16692 0.211" rpy="0 0 0" />
+    <origin xyz="-0.04365 0.1535 0.23765" rpy="0 0 0" />
     <parent link="base_Link" />
     <child link="antenna_L_Link" />
   </joint>
   <joint name="antenna_R_Joint" type="fixed">
-    <origin xyz="-0.0025 -0.16692 0.211" rpy="0 0 0" />
+    <origin xyz="-0.04365 -0.1535 0.23765" rpy="0 0 0" />
     <parent link="base_Link" />
     <child link="antenna_R_Link" />
@@ -925,6 +931,6 @@
   </joint>
   <joint name="radar_Joint" type="fixed">
-    <origin xyz="0.0 0.0 0.0" rpy="0 0 0" />
-    <parent link="camera_mount_Link" />
+    <origin xyz="0.18058 0.0 0.23876" rpy="0 0 0" />
+    <parent link="base_Link" />
     <child link="radar_Link" />
   </joint>

File: tron2a/WFYG_TRON2A/urdf/robot.urdf (robot description, URDF)
Before this commit: robot bipedal_robot, 29 links, 28 joints
Links:
- link antenna_L_Link: mass 0.231 -> 0.073; geometry collision mesh filename=package://bipedal_robot/meshes/antenna_L_Link_collision_1.S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; collision mesh filename=package://bipedal_robot/meshes/antenna_L_Link_collision_2.S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
- link antenna_R_Link: mass 0.231 -> 0.073; geometry collision mesh filename=package://bipedal_robot/meshes/antenna_R_Link_collision_1.S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; collision mesh filename=package://bipedal_robot/meshes/antenna_R_Link_collision_2.S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
- link camera_mount_Link: mass 0.381 -> 0.288; geometry collision mesh filename=package://bipedal_robot/meshes/camera_mount_Link.STL; visual mesh filename=package://bipedal_robot/meshes/camera_mount_Link.STL
- link radar_Link: mass 0.394 -> 0.406
- link transition_Link: geometry collision mesh filename=package://bipedal_robot/meshes/transition_Link_collision_1.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; collision mesh filename=package://bipedal_robot/meshes/transition_Link_collision_2.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
Joints:
- joint antenna_L_Joint: origin xyz=-0.0025 0.16692 0.211 rpy=0.0 0.0 0.0 -> xyz=-0.04365 0.1535 0.23765 rpy=0.0 0.0 0.0
- joint antenna_R_Joint: origin xyz=-0.0025 -0.16692 0.211 rpy=0.0 0.0 0.0 -> xyz=-0.04365 -0.1535 0.23765 rpy=0.0 0.0 0.0
- joint arm_base_Joint: origin xyz=0.006 0.0 0.0 rpy=0.0 0.0 0.0 -> xyz=0.0 0.0 0.0 rpy=0.0 0.0 0.0
- joint radar_Joint: origin xyz=0.0 0.0 0.0 rpy=0.0 0.0 0.0 -> xyz=0.18058 0.0 0.23876 rpy=0.0 0.0 0.0; parent camera_mount_Link -> base_Link

File: tron2a/WFYG_TRON2A/urdf/robot_rl.urdf (robot description, URDF)
Before this commit: robot bipedal_robot, 30 links, 29 joints
Links:
- link antenna_L_Link: mass 0.231 -> 0.073; geometry collision mesh filename=../meshes/antenna_L_Link_collision_1.STL; collision mesh filename=../meshes/antenna_L_Link_collision_2.STL
- link antenna_R_Link: mass 0.231 -> 0.073; geometry collision mesh filename=../meshes/antenna_R_Link_collision_1.STL; collision mesh filename=../meshes/antenna_R_Link_collision_2.STL
- link camera_mount_Link: mass 0.381 -> 0.288; geometry collision mesh filename=../meshes/camera_mount_Link.STL; visual mesh filename=../meshes/camera_mount_Link.STL
- link radar_Link: mass 0.394 -> 0.406
- link transition_Link: geometry collision mesh filename=../meshes/transition_Link_collision_1.STL; collision mesh filename=../meshes/transition_Link_collision_2.STL
Joints:
- joint antenna_L_Joint: origin xyz=-0.0025 0.16692 0.211 rpy=0.0 0.0 0.0 -> xyz=-0.04365 0.1535 0.23765 rpy=0.0 0.0 0.0
- joint antenna_R_Joint: origin xyz=-0.0025 -0.16692 0.211 rpy=0.0 0.0 0.0 -> xyz=-0.04365 -0.1535 0.23765 rpy=0.0 0.0 0.0
- joint arm_base_Joint: origin xyz=0.006 0.0 0.0 rpy=0.0 0.0 0.0 -> xyz=0.0 0.0 0.0 rpy=0.0 0.0 0.0
- joint radar_Joint: origin xyz=0.0 0.0 0.0 rpy=0.0 0.0 0.0 -> xyz=0.18058 0.0 0.23876 rpy=0.0 0.0 0.0; parent camera_mount_Link -> base_Link

File: tron2a/WFYG_TRON2A/xacro/robot.urdf.xacro (robot description, xacro)
@@ -304,8 +304,8 @@
   <link name="transition_Link">
     <inertial>
-      <origin xyz="-0.111727 0.000317 0.014516" rpy="0 0 0" />
+      <origin xyz="-0.109866 -0.002238 0.012131" rpy="0 0 0" />
       <mass value="1.117" />
-      <inertia ixx="0.002739303" ixy="6.6427e-05" ixz="0.000914255"
-        iyy="0.006871988" iyz="-2.0809e-05" izz="0.007888835" />
+      <inertia ixx="0.002748897" ixy="-0.000172411" ixz="0.00101041"
+        iyy="0.007134041" iyz="3.8511e-05" izz="0.008548272" />
     </inertial>
     <visual>
@@ -319,5 +319,11 @@
       <origin xyz="0 0 0" rpy="0 0 0" />
       <geometry>
-        <mesh filename="package://robot_description/tron2/WFYG_TRON2A/meshes/transition_Link_collision.STL" />
+        <mesh filename="package://robot_description/tron2/WFYG_TRON2A/meshes/transition_Link_collision_1.STL" />
+      </geometry>
+    </collision>
+    <collision>
+      <origin xyz="0 0 0" rpy="0 0 0" />
+      <geometry>
+        <mesh filename="package://robot_description/tron2/WFYG_TRON2A/meshes/transition_Link_collision_2.STL" />
       </geometry>
     </collision>
@@ -559,8 +565,8 @@
   <link name="antenna_L_Link">
     <inertial>
-      <origin xyz="-2.7e-05 -0.028426 0.013784" rpy="0 0 0" />
-      <mass value="0.231" />
-      <inertia ixx="0.000424493" ixy="-1.15e-07" ixz="-1.18e-07"
-        iyy="0.000169977" iyz="3.0807e-05" izz="0.00039175" />
+      <origin xyz="0.0 -0.025937 0.00756" rpy="0 0 0" />
+      <mass value="0.073" />
+      <inertia ixx="9.4062e-05" ixy="-1e-09" ixz="0.0"
+        iyy="2.8597e-05" iyz="-2.91e-07" izz="7.7585e-05" />
     </inertial>
     <visual>
@@ -574,11 +580,11 @@
       <origin xyz="0 0 0" rpy="0 0 0" />
       <geometry>
-        <mesh filename="package://robot_description/tron2/WFYG_TRON2A/meshes/antenna_L_Link_collision1.STL" />
-      </geometry>
-    </collision>
-    <collision>
-      <origin xyz="0 0 0" rpy="0 0 0" />
-      <geometry>
-        <mesh filename="package://robot_description/tron2/WFYG_TRON2A/meshes/antenna_L_Link_collision2.STL" />
+        <mesh filename="package://robot_description/tron2/WFYG_TRON2A/meshes/antenna_L_Link_collision_1.STL" />
+      </geometry>
+    </collision>
+    <collision>
+      <origin xyz="0 0 0" rpy="0 0 0" />
+      <geometry>
+        <mesh filename="package://robot_description/tron2/WFYG_TRON2A/meshes/antenna_L_Link_collision_2.STL" />
       </geometry>
     </collision>
@@ -586,8 +592,8 @@
   <link name="antenna_R_Link">
     <inertial>
-      <origin xyz="2.7e-05 0.028426 0.013784" rpy="0 0 0" />
-      <mass value="0.231" />
-      <inertia ixx="0.000424493" ixy="-1.15e-07" ixz="1.17e-07"
-        iyy="0.000169977" iyz="-3.0808e-05" izz="0.000391749" />
+      <origin xyz="0.0 0.025937 0.00756" rpy="0 0 0" />
+      <mass value="0.073" />
+      <inertia ixx="9.4062e-05" ixy="-1e-09" ixz="0.0"
+        iyy="2.8597e-05" iyz="2.9e-07" izz="7.7584e-05" />
     </inertial>
     <visual>
@@ -601,11 +607,11 @@
       <origin xyz="0 0 0" rpy="0 0 0" />
       <geometry>
-        <mesh filename="package://robot_description/tron2/WFYG_TRON2A/meshes/antenna_R_Link_collision1.STL" />
-      </geometry>
-    </collision>
-    <collision>
-      <origin xyz="0 0 0" rpy="0 0 0" />
-      <geometry>
-        <mesh filename="package://robot_description/tron2/WFYG_TRON2A/meshes/antenna_R_Link_collision2.STL" />
+        <mesh filename="package://robot_description/tron2/WFYG_TRON2A/meshes/antenna_R_Link_collision_1.STL" />
+      </geometry>
+    </collision>
+    <collision>
+      <origin xyz="0 0 0" rpy="0 0 0" />
+      <geometry>
+        <mesh filename="package://robot_description/tron2/WFYG_TRON2A/meshes/antenna_R_Link_collision_2.STL" />
       </geometry>
     </collision>
@@ -613,8 +619,8 @@
   <link name="camera_mount_Link">
     <inertial>
-      <origin xyz="0.002536 0.000321 -0.060392" rpy="0 0 0" />
-      <mass value="0.381" />
-      <inertia ixx="0.001630905" ixy="-3.911e-06" ixz="-0.000204624"
-        iyy="0.001504517" iyz="-3.269e-06" izz="0.000548227" />
+      <origin xyz="-0.019708 0.000381 -0.010581" rpy="0 0 0" />
+      <mass value="0.288" />
+      <inertia ixx="0.000766135" ixy="-6.264e-06" ixz="0.000325236"
+        iyy="0.001331301" iyz="-1.455e-06" izz="0.001742907" />
     </inertial>
     <visual>
@@ -628,5 +634,5 @@
       <origin xyz="0 0 0" rpy="0 0 0" />
       <geometry>
-        <mesh filename="package://robot_description/tron2/WFYG_TRON2A/meshes/camera_mount_Link_collision.STL" />
+        <mesh filename="package://robot_description/tron2/WFYG_TRON2A/meshes/camera_mount_Link.STL" />
       </geometry>
     </collision>
@@ -634,8 +640,8 @@
   <link name="radar_Link">
     <inertial>
-      <origin xyz="-4.8e-05 8.4e-05 0.03502" rpy="0 0 0" />
-      <mass value="0.394" />
-      <inertia ixx="0.000308871" ixy="6.27e-07" ixz="-4.96e-07"
-        iyy="0.000308088" iyz="8.62e-07" izz="0.000305305" />
+      <origin xyz="-0.001188 1e-06 0.037286" rpy="0 0 0" />
+      <mass value="0.406" />
+      <inertia ixx="0.000379149" ixy="5.2e-08" ixz="1.011e-06"
+        iyy="0.00036962" iyz="-3e-09" izz="0.000353387" />
     </inertial>
     <visual>
@@ -754,5 +760,5 @@
   </joint>
   <joint name="arm_base_Joint" type="fixed">
-    <origin xyz="0.006 0.0 0.0" rpy="0 0 0" />
+    <origin xyz="0.0 0.0 0.0" rpy="0 0 0" />
     <parent link="transition_Link" />
     <child link="arm_base_Link" />
@@ -820,10 +826,10 @@
   </joint>
   <joint name="antenna_L_Joint" type="fixed">
-    <origin xyz="-0.0025 0.16692 0.211" rpy="0 0 0" />
+    <origin xyz="-0.04365 0.1535 0.23765" rpy="0 0 0" />
     <parent link="base_Link" />
     <child link="antenna_L_Link" />
   </joint>
   <joint name="antenna_R_Joint" type="fixed">
-    <origin xyz="-0.0025 -0.16692 0.211" rpy="0 0 0" />
+    <origin xyz="-0.04365 -0.1535 0.23765" rpy="0 0 0" />
     <parent link="base_Link" />
     <child link="antenna_R_Link" />
@@ -835,6 +841,6 @@
   </joint>
   <joint name="radar_Joint" type="fixed">
-    <origin xyz="0.0 0.0 0.0" rpy="0 0 0" />
-    <parent link="camera_mount_Link" />
+    <origin xyz="0.18058 0.0 0.23876" rpy="0 0 0" />
+    <parent link="base_Link" />
     <child link="radar_Link" />
   </joint>
