Commit message: fix: correct arm6_Link inertia in SFYG / WFYG (TRON2A + TRON2B)
arm6_Link is a 7 g, 38 x 38 x 12 mm part whose mesh extends at most
1.9 cm from its CoM, so the sum of its principal moments cannot exceed
2 * m * r_max^2 ~= 5.2e-6 kg m^2. Several files carried principal
moments of ~(3.1e-4, 1.39e-3, 1.52e-3) kg m^2, about 600x over that
bound. The TRON2A MJCF, TRON2A robot_rl.urdf and TRON2A USD already
carried (7.6e-7, 7.6e-7, 1.4e-6), which matches the mesh-derived
uniform-density inertia; use that value everywhere.

Changed: TRON2A robot.urdf + xacro, and TRON2B MJCF, robot.urdf,
robot_rl.urdf and USD physics layer, for both SFYG and WFYG. All 18
arm6_Link definitions now have identical principal moments.

Refs #3

Co-Authored-By: Claude Opus 5.5 <noreply@anthropic.com>
Claude-Session: https://claude.ai/code/session_01X7zLMAMeCvAtsZnxUtPAdx
Signed-off-by: Claude <noreply@anthropic.com>

File: tron2a/SFYG_TRON2A/xacro/robot.urdf.xacro (robot description, xacro)
@@ -486,6 +486,6 @@
       <origin xyz="0.0 0.0 -0.0035" rpy="0 0 0" />
       <mass value="0.007" />
-      <inertia ixx="0.00152112" ixy="2.02e-06" ixz="2.61e-06"
-        iyy="0.00138626" iyz="2e-08" izz="0.00031152" />
+      <inertia ixx="0.00000076" ixy="0.0" ixz="0.0"
+        iyy="0.00000076" iyz="0.0" izz="0.0000014" />
     </inertial>
     <visual>

File: tron2a/WFYG_TRON2A/xacro/robot.urdf.xacro (robot description, xacro)
@@ -477,6 +477,6 @@
       <origin xyz="0.0 0.0 -0.0035" rpy="0 0 0" />
       <mass value="0.007" />
-      <inertia ixx="0.00152112" ixy="2.02e-06" ixz="2.61e-06"
-        iyy="0.00138626" iyz="2e-08" izz="0.00031152" />
+      <inertia ixx="0.00000076" ixy="0.0" ixz="0.0"
+        iyy="0.00000076" iyz="0.0" izz="0.0000014" />
     </inertial>
     <visual>
